File: pcb/001.sch (KiCad schematic (older format))
At the start: 6 parts, among them J1 AUDIO_JACK, P1 CONN_BATT, SW1 SW_POWER

Commit message: Began cleaning up ERC errors
Other:
- note added: "TODO: ESD protection"
Changed lines of the file:
@@
 	9450 2650 9450 2750
 $Comp
-L GND #PWR3
+L GND #PWR01
 U 1 1 56A6B291
 P 10400 2800
-F 0 "#PWR3" H 10400 2550 50  0001 C CNN
+F 0 "#PWR01" H 10400 2550 50  0001 C CNN
 F 1 "GND" H 10400 2650 50  0000 C CNN
 F 2 "" H 10400 2800 50  0000 C CNN
@@
 	8850 4550 9450 4550
 $Comp
-L GND #PWR1
+L GND #PWR02
 U 1 1 56A8BB9A
 P 9550 4550
-F 0 "#PWR1" H 9550 4300 50  0001 C CNN
+F 0 "#PWR02" H 9550 4300 50  0001 C CNN
 F 1 "GND" H 9550 4400 50  0000 C CNN
 F 2 "" H 9550 4550 50  0000 C CNN
@@
 Connection ~ 9450 4550
 $Comp
-L GND #PWR2
+L GND #PWR03
 U 1 1 56A8D7D0
 P 10000 5250
-F 0 "#PWR2" H 10000 5000 50  0001 C CNN
+F 0 "#PWR03" H 10000 5000 50  0001 C CNN
 F 1 "GND" H 10000 5100 50  0000 C CNN
 F 2 "" H 10000 5250 50  0000 C CNN
@@
 Wire Wire Line
 	6700 3150 7600 3150
+Text Notes 1650 3250 0    60   ~ 0
+TODO: ESD protection
+Text Notes 9100 5650 0    60   ~ 0
+TODO: ESD protection
 $EndSCHEMATC

Commit message: Latest work on footprints and BOM
Parts:
- J1: footprint (none) -> headphones:SJ1-351XN; Manufacturer (none) -> CUI; Manufacturer Part Number (none) -> SJ1-3513N
Changed lines of the file:
@@
 F 0 "J1" H 2000 2550 60  0000 C CNN
 F 1 "AUDIO_JACK" H 2000 1900 60  0000 C CNN
-F 2 "" H 2000 2650 60  0000 C CNN
+F 2 "headphones:SJ1-351XN" H 2000 2650 60  0000 C CNN
 F 3 "" H 2000 2650 60  0000 C CNN
+F 4 "CUI" H 2000 2450 60  0001 C CNN "Manufacturer"
+F 5 "SJ1-3513N" H 2000 2450 60  0001 C CNN "Manufacturer Part Number"
 	1    2000 2450
 	1    0    0    -1
