File: pcb/001.sch (KiCad schematic (older format))
At the start: 6 parts, among them J1 AUDIO_JACK, P1 CONN_BATT, SW1 SW_POWER

Commit message: Finished first pass at BOM
Parts:
- P1: footprint (none) -> Pin_Headers:Pin_Header_Straight_1x02_Pitch2.00mm; Manufacturer (none) -> JST; Manufacturer Part Number (none) -> B2B-PH-K-S
- SW1: footprint (none) -> headphones:SWITCH_SPDT_OS; Manufacturer (none) -> C&K Components; Manufacturer Part Number (none) -> OS102011MS2QN1
Changed lines of the file:
@@
 	9450 2650 9450 2750
 $Comp
-L GND #PWR3
+L GND #PWR01
 U 1 1 56A6B291
 P 10400 2800
-F 0 "#PWR3" H 10400 2550 50  0001 C CNN
+F 0 "#PWR01" H 10400 2550 50  0001 C CNN
 F 1 "GND" H 10400 2650 50  0000 C CNN
 F 2 "" H 10400 2800 50  0000 C CNN
@@
 F 0 "P1" H 9500 4500 50  0000 C CNN
 F 1 "CONN_BATT" V 9600 4350 50  0000 C CNN
-F 2 "" H 9500 4350 50  0000 C CNN
+F 2 "Pin_Headers:Pin_Header_Straight_1x02_Pitch2.00mm" H 9500 4350 50  0001 C CNN
 F 3 "" H 9500 4350 50  0000 C CNN
+F 4 "JST" H 9500 4350 60  0001 C CNN "Manufacturer"
+F 5 "B2B-PH-K-S" H 9500 4350 60  0001 C CNN "Manufacturer Part Number"
 	1    9500 4350
 	0    -1   -1   0
@@
 	8850 4550 9450 4550
 $Comp
-L GND #PWR1
+L GND #PWR02
 U 1 1 56A8BB9A
 P 9550 4550
-F 0 "#PWR1" H 9550 4300 50  0001 C CNN
+F 0 "#PWR02" H 9550 4300 50  0001 C CNN
 F 1 "GND" H 9550 4400 50  0000 C CNN
 F 2 "" H 9550 4550 50  0000 C CNN
@@
 F 0 "SW1" H 9300 5300 50  0000 C CNN
 F 1 "SW_POWER" H 9350 5000 50  0000 C CNN
-F 2 "" H 9500 5150 50  0000 C CNN
+F 2 "headphones:SWITCH_SPDT_OS" H 9500 5150 50  0001 C CNN
 F 3 "" H 9500 5150 50  0000 C CNN
+F 4 "C&K Components" H 9500 5150 60  0001 C CNN "Manufacturer"
+F 5 "OS102011MS2QN1" H 9500 5150 60  0001 C CNN "Manufacturer Part Number"
 	1    9500 5150
 	1    0    0    -1
@@
 Connection ~ 9450 4550
 $Comp
-L GND #PWR2
+L GND #PWR03
 U 1 1 56A8D7D0
 P 10000 5250
-F 0 "#PWR2" H 10000 5000 50  0001 C CNN
+F 0 "#PWR03" H 10000 5000 50  0001 C CNN
 F 1 "GND" H 10000 5100 50  0000 C CNN
 F 2 "" H 10000 5250 50  0000 C CNN
