File: pcb/001.sch (KiCad schematic (older format))
At the start: 6 parts, among them J1 AUDIO_JACK, P1 CONN_BATT, SW1 SW_POWER

Commit message: Fixing up some part numbers
Parts:
- P1: Manufacturer Part Number B2B-PH-K-S -> B2B-PH-K-S(LF)(SN)
Changed lines of the file:
@@
 F 3 "" H 9500 4350 50  0000 C CNN
 F 4 "JST" H 9500 4350 60  0001 C CNN "Manufacturer"
-F 5 "B2B-PH-K-S" H 9500 4350 60  0001 C CNN "Manufacturer Part Number"
+F 5 "B2B-PH-K-S(LF)(SN)" H 9500 4350 60  0001 C CNN "Manufacturer Part Number"
 	1    9500 4350
 	0    -1   -1   0
