File: pcb/xc6slx9.sch (KiCad schematic (older format))
At the start: 50 parts, among them SW2 SW_RESET, U12 24C16, U13 W25Q64FVSSIG, U14 XC6SLX9TQG144, X3 12.288MHz

Commit message: Cleaned up ERC
Parts:
- added R97, R98, R99: 0, symbol R
Connections:
- wire segments 162 -> 163
- no-connect marks 64 -> 67

Commit message: Latest work on footprints and BOM
Changed lines of the file:
@@
 	13450 3500 13350 3500
 Wire Wire Line
-	13350 3700 13350 3500
+	13350 3500 13350 3700
 Wire Wire Line
 	11950 3700 13450 3700

Commit message: Started filling out FPGA sheet BOM
Parts:
- D12: footprint (none) -> LEDs:LED_0603; Manufacturer (none) -> Lite-On; Manufacturer Part Number (none) -> LTST-C191KRKT
- D13: footprint (none) -> LEDs:LED_0603; Manufacturer (none) -> Lite-On; Manufacturer Part Number (none) -> LTST-C191KGKT
- R75, R99: footprint (none) -> Resistors_SMD:R_0603; Manufacturer (none) -> Panasonic; Manufacturer Part Number (none) -> ERJ-3GEY0R00V
- R76, R81, R82, R87, R88, R89, R90, R93: footprint (none) -> Resistors_SMD:R_0603; Manufacturer (none) -> Panasonic; Manufacturer Part Number (none) -> ERJ-3EKF68R0V
- R77, R78: footprint (none) -> Resistors_SMD:R_0603; Manufacturer (none) -> Panasonic; Manufacturer Part Number (none) -> ERJ-3GEYJ103V
- R79, R80: footprint (none) -> Resistors_SMD:R_0603; Manufacturer (none) -> Panasonic; Manufacturer Part Number (none) -> ERJ-3GEYJ472V
- R83: footprint (none) -> Resistors_SMD:R_0603; Manufacturer (none) -> Panasonic; Manufacturer Part Number (none) -> ERJ-3EKF2401V
- R84: value 4.7K -> 0; footprint (none) -> Resistors_SMD:R_0603; Manufacturer (none) -> Panasonic; Manufacturer Part Number (none) -> ERJ-3GEY0R00V
- R85: value 68 -> 4.7K; footprint (none) -> Resistors_SMD:R_0603; Manufacturer (none) -> Panasonic; Manufacturer Part Number (none) -> ERJ-3GEYJ472V
- R86: value 68 -> 0; footprint (none) -> Resistors_SMD:R_0603; Manufacturer (none) -> Panasonic; Manufacturer Part Number (none) -> ERJ-3GEY0R00V
- R91: footprint (none) -> Resistors_SMD:R_0603; Manufacturer (none) -> Panasonic; Manufacturer Part Number (none) -> ERJ-3EKF3300V
- R92: value 4.7K -> 68; footprint (none) -> Resistors_SMD:R_0603; Manufacturer (none) -> Panasonic; Manufacturer Part Number (none) -> ERJ-3EKF68R0V
- R97: value 0 -> 4.7K; footprint (none) -> Resistors_SMD:R_0603; Manufacturer (none) -> Panasonic; Manufacturer Part Number (none) -> ERJ-3GEYJ472V
- R98: value 0 -> 68; footprint (none) -> Resistors_SMD:R_0603; Manufacturer (none) -> Panasonic; Manufacturer Part Number (none) -> ERJ-3EKF68R0V
- U14: footprint (none) -> Housings_QFP:TQFP-144_20x20mm_Pitch0.5mm; Manufacturer (none) -> Xilinx; Manufacturer Part Number (none) -> XC6SLX9-2TQG144C
- X3: footprint (none) -> headphones:Oscillator_SMD_2520_4Pads; Manufacturer (none) -> Microchip; Manufacturer Part Number (none) -> DSC1033DI2-012.2880
Other:
- note added: "Green"
- note added: "Red"

Commit message: Switched to microchip SPI flash
Parts:
- removed U13: W25Q64FVSSIG, symbol W25Q64FVSSIG
- added U13: M25P40, symbol M25P40
Connections:
- wire segments 163 -> 227

Commit message: Picked components for FPGA sheet
Parts:
- C72, C73, C74: footprint (none) -> Capacitors_SMD:C_0603; Manufacturer (none) -> Murata; Manufacturer Part Number (none) -> GRM188R61C104KA01
- C75, C76, C77, C78, C79, C80, C81, C82, C83, C84, C85, C86, C87: footprint (none) -> Capacitors_SMD:C_0603; Manufacturer (none) -> Murata; Manufacturer Part Number (none) -> GRM188R61A475KE15
- C88, C89, C90, C91, C92, C93, C94, C95: footprint (none) -> Capacitors_SMD:C_0603; Manufacturer (none) -> Murata; Manufacturer Part Number (none) -> GRM188R61A474KA61
- SW2: footprint (none) -> headphones:SW_PUSH_6X6; Manufacturer (none) -> Omron; Manufacturer Part Number (none) -> B3F-1000
- U12: footprint (none) -> Housings_SOIC:SOIC-8_3.9x4.9mm_Pitch1.27mm; Manufacturer (none) -> ON Semiconductor; Manufacturer Part Number (none) -> CAT24C16WI
- U13: footprint (none) -> Housings_SOIC:SOIC-8_3.9x4.9mm_Pitch1.27mm; Manufacturer (none) -> Micron; Manufacturer Part Number (none) -> M25P40-VMN6TPB
Connections:
- wire segments 227 -> 163
