File: pcb/xc6slx9.sch (KiCad schematic (older format))
At the start: 53 parts, among them SW2 SW_RESET, U12 24C16, U13 M25P40, U14 XC6SLX9TQG144, X3 12.288MHz

Commit message: Reordering the ADC->FPGA pins for layout
Changed lines of the file:
@@
 	13350 3300 13450 3300
 Connection ~ 13350 3200
-Text HLabel 4250 2000 0    60   Output ~ 0
+Text HLabel 4250 3200 0    60   Output ~ 0
 ADC_RST
-Text HLabel 4250 2100 0    60   Input ~ 0
+Text HLabel 4250 2700 0    60   Input ~ 0
 ADC_OVFL
-Text HLabel 4250 2400 0    60   Output ~ 0
+Text HLabel 4250 2200 0    60   Output ~ 0
 ADC_HPF
 Text HLabel 4250 3100 0    60   Input ~ 0
@@
 Text HLabel 4250 2900 0    60   Output ~ 0
 ADC_MCLK
-Text HLabel 4250 3200 0    60   Input ~ 0
+Text HLabel 4250 2000 0    60   Input ~ 0
 ADC_SDO
-Text HLabel 4250 2200 0    60   Output ~ 0
+Text HLabel 4250 2300 0    60   Output ~ 0
 ADC_I2S_LJ
-Text HLabel 4250 2300 0    60   Output ~ 0
+Text HLabel 4250 2400 0    60   Output ~ 0
 ADC_MS
 Text HLabel 4250 2500 0    60   Output ~ 0
@@
 Text HLabel 4250 2600 0    60   Output ~ 0
 ADC_M1
-Text HLabel 4250 2700 0    60   Output ~ 0
+Text HLabel 4250 2100 0    60   Output ~ 0
 ADC_MDIV
 Wire Wire Line

Commit message: Finished pin swapping the FPGA ADC signals
Still not super jazzed about how coupled the ADC I2S traces are, and I
need to look into the MCLK situation for the ADC.  Ideally the FPGA
shouldn't be generating it since it's a lousy clock driver.  Will
probably need another oscillator for the ADC same as the FPGA and DAC.
Changed lines of the file:
@@
 	13350 3300 13450 3300
 Connection ~ 13350 3200
-Text HLabel 4250 3200 0    60   Output ~ 0
+Text HLabel 4250 2700 0    60   Output ~ 0
 ADC_RST
-Text HLabel 4250 2700 0    60   Input ~ 0
+Text HLabel 4250 2600 0    60   Input ~ 0
 ADC_OVFL
 Text HLabel 4250 2200 0    60   Output ~ 0
 ADC_HPF
+Text HLabel 4250 3000 0    60   Input ~ 0
+ADC_LRCLK
 Text HLabel 4250 3100 0    60   Input ~ 0
-ADC_LRCLK
-Text HLabel 4250 3000 0    60   Input ~ 0
 ADC_SCLK
-Text HLabel 4250 2900 0    60   Output ~ 0
+Text HLabel 4250 3200 0    60   Output ~ 0
 ADC_MCLK
 Text HLabel 4250 2000 0    60   Input ~ 0
@@
 Text HLabel 4250 2300 0    60   Output ~ 0
 ADC_I2S_LJ
+Text HLabel 4250 2900 0    60   Output ~ 0
+ADC_MS
 Text HLabel 4250 2400 0    60   Output ~ 0
-ADC_MS
+ADC_M0
 Text HLabel 4250 2500 0    60   Output ~ 0
-ADC_M0
-Text HLabel 4250 2600 0    60   Output ~ 0
 ADC_M1
 Text HLabel 4250 2100 0    60   Output ~ 0
@@
 	4250 3100 5300 3100
 Wire Wire Line
-	4250 3200 5300 3200
-Wire Wire Line
-	4750 2900 5300 2900
-Wire Wire Line
-	4250 2900 4450 2900
+	4250 2900 5300 2900
 $Comp
 L GND #PWR0164
@@
 L R R82
 U 1 1 57183388
-P 4600 2900
-F 0 "R82" V 4550 2700 50  0000 C CNN
-F 1 "68" V 4600 2900 50  0000 C CNN
-F 2 "Resistors_SMD:R_0603" V 4530 2900 50  0001 C CNN
-F 3 "" H 4600 2900 50  0000 C CNN
-F 4 "Panasonic" V 4600 2900 60  0001 C CNN "Manufacturer"
-F 5 "ERJ-3EKF68R0V" V 4600 2900 60  0001 C CNN "Manufacturer Part Number"
-	1    4600 2900
+P 4600 3200
+F 0 "R82" V 4550 3000 50  0000 C CNN
+F 1 "68" V 4600 3200 50  0000 C CNN
+F 2 "Resistors_SMD:R_0603" V 4530 3200 50  0001 C CNN
+F 3 "" H 4600 3200 50  0000 C CNN
+F 4 "Panasonic" V 4600 3200 60  0001 C CNN "Manufacturer"
+F 5 "ERJ-3EKF68R0V" V 4600 3200 60  0001 C CNN "Manufacturer Part Number"
+	1    4600 3200
 	0    1    1    0
 $EndComp
@@
 	1    0    0    -1
 $EndComp
+Wire Wire Line
+	4250 3200 4450 3200
+Wire Wire Line
+	4750 3200 5300 3200
 $EndSCHEMATC

Commit message: Added an oscillator for the ADC
Parts:
- removed R82: 68, Resistors_SMD:R_0603, symbol R
Connections:
- net labels added: ADC_MCLK_EN
- net labels removed: ADC_MCLK
- wire segments 163 -> 162

Commit message: Replaced output test pads with an audio jack
Changed lines of the file:
@@
 	13450 3500 13350 3500
 Wire Wire Line
-	13350 3700 13350 3500
+	13350 3500 13350 3700
 Wire Wire Line
 	11950 3700 13450 3700

Commit message: Fixed placement of series termination resistors
I had the logical placement of the series termination resistors wrong
in the schematics (i.e. I had them placed at the source rather than
the load) so I moved all those around to the correct sheets.  I also
moved the ADC resistors in the layout, but haven't gotten to the DAC
ones yet.
Parts:
- removed R87, R88, R89, R92, R93: 68, Resistors_SMD:R_0603, symbol R
- added R2, R3, R4: 68, Resistors_SMD:R_0603, symbol R
Connections:
- wire segments 162 -> 160
Changed lines of the file:
@@
 ADC_MDIV
-Wire Wire Line
-	4250 2000 5300 2000
 Wire Wire Line
 	4250 2100 5300 2100
@@
 Text HLabel 7750 2900 0    60   Output ~ 0
 DAC_RST
-Wire Wire Line
-	4250 3000 5300 3000
-Wire Wire Line
-	4250 3100 5300 3100
 Wire Wire Line
 	4250 2900 5300 2900
@@
 	7750 2500 8700 2500
 Wire Wire Line
-	7750 2400 8050 2400
-Wire Wire Line
-	8350 2400 8700 2400
-Wire Wire Line
-	8700 2300 8350 2300
-Wire Wire Line
-	7750 2300 8050 2300
+	7750 2400 8700 2400
+Wire Wire Line
+	7750 2300 8700 2300
 Wire Wire Line
 	7750 2200 8050 2200
 Wire Wire Line
-	7750 2100 8050 2100
-Wire Wire Line
-	7750 2000 8050 2000
-Wire Wire Line
-	7750 1900 8050 1900
-Wire Wire Line
-	8350 1900 8700 1900
-Wire Wire Line
-	8350 2000 8700 2000
-Wire Wire Line
-	8350 2100 8700 2100
+	7750 2100 8700 2100
+Wire Wire Line
+	7750 2000 8700 2000
+Wire Wire Line
+	7750 1900 8700 1900
 Wire Wire Line
 	8350 2200 8700 2200
@@
 $EndComp
 $Comp
-L R R87
-U 1 1 5718481E
-P 8200 1900
-F 0 "R87" V 8150 1700 50  0000 C CNN
-F 1 "68" V 8200 1900 50  0000 C CNN
-F 2 "Resistors_SMD:R_0603" V 8130 1900 50  0001 C CNN
-F 3 "" H 8200 1900 50  0000 C CNN
-F 4 "Panasonic" V 8200 1900 60  0001 C CNN "Manufacturer"
-F 5 "ERJ-3EKF68R0V" V 8200 1900 60  0001 C CNN "Manufacturer Part Number"
-	1    8200 1900
-	0    1    1    0
-$EndComp
-$Comp
-L R R88
-U 1 1 57184947
-P 8200 2000
-F 0 "R88" V 8150 1800 50  0000 C CNN
-F 1 "68" V 8200 2000 50  0000 C CNN
-F 2 "Resistors_SMD:R_0603" V 8130 2000 50  0001 C CNN
-F 3 "" H 8200 2000 50  0000 C CNN
-F 4 "Panasonic" V 8200 2000 60  0001 C CNN "Manufacturer"
-F 5 "ERJ-3EKF68R0V" V 8200 2000 60  0001 C CNN "Manufacturer Part Number"
-	1    8200 2000
-	0    1    1    0
-$EndComp
-$Comp
-L R R89
-U 1 1 571849FD
-P 8200 2100
-F 0 "R89" V 8150 1900 50  0000 C CNN
-F 1 "68" V 8200 2100 50  0000 C CNN
-F 2 "Resistors_SMD:R_0603" V 8130 2100 50  0001 C CNN
-F 3 "" H 8200 2100 50  0000 C CNN
-F 4 "Panasonic" V 8200 2100 60  0001 C CNN "Manufacturer"
-F 5 "ERJ-3EKF68R0V" V 8200 2100 60  0001 C CNN "Manufacturer Part Number"
-	1    8200 2100
-	0    1    1    0
-$EndComp
-$Comp
 L R R90
 U 1 1 57184AB6
@@
 $EndComp
 $Comp
-L R R92
-U 1 1 57184B72
-P 8200 2300
-F 0 "R92" V 8150 2100 50  0000 C CNN
-F 1 "68" V 8200 2300 50  0000 C CNN
-F 2 "Resistors_SMD:R_0603" V 8130 2300 50  0001 C CNN
-F 3 "" H 8200 2300 50  0000 C CNN
-F 4 "Panasonic" V 8200 2300 60  0001 C CNN "Manufacturer"
-F 5 "ERJ-3EKF68R0V" V 8200 2300 60  0001 C CNN "Manufacturer Part Number"
-	1    8200 2300
-	0    1    1    0
-$EndComp
-$Comp
-L R R93
-U 1 1 57184C31
-P 8200 2400
-F 0 "R93" V 8150 2200 50  0000 C CNN
-F 1 "68" V 8200 2400 50  0000 C CNN
-F 2 "Resistors_SMD:R_0603" V 8130 2400 50  0001 C CNN
-F 3 "" H 8200 2400 50  0000 C CNN
-F 4 "Panasonic" V 8200 2400 60  0001 C CNN "Manufacturer"
-F 5 "ERJ-3EKF68R0V" V 8200 2400 60  0001 C CNN "Manufacturer Part Number"
-	1    8200 2400
-	0    1    1    0
-$EndComp
-$Comp
 L R R81
 U 1 1 57186515
@@
 Wire Wire Line
 	4250 3200 5300 3200
+$Comp
+L R R3
+U 1 1 574D9505
+P 4700 3000
+F 0 "R3" V 4650 2800 50  0000 C CNN
+F 1 "68" V 4700 3000 50  0000 C CNN
+F 2 "Resistors_SMD:R_0603" V 4630 3000 50  0001 C CNN
+F 3 "" H 4700 3000 50  0000 C CNN
+F 4 "Panasonic" V 4700 3000 60  0001 C CNN "Manufacturer"
+F 5 "ERJ-3EKF68R0V" V 4700 3000 60  0001 C CNN "Manufacturer Part Number"
+	1    4700 3000
+	0    1    1    0
+$EndComp
+$Comp
+L R R4
+U 1 1 574D950E
+P 4700 3100
+F 0 "R4" V 4650 2900 50  0000 C CNN
+F 1 "68" V 4700 3100 50  0000 C CNN
+F 2 "Resistors_SMD:R_0603" V 4630 3100 50  0001 C CNN
+F 3 "" H 4700 3100 50  0000 C CNN
+F 4 "Panasonic" V 4700 3100 60  0001 C CNN "Manufacturer"
+F 5 "ERJ-3EKF68R0V" V 4700 3100 60  0001 C CNN "Manufacturer Part Number"
+	1    4700 3100
+	0    1    1    0
+$EndComp
+Wire Wire Line
+	4250 3000 4550 3000
+Wire Wire Line
+	4250 3100 4550 3100
+Wire Wire Line
+	4850 3000 5300 3000
+Wire Wire Line
+	4850 3100 5300 3100
+$Comp
+L R R2
+U 1 1 574DAAB4
+P 4700 2000
+F 0 "R2" V 4650 1800 50  0000 C CNN
+F 1 "68" V 4700 2000 50  0000 C CNN
+F 2 "Resistors_SMD:R_0603" V 4630 2000 50  0001 C CNN
+F 3 "" H 4700 2000 50  0000 C CNN
+F 4 "Panasonic" V 4700 2000 60  0001 C CNN "Manufacturer"
+F 5 "ERJ-3EKF68R0V" V 4700 2000 60  0001 C CNN "Manufacturer Part Number"
+	1    4700 2000
+	0    1    1    0
+$EndComp
+Wire Wire Line
+	4850 2000 5300 2000
+Wire Wire Line
+	4550 2000 4250 2000
 $EndSCHEMATC

Commit message: Cleaned up a lot of the FT2232D->FPGA connections
Moved the series termination resistors into the right spots and
cleaned up and aligned all the traces to the FPGA.
Parts:
- removed R98: 68, Resistors_SMD:R_0603, symbol R
- added R38, R39, R89: 68, Resistors_SMD:R_0603, symbol R
