File: pcb/xc6slx9.sch (KiCad schematic (older format))
At the start: 52 parts, among them SW2 SW_RESET, U12 24C16, U13 M25P40, U14 XC6SLX9TQG144, X3 12.288MHz

Commit message: Fixing up USB connector
- Had to go back through and re-annotate all the 0603 caps and
  resistors to the hand-solderding versions since those changes didn't
  make it back into the schematics the last time I tried.

- Added a new footprint for the USB connector to connect to all the
  shield pins.
Parts:
- C72, C73, C74, C75, C76, C77, C78, C79, C80, C81, C82, C83, C84, C85, C86, C87, C88, C89, C90, C91, C92, C93, C94, C95: footprint Capacitors_SMD:C_0603 -> Capacitors_SMD:C_0603_HandSoldering
- R2, R3, R38, R39, R4, R75, R76, R77, R78, R79, R80, R81, R83, R84, R85, R86, R89, R90, R91, R97, R99: footprint Resistors_SMD:R_0603 -> Resistors_SMD:R_0603_HandSoldering

Commit message: Added sense resistors everywhere
Parts:
- added P3: CONN_01X07, Pin_Headers:Pin_Header_Straight_1x07, symbol CONN_01X07
- added P4, P5: CONN_01X12, Pin_Headers:Pin_Header_Straight_1x12, symbol CONN_01X12
- added R121, R122, R123, R124, R125, R126, R127, R128: 0.01, symbol R
Connections:
- net labels added: VCCAUX, VCCINT, VCCO_0, VCCO_1, VCCO_2
- wire segments 160 -> 203
Other:
- note added: "DEBUG CONNECTIONS"

Commit message: Still need to route all the new resistors
Parts:
- R121, R122, R123, R124, R125, R126, R127, R128: footprint (none) -> Resistors_SMD:R_0603_HandSoldering
Changed lines of the file:
@@
 F 0 "R128" V 11830 1900 50  0000 C CNN
 F 1 "0.01" V 11750 1900 50  0000 C CNN
-F 2 "" V 11680 1900 50  0000 C CNN
+F 2 "Resistors_SMD:R_0603_HandSoldering" V 11680 1900 50  0001 C CNN
 F 3 "" H 11750 1900 50  0000 C CNN
 	1    11750 1900
@@
 	13450 3500 13350 3500
 Wire Wire Line
-	13350 3700 13350 3500
+	13350 3500 13350 3700
 Wire Wire Line
 	11550 3700 13450 3700
@@
 F 0 "R124" V 10480 2500 50  0000 C CNN
 F 1 "0.01" V 10400 2500 50  0000 C CNN
-F 2 "" V 10330 2500 50  0000 C CNN
+F 2 "Resistors_SMD:R_0603_HandSoldering" V 10330 2500 50  0001 C CNN
 F 3 "" H 10400 2500 50  0000 C CNN
 	1    10400 2500
@@
 F 0 "R125" V 11480 3300 50  0000 C CNN
 F 1 "0.01" V 11400 3300 50  0000 C CNN
-F 2 "" V 11330 3300 50  0000 C CNN
+F 2 "Resistors_SMD:R_0603_HandSoldering" V 11330 3300 50  0001 C CNN
 F 3 "" H 11400 3300 50  0000 C CNN
 	1    11400 3300
@@
 F 0 "R126" V 11480 3700 50  0000 C CNN
 F 1 "0.01" V 11400 3700 50  0000 C CNN
-F 2 "" V 11330 3700 50  0000 C CNN
+F 2 "Resistors_SMD:R_0603_HandSoldering" V 11330 3700 50  0001 C CNN
 F 3 "" H 11400 3700 50  0000 C CNN
 	1    11400 3700
@@
 F 0 "R127" V 11480 4300 50  0000 C CNN
 F 1 "0.01" V 11400 4300 50  0000 C CNN
-F 2 "" V 11330 4300 50  0000 C CNN
+F 2 "Resistors_SMD:R_0603_HandSoldering" V 11330 4300 50  0001 C CNN
 F 3 "" H 11400 4300 50  0000 C CNN
 	1    11400 4300
@@
 F 0 "R122" V 1830 2800 50  0000 C CNN
 F 1 "0.01" V 1750 2800 50  0000 C CNN
-F 2 "" V 1680 2800 50  0000 C CNN
+F 2 "Resistors_SMD:R_0603_HandSoldering" V 1680 2800 50  0001 C CNN
 F 3 "" H 1750 2800 50  0000 C CNN
 	1    1750 2800
@@
 F 0 "R121" V 1330 7600 50  0000 C CNN
 F 1 "0.01" V 1250 7600 50  0000 C CNN
-F 2 "" V 1180 7600 50  0000 C CNN
+F 2 "Resistors_SMD:R_0603_HandSoldering" V 1180 7600 50  0001 C CNN
 F 3 "" H 1250 7600 50  0000 C CNN
 	1    1250 7600
@@
 F 0 "R123" V 2830 6200 50  0000 C CNN
 F 1 "0.01" V 2750 6200 50  0000 C CNN
-F 2 "" V 2680 6200 50  0000 C CNN
+F 2 "Resistors_SMD:R_0603_HandSoldering" V 2680 6200 50  0001 C CNN
 F 3 "" H 2750 6200 50  0000 C CNN
 	1    2750 6200

Commit message: Cleanup and added testpoints
Cleaned up some of the schematic layout without changing any nets.  Also
added testpoints to all the power rails for easy debug.
Connections:
- wire segments 203 -> 271

Commit message: More cleanup and switched sense resistors
Increased the resistance of the current sense resistors up to 0.1 ohm.
Parts:
- R121, R122, R123, R124, R125, R126, R127, R128: value 0.01 -> 0.1
Changed lines of the file:
@@
 P 12200 1900
 F 0 "R128" V 12280 1900 50  0000 C CNN
-F 1 "0.01" V 12200 1900 50  0000 C CNN
+F 1 "0.1" V 12200 1900 50  0000 C CNN
 F 2 "Resistors_SMD:R_0603_HandSoldering" V 12130 1900 50  0001 C CNN
 F 3 "" H 12200 1900 50  0000 C CNN
@@
 P 10850 2500
 F 0 "R124" V 10930 2500 50  0000 C CNN
-F 1 "0.01" V 10850 2500 50  0000 C CNN
+F 1 "0.1" V 10850 2500 50  0000 C CNN
 F 2 "Resistors_SMD:R_0603_HandSoldering" V 10780 2500 50  0001 C CNN
 F 3 "" H 10850 2500 50  0000 C CNN
@@
 P 11850 3300
 F 0 "R125" V 11930 3300 50  0000 C CNN
-F 1 "0.01" V 11850 3300 50  0000 C CNN
+F 1 "0.1" V 11850 3300 50  0000 C CNN
 F 2 "Resistors_SMD:R_0603_HandSoldering" V 11780 3300 50  0001 C CNN
 F 3 "" H 11850 3300 50  0000 C CNN
@@
 P 11850 3700
 F 0 "R126" V 11930 3700 50  0000 C CNN
-F 1 "0.01" V 11850 3700 50  0000 C CNN
+F 1 "0.1" V 11850 3700 50  0000 C CNN
 F 2 "Resistors_SMD:R_0603_HandSoldering" V 11780 3700 50  0001 C CNN
 F 3 "" H 11850 3700 50  0000 C CNN
@@
 P 11850 4300
 F 0 "R127" V 11930 4300 50  0000 C CNN
-F 1 "0.01" V 11850 4300 50  0000 C CNN
+F 1 "0.1" V 11850 4300 50  0000 C CNN
 F 2 "Resistors_SMD:R_0603_HandSoldering" V 11780 4300 50  0001 C CNN
 F 3 "" H 11850 4300 50  0000 C CNN
@@
 P 1750 2800
 F 0 "R122" V 1830 2800 50  0000 C CNN
-F 1 "0.01" V 1750 2800 50  0000 C CNN
+F 1 "0.1" V 1750 2800 50  0000 C CNN
 F 2 "Resistors_SMD:R_0603_HandSoldering" V 1680 2800 50  0001 C CNN
 F 3 "" H 1750 2800 50  0000 C CNN
@@
 P 1250 7600
 F 0 "R121" V 1330 7600 50  0000 C CNN
-F 1 "0.01" V 1250 7600 50  0000 C CNN
+F 1 "0.1" V 1250 7600 50  0000 C CNN
 F 2 "Resistors_SMD:R_0603_HandSoldering" V 1180 7600 50  0001 C CNN
 F 3 "" H 1250 7600 50  0000 C CNN
@@
 P 2750 6200
 F 0 "R123" V 2830 6200 50  0000 C CNN
-F 1 "0.01" V 2750 6200 50  0000 C CNN
+F 1 "0.1" V 2750 6200 50  0000 C CNN
 F 2 "Resistors_SMD:R_0603_HandSoldering" V 2680 6200 50  0001 C CNN
 F 3 "" H 2750 6200 50  0000 C CNN

Commit message: Ran DRC and added some more notes
Connections:
- wire segments 271 -> 204

Commit message: Traces on a plane
- Finished placing testpoints and got footprints for them
- Cleaned up the last of the unconnected tracks
- Switched up supply rails for PWRGOOD LEDs
Parts:
- D12, D13: symbol LED -> LED-RESCUE-NYCDB-01
