File: pcb/ti_dac.sch (KiCad schematic (older format))
At the start: 45 parts, among them U10 OPA4134, U11 TPA6120A2, U9 PCM1792A, X2 12.288MHz

Commit message: Moved kicad design under pcb/
Connections:
- wire segments 216 -> 166
Changed lines of the file:
@@
 $EndComp
 Wire Wire Line
-	3900 950  3900 1000
-Wire Wire Line
-	3900 1000 3900 1050
-Wire Wire Line
-	3450 1000 3600 1000
-Wire Wire Line
-	3600 1000 3900 1000
+	3900 950  3900 1050
+Wire Wire Line
+	3450 1000 3900 1000
 Wire Wire Line
 	3600 1000 3600 1050
 Connection ~ 3900 1000
 Wire Wire Line
-	3900 1350 3900 1400
-Wire Wire Line
-	3900 1400 3900 1450
+	3900 1350 3900 1450
 Wire Wire Line
 	3900 1400 3600 1400
@@
 	3150 4850 3150 4900
 Wire Wire Line
-	3150 4900 3250 4900
-Wire Wire Line
-	3250 4900 3350 4900
-Wire Wire Line
-	3350 4900 3450 4900
-Wire Wire Line
-	3450 4900 3550 4900
-Wire Wire Line
-	3350 4850 3350 4900
-Wire Wire Line
-	3350 4900 3350 4950
+	3150 4900 3550 4900
+Wire Wire Line
+	3350 4850 3350 4950
 Wire Wire Line
 	3550 4900 3550 4850
@@
 $EndComp
 Wire Wire Line
-	10550 950  10550 1000
-Wire Wire Line
-	10550 1000 10550 1050
+	10550 950  10550 1050
 Wire Wire Line
 	10550 1000 10850 1000
@@
 Connection ~ 10550 1000
 Wire Wire Line
-	10550 1350 10550 1400
-Wire Wire Line
-	10550 1400 10550 1450
+	10550 1350 10550 1450
 Wire Wire Line
 	10550 1400 10850 1400
@@
 Connection ~ 10550 1400
 Wire Wire Line
-	10150 1350 10150 1400
-Wire Wire Line
-	10150 1400 10150 1450
+	10150 1350 10150 1450
 Wire Wire Line
 	10150 1400 9850 1400
@@
 	9850 1000 10150 1000
 Wire Wire Line
-	10150 950  10150 1000
-Wire Wire Line
-	10150 1000 10150 1050
+	10150 950  10150 1050
 Connection ~ 10150 1000
 Wire Wire Line
-	4250 1700 5800 1700
-Wire Wire Line
-	5800 1700 5850 1700
+	4250 1700 5850 1700
 $Comp
 L GND #PWR119
@@
 $EndComp
 Wire Wire Line
-	5800 850  5800 1200
-Wire Wire Line
-	5800 1200 5800 1700
+	5800 850  5800 1700
 Wire Wire Line
 	5800 1200 6100 1200
 Connection ~ 5800 1700
 Wire Wire Line
-	6450 1800 6650 1800
-Wire Wire Line
-	6650 1800 6750 1800
-Wire Wire Line
-	6650 850  6650 1200
-Wire Wire Line
-	6650 1200 6650 1800
+	6450 1800 6750 1800
+Wire Wire Line
+	6650 850  6650 1800
 Wire Wire Line
 	6650 1200 6400 1200
@@
 	5800 3500 5800 3550
 Wire Wire Line
-	4100 3300 5800 3300
-Wire Wire Line
-	5800 3300 5850 3300
+	4100 3300 5850 3300
 $Comp
 L R R62
@@
 	6100 2800 5800 2800
 Wire Wire Line
-	5800 2450 5800 2800
-Wire Wire Line
-	5800 2800 5800 3300
+	5800 2450 5800 3300
 Connection ~ 5800 3300
 Wire Wire Line
-	6450 3400 6650 3400
-Wire Wire Line
-	6650 3400 6750 3400
-Wire Wire Line
-	6650 2450 6650 2800
-Wire Wire Line
-	6650 2800 6650 3400
+	6450 3400 6750 3400
+Wire Wire Line
+	6650 2450 6650 3400
 Wire Wire Line
 	6650 2800 6400 2800
@@
 	5800 5100 5800 5150
 Wire Wire Line
-	4250 4900 5800 4900
-Wire Wire Line
-	5800 4900 5850 4900
+	4250 4900 5850 4900
 $Comp
 L R R63
@@
 	6100 4400 5800 4400
 Wire Wire Line
-	5800 4050 5800 4400
-Wire Wire Line
-	5800 4400 5800 4900
+	5800 4050 5800 4900
 Connection ~ 5800 4900
 Wire Wire Line
-	6450 5000 6650 5000
-Wire Wire Line
-	6650 5000 6750 5000
-Wire Wire Line
-	6650 4050 6650 4400
-Wire Wire Line
-	6650 4400 6650 5000
+	6450 5000 6750 5000
+Wire Wire Line
+	6650 4050 6650 5000
 Wire Wire Line
 	6650 4400 6400 4400
@@
 	5800 6700 5800 6750
 Wire Wire Line
-	4150 6500 5800 6500
-Wire Wire Line
-	5800 6500 5850 6500
+	4150 6500 5850 6500
 $Comp
 L R R64
@@
 	6100 6000 5800 6000
 Wire Wire Line
-	5800 5650 5800 6000
-Wire Wire Line
-	5800 6000 5800 6500
+	5800 5650 5800 6500
 Connection ~ 5800 6500
 Wire Wire Line
-	6450 6600 6650 6600
-Wire Wire Line
-	6650 6600 6750 6600
-Wire Wire Line
-	6650 5650 6650 6000
-Wire Wire Line
-	6650 6000 6650 6600
+	6450 6600 6750 6600
+Wire Wire Line
+	6650 5650 6650 6600
 Wire Wire Line
 	6650 6000 6400 6000
@@
 	4800 3500 5150 3500
 Wire Wire Line
-	5150 3500 5150 3600
-Wire Wire Line
-	5150 3600 5150 4000
+	5150 3500 5150 4000
 Wire Wire Line
 	5150 3600 5350 3600
 Wire Wire Line
-	5350 3550 5350 3600
-Wire Wire Line
-	5350 3600 5350 3650
+	5350 3550 5350 3650
 Connection ~ 5350 3600
 Wire Wire Line
@@
 $EndComp
 Wire Wire Line
-	2900 950  2900 1000
-Wire Wire Line
-	2900 1000 2900 1050
-Wire Wire Line
-	2900 1000 3200 1000
-Wire Wire Line
-	3200 1000 3350 1000
+	2900 950  2900 1050
+Wire Wire Line
+	2900 1000 3350 1000
 Wire Wire Line
 	3200 1000 3200 1050
 Connection ~ 2900 1000
 Wire Wire Line
-	2900 1350 2900 1400
-Wire Wire Line
-	2900 1400 2900 1450
+	2900 1350 2900 1450
 Wire Wire Line
 	2900 1400 3200 1400
@@
 $EndComp
 Wire Wire Line
-	7400 2250 7450 2250
-Wire Wire Line
-	7450 2250 7500 2250
+	7400 2250 7500 2250
 Wire Wire Line
 	7450 2250 7450 2300
 Connection ~ 7450 2250
 Wire Wire Line
-	7400 2050 7450 2050
-Wire Wire Line
-	7450 2050 7500 2050
+	7400 2050 7500 2050
 $Comp
 L +12VA #PWR141
@@
 $EndComp
 Wire Wire Line
-	10550 2300 10550 2350
-Wire Wire Line
-	10550 2350 10550 2400
+	10550 2300 10550 2400
 Wire Wire Line
 	10550 2350 10850 2350
@@
 Connection ~ 10550 2350
 Wire Wire Line
-	10150 2300 10150 2350
-Wire Wire Line
-	10150 2350 10150 2400
+	10150 2300 10150 2400
 Wire Wire Line
 	10150 2350 9850 2350
@@
 $EndComp
 Wire Wire Line
-	10550 2700 10550 2750
-Wire Wire Line
-	10550 2750 10550 2800
+	10550 2700 10550 2800
 Wire Wire Line
 	10550 2750 10850 2750
@@
 Connection ~ 10550 2750
 Wire Wire Line
-	10150 2700 10150 2750
-Wire Wire Line
-	10150 2750 10150 2800
+	10150 2700 10150 2800
 Wire Wire Line
 	10150 2750 9850 2750
@@
 $EndComp
 Wire Wire Line
-	7850 2450 7850 2600
-Wire Wire Line
-	7850 2600 7850 2700
+	7850 2450 7850 2700
 Wire Wire Line
 	7900 2600 7850 2600
 Connection ~ 7850 2600
 Wire Wire Line
-	7850 1600 7850 1700
-Wire Wire Line
-	7850 1700 7850 1850
+	7850 1600 7850 1850
 Wire Wire Line
 	7900 1700 7850 1700
@@
 	8550 1200 8550 2150
 Wire Wire Line
-	8350 2150 8550 2150
-Wire Wire Line
-	8550 2150 8750 2150
+	8350 2150 8750 2150
 Connection ~ 8550 2150
 $Comp
@@
 $EndComp
 Wire Wire Line
-	7400 5450 7450 5450
-Wire Wire Line
-	7450 5450 7500 5450
+	7400 5450 7500 5450
 Wire Wire Line
 	7450 5450 7450 5500
 Connection ~ 7450 5450
 Wire Wire Line
-	7400 5250 7450 5250
-Wire Wire Line
-	7450 5250 7500 5250
+	7400 5250 7500 5250
 $Comp
 L C C63
@@
 $EndComp
 Wire Wire Line
-	7850 5650 7850 5800
-Wire Wire Line
-	7850 5800 7850 5900
+	7850 5650 7850 5900
 Wire Wire Line
 	7900 5800 7850 5800
 Connection ~ 7850 5800
 Wire Wire Line
-	7850 4800 7850 4900
-Wire Wire Line
-	7850 4900 7850 5050
+	7850 4800 7850 5050
 Wire Wire Line
 	7900 4900 7850 4900
@@
 	8550 4400 8550 5350
 Wire Wire Line
-	8350 5350 8550 5350
-Wire Wire Line
-	8550 5350 8750 5350
+	8350 5350 8750 5350
 Connection ~ 8550 5350
 Wire Wire Line
@@
 $EndComp
 Wire Wire Line
-	2700 2300 2700 2350
-Wire Wire Line
-	2700 2350 2700 2400
+	2700 2300 2700 2400
 Wire Wire Line
 	2700 2350 3000 2350
@@
 Connection ~ 2700 2350
 Wire Wire Line
-	2700 1900 2700 1950
-Wire Wire Line
-	2700 1950 2700 2000
-Wire Wire Line
-	2700 1950 3000 1950
-Wire Wire Line
-	3000 1950 3150 1950
+	2700 1900 2700 2000
+Wire Wire Line
+	2700 1950 3150 1950
 Wire Wire Line
 	3000 1950 3000 2000
@@
 	1250 1950 950  1950
 Wire Wire Line
-	950  1900 950  1950
-Wire Wire Line
-	950  1950 950  2000
+	950  1900 950  2000
 Connection ~ 950  1950
 Wire Wire Line

Commit message: Cleaned up ERC
Connections:
- net labels added: +5VA, -5VA
- net labels removed: -5V0

Commit message: Populated BOM for DAC + amp
Parts:
- C46, C49, C50, C51, C60, C61, C62, C63, C66, C68: value 0.1u -> 0.1uF; footprint (none) -> Capacitors_SMD:C_0603; Manufacturer (none) -> Murata; Manufacturer Part Number (none) -> GRM188R61C104KA01
- C47, C48, C52, C64, C67, C69, C70: value 10u -> 10uF; footprint (none) -> Capacitors_ThroughHole:C_Radial_D5_L11_P2; Manufacturer (none) -> Panasonic; Manufacturer Part Number (none) -> P13478-ND
- C53, C54: value 47u -> 47uF; footprint (none) -> Capacitors_ThroughHole:C_Radial_D5_L11_P2; Manufacturer (none) -> Panasonic; Manufacturer Part Number (none) -> ECA-1EHG470
- C55: value CP -> 10uF; footprint (none) -> Capacitors_ThroughHole:C_Radial_D5_L11_P2; Manufacturer (none) -> Panasonic; Manufacturer Part Number (none) -> P13478-ND
- C56, C57, C58, C59: value 2.7n -> 2.7nF; footprint (none) -> Capacitors_SMD:C_0603; Manufacturer (none) -> Murata; Manufacturer Part Number (none) -> GRM1885C1H272JA01
- C65, C71: value 100u -> 100uF; footprint (none) -> Capacitors_ThroughHole:C_Radial_D8_L11.5_P3.5; Manufacturer (none) -> Panasonic; Manufacturer Part Number (none) -> ECA-1HM101
- R60: footprint (none) -> Resistors_SMD:R_0603; Manufacturer (none) -> Panasonic; Manufacturer Part Number (none) -> ERJ-3GEYJ103V
- R61, R62, R63, R64, R65, R66, R67, R68, R69, R70, R71, R72: footprint (none) -> Resistors_SMD:R_0603; Manufacturer (none) -> Panasonic; Manufacturer Part Number (none) -> ERJ-3EKF1001V
- R73, R74: footprint (none) -> Resistors_SMD:R_0603; Manufacturer (none) -> Panasonic; Manufacturer Part Number (none) -> ERJ-3EKF39R2V
- U10: footprint (none) -> Housings_SOIC:SOIC-14_3.9x8.7mm_Pitch1.27mm; Manufacturer (none) -> Texas Instruments; Manufacturer Part Number (none) -> OPA4134UA
- U11: footprint (none) -> Housings_SOIC:SOIC-20_7.5x12.8mm_Pitch1.27mm; Manufacturer (none) -> Texas Instruments; Manufacturer Part Number (none) -> TPA6120A2DWP
- U9: footprint (none) -> Housings_SSOP:SSOP-28_5.3x10.2mm_Pitch0.65mm; Manufacturer (none) -> Texas Instruments; Manufacturer Part Number (none) -> PCM1792ADB
- X2: footprint (none) -> headphones:Oscillator_SMD_2520_4Pads; Manufacturer (none) -> Microchip; Manufacturer Part Number (none) -> DSC1033DI2-012.2880
