File: pcb/ti_dac.sch (KiCad schematic (older format))
At the start: 45 parts, among them U10 OPA4134, U11 TPA6120A2, U9 PCM1792A, X2 12.288MHz

Commit message: Fixed placement of series termination resistors
I had the logical placement of the series termination resistors wrong
in the schematics (i.e. I had them placed at the source rather than
the load) so I moved all those around to the correct sheets.  I also
moved the ADC resistors in the layout, but haven't gotten to the DAC
ones yet.
Parts:
- added R58, R59, R82, R87, R88: 68, Resistors_SMD:R_0603, symbol R
Connections:
- wire segments 166 -> 171
Changed lines of the file:
@@
 Wire Wire Line
 	3250 1900 3250 2600
-Text HLabel 2300 3100 0    60   Input ~ 0
+Text HLabel 1700 3100 0    60   Input ~ 0
 DAC_LRCK
 Wire Wire Line
-	2300 3100 2600 3100
-Text HLabel 2300 3200 0    60   Input ~ 0
+	2150 3100 2600 3100
+Text HLabel 1700 3200 0    60   Input ~ 0
 DAC_BCK
-Text HLabel 2300 3300 0    60   Input ~ 0
+Text HLabel 1700 3300 0    60   Input ~ 0
 DAC_DATA
-Text HLabel 2300 3500 0    60   Input ~ 0
+Text HLabel 1700 3500 0    60   Input ~ 0
 DAC_RST
 Wire Wire Line
-	2300 3200 2600 3200
-Wire Wire Line
-	2300 3300 2600 3300
-Wire Wire Line
-	2300 3500 2600 3500
-Text HLabel 2300 3700 0    60   Output ~ 0
+	2150 3200 2600 3200
+Wire Wire Line
+	2150 3300 2600 3300
+Wire Wire Line
+	1700 3500 2600 3500
+Text HLabel 1700 3700 0    60   Output ~ 0
 DAC_MDO
-Text HLabel 2300 3800 0    60   Input ~ 0
+Text HLabel 1700 3800 0    60   Input ~ 0
 DAC_MDI
-Text HLabel 2300 3900 0    60   Input ~ 0
+Text HLabel 1700 3900 0    60   Input ~ 0
 DAC_MC
-Text HLabel 2300 4000 0    60   Input ~ 0
+Text HLabel 1700 4000 0    60   Input ~ 0
 DAC_MS
-Text HLabel 2300 4200 0    60   Input ~ 0
+Text HLabel 1700 4200 0    60   Input ~ 0
 DAC_MSEL
 Text HLabel 1250 2650 0    60   Input ~ 0
@@
 Connection ~ 950  1950
 Wire Wire Line
-	2300 3700 2600 3700
-Wire Wire Line
-	2300 3800 2600 3800
-Wire Wire Line
-	2300 3900 2600 3900
-Wire Wire Line
-	2300 4000 2600 4000
-Wire Wire Line
-	2300 4200 2600 4200
-Text HLabel 2300 4400 0    60   Output ~ 0
+	1700 3700 2600 3700
+Wire Wire Line
+	2150 3800 2600 3800
+Wire Wire Line
+	2150 3900 2600 3900
+Wire Wire Line
+	1700 4000 2600 4000
+Wire Wire Line
+	1700 4200 2600 4200
+Text HLabel 1700 4400 0    60   Output ~ 0
 DAC_ZEROL
-Text HLabel 2300 4500 0    60   Output ~ 0
+Text HLabel 1700 4500 0    60   Output ~ 0
 DAC_ZEROR
 Wire Wire Line
-	2300 4400 2600 4400
-Wire Wire Line
-	2300 4500 2600 4500
+	1700 4400 2600 4400
+Wire Wire Line
+	1700 4500 2600 4500
 Text Notes 9850 700  0    60   ~ 0
 OPA4134 DECOUPLING
@@
 	1    0    0    1
 $EndComp
+$Comp
+L R R58
+U 1 1 574D2C2C
+P 2000 3100
+F 0 "R58" V 1950 2900 50  0000 C CNN
+F 1 "68" V 2000 3100 50  0000 C CNN
+F 2 "Resistors_SMD:R_0603" V 1930 3100 50  0001 C CNN
+F 3 "" H 2000 3100 50  0000 C CNN
+F 4 "Panasonic" V 2000 3100 60  0001 C CNN "Manufacturer"
+F 5 "ERJ-3EKF68R0V" V 2000 3100 60  0001 C CNN "Manufacturer Part Number"
+	1    2000 3100
+	0    1    1    0
+$EndComp
+$Comp
+L R R59
+U 1 1 574D2C35
+P 2000 3200
+F 0 "R59" V 1950 3000 50  0000 C CNN
+F 1 "68" V 2000 3200 50  0000 C CNN
+F 2 "Resistors_SMD:R_0603" V 1930 3200 50  0001 C CNN
+F 3 "" H 2000 3200 50  0000 C CNN
+F 4 "Panasonic" V 2000 3200 60  0001 C CNN "Manufacturer"
+F 5 "ERJ-3EKF68R0V" V 2000 3200 60  0001 C CNN "Manufacturer Part Number"
+	1    2000 3200
+	0    1    1    0
+$EndComp
+$Comp
+L R R82
+U 1 1 574D2C3E
+P 2000 3300
+F 0 "R82" V 1950 3100 50  0000 C CNN
+F 1 "68" V 2000 3300 50  0000 C CNN
+F 2 "Resistors_SMD:R_0603" V 1930 3300 50  0001 C CNN
+F 3 "" H 2000 3300 50  0000 C CNN
+F 4 "Panasonic" V 2000 3300 60  0001 C CNN "Manufacturer"
+F 5 "ERJ-3EKF68R0V" V 2000 3300 60  0001 C CNN "Manufacturer Part Number"
+	1    2000 3300
+	0    1    1    0
+$EndComp
+$Comp
+L R R87
+U 1 1 574D34F2
+P 2000 3800
+F 0 "R87" V 1950 3600 50  0000 C CNN
+F 1 "68" V 2000 3800 50  0000 C CNN
+F 2 "Resistors_SMD:R_0603" V 1930 3800 50  0001 C CNN
+F 3 "" H 2000 3800 50  0000 C CNN
+F 4 "Panasonic" V 2000 3800 60  0001 C CNN "Manufacturer"
+F 5 "ERJ-3EKF68R0V" V 2000 3800 60  0001 C CNN "Manufacturer Part Number"
+	1    2000 3800
+	0    1    1    0
+$EndComp
+$Comp
+L R R88
+U 1 1 574D34FB
+P 2000 3900
+F 0 "R88" V 1950 3700 50  0000 C CNN
+F 1 "68" V 2000 3900 50  0000 C CNN
+F 2 "Resistors_SMD:R_0603" V 1930 3900 50  0001 C CNN
+F 3 "" H 2000 3900 50  0000 C CNN
+F 4 "Panasonic" V 2000 3900 60  0001 C CNN "Manufacturer"
+F 5 "ERJ-3EKF68R0V" V 2000 3900 60  0001 C CNN "Manufacturer Part Number"
+	1    2000 3900
+	0    1    1    0
+$EndComp
+Wire Wire Line
+	1700 3100 1850 3100
+Wire Wire Line
+	1700 3200 1850 3200
+Wire Wire Line
+	1700 3300 1850 3300
+Wire Wire Line
+	1700 3800 1850 3800
+Wire Wire Line
+	1700 3900 1850 3900
 $EndSCHEMATC

Commit message: Fixing up USB connector
- Had to go back through and re-annotate all the 0603 caps and
  resistors to the hand-solderding versions since those changes didn't
  make it back into the schematics the last time I tried.

- Added a new footprint for the USB connector to connect to all the
  shield pins.
Parts:
- C46, C49, C50, C51, C56, C57, C58, C59, C60, C61, C62, C63, C66, C68: footprint Capacitors_SMD:C_0603 -> Capacitors_SMD:C_0603_HandSoldering
- R58, R59, R60, R61, R62, R63, R64, R65, R66, R67, R68, R69, R70, R71, R72, R73, R74, R82, R87, R88: footprint Resistors_SMD:R_0603 -> Resistors_SMD:R_0603_HandSoldering

Commit message: Added sense resistors everywhere
Parts:
- added R112, R113, R114, R115, R116, R117, R118, R119, R120: 0.01, symbol R
Connections:
- wire segments 171 -> 188

Commit message: Still need to route all the new resistors
Parts:
- R112, R113, R114, R115, R116, R117, R118, R119, R120: footprint (none) -> Resistors_SMD:R_0603_HandSoldering
Changed lines of the file:
@@
 F 0 "R112" V 830 1950 50  0000 C CNN
 F 1 "0.01" V 750 1950 50  0000 C CNN
-F 2 "" V 680 1950 50  0000 C CNN
+F 2 "Resistors_SMD:R_0603_HandSoldering" V 680 1950 50  0001 C CNN
 F 3 "" H 750 1950 50  0000 C CNN
 	1    750  1950
@@
 F 0 "R113" V 2430 1950 50  0000 C CNN
 F 1 "0.01" V 2350 1950 50  0000 C CNN
-F 2 "" V 2280 1950 50  0000 C CNN
+F 2 "Resistors_SMD:R_0603_HandSoldering" V 2280 1950 50  0001 C CNN
 F 3 "" H 2350 1950 50  0000 C CNN
 	1    2350 1950
@@
 F 0 "R114" V 2580 1000 50  0000 C CNN
 F 1 "0.01" V 2500 1000 50  0000 C CNN
-F 2 "" V 2430 1000 50  0000 C CNN
+F 2 "Resistors_SMD:R_0603_HandSoldering" V 2430 1000 50  0001 C CNN
 F 3 "" H 2500 1000 50  0000 C CNN
 	1    2500 1000
@@
 F 0 "R116" V 4430 1000 50  0000 C CNN
 F 1 "0.01" V 4350 1000 50  0000 C CNN
-F 2 "" V 4280 1000 50  0000 C CNN
+F 2 "Resistors_SMD:R_0603_HandSoldering" V 4280 1000 50  0001 C CNN
 F 3 "" H 4350 1000 50  0000 C CNN
 	1    4350 1000
@@
 F 0 "R115" V 3130 1850 50  0000 C CNN
 F 1 "0.01" V 3050 1850 50  0000 C CNN
-F 2 "" V 2980 1850 50  0000 C CNN
+F 2 "Resistors_SMD:R_0603_HandSoldering" V 2980 1850 50  0001 C CNN
 F 3 "" H 3050 1850 50  0000 C CNN
 	1    3050 1850
@@
 F 0 "R117" V 9180 2900 50  0000 C CNN
 F 1 "0.01" V 9100 2900 50  0000 C CNN
-F 2 "" V 9030 2900 50  0000 C CNN
+F 2 "Resistors_SMD:R_0603_HandSoldering" V 9030 2900 50  0001 C CNN
 F 3 "" H 9100 2900 50  0000 C CNN
 	1    9100 2900
@@
 F 0 "R119" V 10780 2900 50  0000 C CNN
 F 1 "0.01" V 10700 2900 50  0000 C CNN
-F 2 "" V 10630 2900 50  0000 C CNN
+F 2 "Resistors_SMD:R_0603_HandSoldering" V 10630 2900 50  0001 C CNN
 F 3 "" H 10700 2900 50  0000 C CNN
 	1    10700 2900
@@
 F 0 "R118" V 9180 4050 50  0000 C CNN
 F 1 "0.01" V 9100 4050 50  0000 C CNN
-F 2 "" V 9030 4050 50  0000 C CNN
+F 2 "Resistors_SMD:R_0603_HandSoldering" V 9030 4050 50  0001 C CNN
 F 3 "" H 9100 4050 50  0000 C CNN
 	1    9100 4050
@@
 F 0 "R120" V 10780 4050 50  0000 C CNN
 F 1 "0.01" V 10700 4050 50  0000 C CNN
-F 2 "" V 10630 4050 50  0000 C CNN
+F 2 "Resistors_SMD:R_0603_HandSoldering" V 10630 4050 50  0001 C CNN
 F 3 "" H 10700 4050 50  0000 C CNN
 	1    10700 4050

Commit message: Placed and laid tracks for all sense resistors
Connections:
- net labels added: +12VL, +5VL, -12VL, -5VL
- wire segments 188 -> 204
Changed lines of the file:
@@
 	0    -1   -1   0
 $EndComp
-$Comp
-L +12VA #PWR0165
-U 1 1 57058BB3
-P 7850 2700
-F 0 "#PWR0165" H 7850 2550 50  0001 C CNN
-F 1 "+12VA" H 7850 2840 50  0000 C CNN
-F 2 "" H 7850 2700 50  0000 C CNN
-F 3 "" H 7850 2700 50  0000 C CNN
-	1    7850 2700
-	-1   0    0    1
-$EndComp
-$Comp
-L -12VA #PWR0166
-U 1 1 57058C2A
-P 7850 1600
-F 0 "#PWR0166" H 7850 1450 50  0001 C CNN
-F 1 "-12VA" H 7850 1740 50  0000 C CNN
-F 2 "" H 7850 1600 50  0000 C CNN
-F 3 "" H 7850 1600 50  0000 C CNN
-	1    7850 1600
-	1    0    0    -1
-$EndComp
-Wire Wire Line
-	7850 2450 7850 2700
-Wire Wire Line
-	7900 2600 7850 2600
-Connection ~ 7850 2600
-Wire Wire Line
-	7850 1600 7850 1850
+Wire Wire Line
+	7850 2450 7850 2600
+Wire Wire Line
+	7850 2600 7900 2600
+Wire Wire Line
+	7850 1700 7850 1850
 Wire Wire Line
 	7900 1700 7850 1700
-Connection ~ 7850 1700
 Wire Wire Line
 	7800 1200 7450 1200
@@
 	0    -1   -1   0
 $EndComp
-$Comp
-L +12VA #PWR0169
-U 1 1 5705A72F
-P 7850 5900
-F 0 "#PWR0169" H 7850 5750 50  0001 C CNN
-F 1 "+12VA" H 7850 6040 50  0000 C CNN
-F 2 "" H 7850 5900 50  0000 C CNN
-F 3 "" H 7850 5900 50  0000 C CNN
-	1    7850 5900
-	-1   0    0    1
-$EndComp
-$Comp
-L -12VA #PWR0170
-U 1 1 5705A735
-P 7850 4800
-F 0 "#PWR0170" H 7850 4650 50  0001 C CNN
-F 1 "-12VA" H 7850 4940 50  0000 C CNN
-F 2 "" H 7850 4800 50  0000 C CNN
-F 3 "" H 7850 4800 50  0000 C CNN
-	1    7850 4800
-	1    0    0    -1
-$EndComp
-Wire Wire Line
-	7850 5650 7850 5900
-Wire Wire Line
-	7900 5800 7850 5800
-Connection ~ 7850 5800
-Wire Wire Line
-	7850 4800 7850 5050
+Wire Wire Line
+	7850 5650 7850 5800
+Wire Wire Line
+	7850 5800 7900 5800
+Wire Wire Line
+	7850 4900 7850 5050
 Wire Wire Line
 	7900 4900 7850 4900
-Connection ~ 7850 4900
 Wire Wire Line
 	7800 4400 7450 4400
@@
 Text Notes 9400 2600 0    60   ~ 0
 OPA4134 DECOUPLING
-Text Notes 9400 3850 0    60   ~ 0
+Text Notes 9400 3750 0    60   ~ 0
 TPA6120A2 DECOUPLING
 $Comp
@@
 $EndComp
 $Comp
-L -5VA #PWR149
-U 1 1 5715857E
-P 6050 1500
-F 0 "#PWR149" H 6050 1600 50  0001 C CNN
-F 1 "-5VA" H 6050 1650 50  0000 C CNN
-F 2 "" H 6050 1500 50  0000 C CNN
-F 3 "" H 6050 1500 50  0000 C CNN
-	1    6050 1500
-	1    0    0    -1
-$EndComp
-$Comp
-L -5VA #PWR151
-U 1 1 5715861C
-P 6050 3100
-F 0 "#PWR151" H 6050 3200 50  0001 C CNN
-F 1 "-5VA" H 6050 3250 50  0000 C CNN
-F 2 "" H 6050 3100 50  0000 C CNN
-F 3 "" H 6050 3100 50  0000 C CNN
-	1    6050 3100
-	1    0    0    -1
-$EndComp
-$Comp
-L -5VA #PWR155
-U 1 1 57158947
-P 6050 6300
-F 0 "#PWR155" H 6050 6400 50  0001 C CNN
-F 1 "-5VA" H 6050 6450 50  0000 C CNN
-F 2 "" H 6050 6300 50  0000 C CNN
-F 3 "" H 6050 6300 50  0000 C CNN
-	1    6050 6300
-	1    0    0    -1
-$EndComp
-$Comp
-L -5VA #PWR153
-U 1 1 571589E5
-P 6050 4700
-F 0 "#PWR153" H 6050 4800 50  0001 C CNN
-F 1 "-5VA" H 6050 4850 50  0000 C CNN
-F 2 "" H 6050 4700 50  0000 C CNN
-F 3 "" H 6050 4700 50  0000 C CNN
-	1    6050 4700
-	1    0    0    -1
-$EndComp
-$Comp
 L -5VA #PWR173
 U 1 1 57159F78
@@
 	1    8850 2850
 	1    0    0    -1
-$EndComp
-$Comp
-L +5VA #PWR0180
-U 1 1 57163679
-P 6050 2100
-F 0 "#PWR0180" H 6050 1950 50  0001 C CNN
-F 1 "+5VA" H 6050 2240 50  0000 C CNN
-F 2 "" H 6050 2100 50  0000 C CNN
-F 3 "" H 6050 2100 50  0000 C CNN
-	1    6050 2100
-	-1   0    0    1
-$EndComp
-$Comp
-L +5VA #PWR0181
-U 1 1 57163F8C
-P 6050 3700
-F 0 "#PWR0181" H 6050 3550 50  0001 C CNN
-F 1 "+5VA" H 6050 3840 50  0000 C CNN
-F 2 "" H 6050 3700 50  0000 C CNN
-F 3 "" H 6050 3700 50  0000 C CNN
-	1    6050 3700
-	-1   0    0    1
-$EndComp
-$Comp
-L +5VA #PWR0182
-U 1 1 571652F5
-P 6050 5300
-F 0 "#PWR0182" H 6050 5150 50  0001 C CNN
-F 1 "+5VA" H 6050 5440 50  0000 C CNN
-F 2 "" H 6050 5300 50  0000 C CNN
-F 3 "" H 6050 5300 50  0000 C CNN
-	1    6050 5300
-	-1   0    0    1
-$EndComp
-$Comp
-L +5VA #PWR0183
-U 1 1 5716536B
-P 6050 6900
-F 0 "#PWR0183" H 6050 6750 50  0001 C CNN
-F 1 "+5VA" H 6050 7040 50  0000 C CNN
-F 2 "" H 6050 6900 50  0000 C CNN
-F 3 "" H 6050 6900 50  0000 C CNN
-	1    6050 6900
-	-1   0    0    1
 $EndComp
 $Comp
@@
 	1    0    0    -1
 $EndComp
+$Comp
+L PWR_FLAG #FLG?
+U 1 1 5801AB81
+P 9300 2900
+F 0 "#FLG?" H 9300 2995 50  0001 C CNN
+F 1 "PWR_FLAG" H 9300 3080 50  0000 C CNN
+F 2 "" H 9300 2900 50  0000 C CNN
+F 3 "" H 9300 2900 50  0000 C CNN
+	1    9300 2900
+	1    0    0    -1
+$EndComp
+$Comp
+L PWR_FLAG #FLG?
+U 1 1 5801B07F
+P 10500 2900
+F 0 "#FLG?" H 10500 2995 50  0001 C CNN
+F 1 "PWR_FLAG" H 10500 3080 50  0000 C CNN
+F 2 "" H 10500 2900 50  0000 C CNN
+F 3 "" H 10500 2900 50  0000 C CNN
+	1    10500 2900
+	1    0    0    -1
+$EndComp
+$Comp
+L PWR_FLAG #FLG?
+U 1 1 5801B76E
+P 9300 4050
+F 0 "#FLG?" H 9300 4145 50  0001 C CNN
+F 1 "PWR_FLAG" H 9300 4230 50  0000 C CNN
+F 2 "" H 9300 4050 50  0000 C CNN
+F 3 "" H 9300 4050 50  0000 C CNN
+	1    9300 4050
+	1    0    0    -1
+$EndComp
+$Comp
+L PWR_FLAG #FLG?
+U 1 1 5801B836
+P 10500 4050
+F 0 "#FLG?" H 10500 4145 50  0001 C CNN
+F 1 "PWR_FLAG" H 10500 4230 50  0000 C CNN
+F 2 "" H 10500 4050 50  0000 C CNN
+F 3 "" H 10500 4050 50  0000 C CNN
+	1    10500 4050
+	1    0    0    -1
+$EndComp
+Text Label 9500 2900 0    60   ~ 0
++5VL
+Text Label 10100 2900 0    60   ~ 0
+-5VL
+Text Label 9450 4050 0    60   ~ 0
++12VL
+Text Label 10100 4050 0    60   ~ 0
+-12VL
+Text Label 7850 1700 1    60   ~ 0
+-12VL
+Text Label 7850 2600 3    60   ~ 0
++12VL
+Text Label 7850 5800 3    60   ~ 0
++12VL
+Text Label 7850 4900 1    60   ~ 0
+-12VL
+Text Label 6050 7000 0    60   ~ 0
++5VL
+Text Label 6050 6250 0    60   ~ 0
+-5VL
+Wire Wire Line
+	6050 6900 6050 7000
+Wire Wire Line
+	6050 7000 6300 7000
+Wire Wire Line
+	6050 6300 6050 6250
+Wire Wire Line
+	6050 6250 6300 6250
+Wire Wire Line
+	6050 4700 6050 4650
+Wire Wire Line
+	6050 4650 6300 4650
+Wire Wire Line
+	6050 5300 6050 5400
+Wire Wire Line
+	6050 5400 6300 5400
+Wire Wire Line
+	6050 3100 6050 3050
+Wire Wire Line
+	6050 3050 6300 3050
+Wire Wire Line
+	6050 3700 6050 3750
+Wire Wire Line
+	6050 3750 6300 3750
+Wire Wire Line
+	6050 2100 6050 2200
+Wire Wire Line
+	6050 2200 6300 2200
+Wire Wire Line
+	6050 1500 6050 1450
+Wire Wire Line
+	6050 1450 6300 1450
+Text Label 6050 4650 0    60   ~ 0
+-5VL
+Text Label 6050 5400 0    60   ~ 0
++5VL
+Text Label 6050 3750 0    60   ~ 0
++5VL
+Text Label 6050 3050 0    60   ~ 0
+-5VL
+Text Label 6050 1450 0    60   ~ 0
+-5VL
+Text Label 6050 2200 0    60   ~ 0
++5VL
 $EndSCHEMATC

Commit message: Added two more sense resistors
Parts:
- added R130: 0.01, Resistors_SMD:R_0603_HandSoldering, symbol R
