File: pcb/ti_dac.sch (KiCad schematic (older format))
At the start: 60 parts, among them U10 OPA4134, U11 TPA6120A2, U9 PCM1792A, X2 12.288MHz

Commit message: Cleanup and added testpoints
Cleaned up some of the schematic layout without changing any nets.  Also
added testpoints to all the power rails for easy debug.
Connections:
- wire segments 204 -> 255

Commit message: More cleanup and switched sense resistors
Increased the resistance of the current sense resistors up to 0.1 ohm.
Parts:
- R112, R113, R114, R115, R116, R117, R118, R119, R120, R130: value 0.01 -> 0.1
Changed lines of the file:
@@
 P 2400 3900
 F 0 "R112" V 2480 3900 50  0000 C CNN
-F 1 "0.01" V 2400 3900 50  0000 C CNN
+F 1 "0.1" V 2400 3900 50  0000 C CNN
 F 2 "Resistors_SMD:R_0603_HandSoldering" V 2330 3900 50  0001 C CNN
 F 3 "" H 2400 3900 50  0000 C CNN
@@
 P 4700 3300
 F 0 "R113" V 4780 3300 50  0000 C CNN
-F 1 "0.01" V 4700 3300 50  0000 C CNN
+F 1 "0.1" V 4700 3300 50  0000 C CNN
 F 2 "Resistors_SMD:R_0603_HandSoldering" V 4630 3300 50  0001 C CNN
 F 3 "" H 4700 3300 50  0000 C CNN
@@
 P 4850 2000
 F 0 "R114" V 4930 2000 50  0000 C CNN
-F 1 "0.01" V 4850 2000 50  0000 C CNN
+F 1 "0.1" V 4850 2000 50  0000 C CNN
 F 2 "Resistors_SMD:R_0603_HandSoldering" V 4780 2000 50  0001 C CNN
 F 3 "" H 4850 2000 50  0000 C CNN
@@
 P 6700 2000
 F 0 "R116" V 6780 2000 50  0000 C CNN
-F 1 "0.01" V 6700 2000 50  0000 C CNN
+F 1 "0.1" V 6700 2000 50  0000 C CNN
 F 2 "Resistors_SMD:R_0603_HandSoldering" V 6630 2000 50  0001 C CNN
 F 3 "" H 6700 2000 50  0000 C CNN
@@
 P 5250 2950
 F 0 "R115" V 5330 2950 50  0000 C CNN
-F 1 "0.01" V 5250 2950 50  0000 C CNN
+F 1 "0.1" V 5250 2950 50  0000 C CNN
 F 2 "Resistors_SMD:R_0603_HandSoldering" V 5180 2950 50  0001 C CNN
 F 3 "" H 5250 2950 50  0000 C CNN
@@
 P 12400 4300
 F 0 "R117" V 12480 4300 50  0000 C CNN
-F 1 "0.01" V 12400 4300 50  0000 C CNN
+F 1 "0.1" V 12400 4300 50  0000 C CNN
 F 2 "Resistors_SMD:R_0603_HandSoldering" V 12330 4300 50  0001 C CNN
 F 3 "" H 12400 4300 50  0000 C CNN
@@
 P 14000 4300
 F 0 "R119" V 14080 4300 50  0000 C CNN
-F 1 "0.01" V 14000 4300 50  0000 C CNN
+F 1 "0.1" V 14000 4300 50  0000 C CNN
 F 2 "Resistors_SMD:R_0603_HandSoldering" V 13930 4300 50  0001 C CNN
 F 3 "" H 14000 4300 50  0000 C CNN
@@
 P 12400 5450
 F 0 "R118" V 12480 5450 50  0000 C CNN
-F 1 "0.01" V 12400 5450 50  0000 C CNN
+F 1 "0.1" V 12400 5450 50  0000 C CNN
 F 2 "Resistors_SMD:R_0603_HandSoldering" V 12330 5450 50  0001 C CNN
 F 3 "" H 12400 5450 50  0000 C CNN
@@
 P 14000 5450
 F 0 "R120" V 14080 5450 50  0000 C CNN
-F 1 "0.01" V 14000 5450 50  0000 C CNN
+F 1 "0.1" V 14000 5450 50  0000 C CNN
 F 2 "Resistors_SMD:R_0603_HandSoldering" V 13930 5450 50  0001 C CNN
 F 3 "" H 14000 5450 50  0000 C CNN
@@
 P 7700 5050
 F 0 "R130" V 7780 5050 50  0000 C CNN
-F 1 "0.01" V 7700 5050 50  0000 C CNN
+F 1 "0.1" V 7700 5050 50  0000 C CNN
 F 2 "Resistors_SMD:R_0603_HandSoldering" V 7630 5050 50  0001 C CNN
 F 3 "" H 7700 5050 50  0000 C CNN

Commit message: Ran DRC and added some more notes
Connections:
- wire segments 255 -> 203
