File: pcb/analog_input_buffer.sch (KiCad schematic (older format))
At the start: 18 parts, among them U2 OP1642

Commit message: Began cleaning up ERC errors
Connections:
- wire segments 37 -> 41

Commit message: Cleaned up ERC
Connections:
- net labels added: GND
- net labels removed: GNDA
Changed lines of the file:
@@
 $EndComp
 $Comp
-L +12VA #PWR21
+L +12VA #PWR017
 U 1 1 56A21F3D
 P 5350 4000
-AR Path="/56888583/56A2193A/56A21F3D" Ref="#PWR21"  Part="1"
-AR Path="/56888583/56A25341/56A21F3D" Ref="#PWR28"  Part="1"
-F 0 "#PWR28" H 5350 3850 50  0001 C CNN
+AR Path="/56888583/56A2193A/56A21F3D" Ref="#PWR017"  Part="1"
+AR Path="/56888583/56A25341/56A21F3D" Ref="#PWR024"  Part="1"
+F 0 "#PWR024" H 5350 3850 50  0001 C CNN
 F 1 "+12VA" H 5350 4140 50  0000 C CNN
 F 2 "" H 5350 4000 50  0000 C CNN
@@
 $EndComp
 $Comp
-L -12VA #PWR22
+L -12VA #PWR018
 U 1 1 56A21F49
 P 5350 4800
-AR Path="/56888583/56A2193A/56A21F49" Ref="#PWR22"  Part="1"
-AR Path="/56888583/56A25341/56A21F49" Ref="#PWR29"  Part="1"
-F 0 "#PWR29" H 5350 4650 50  0001 C CNN
+AR Path="/56888583/56A2193A/56A21F49" Ref="#PWR018"  Part="1"
+AR Path="/56888583/56A25341/56A21F49" Ref="#PWR025"  Part="1"
+F 0 "#PWR025" H 5350 4650 50  0001 C CNN
 F 1 "-12VA" H 5350 4940 50  0000 C CNN
 F 2 "" H 5350 4800 50  0000 C CNN
@@
 F 3 "" H 4500 3550 50  0000 C CNN
 	1    4500 3550
-	1    0    0    -1
-$EndComp
-$Comp
-L GNDA #PWR17
-U 1 1 56A2330E
-P 4500 3700
-AR Path="/56888583/56A2193A/56A2330E" Ref="#PWR17"  Part="1"
-AR Path="/56888583/56A25341/56A2330E" Ref="#PWR24"  Part="1"
-F 0 "#PWR24" H 4500 3450 50  0001 C CNN
-F 1 "GNDA" H 4500 3550 50  0000 C CNN
-F 2 "" H 4500 3700 50  0000 C CNN
-F 3 "" H 4500 3700 50  0000 C CNN
-	1    4500 3700
-	1    0    0    -1
-$EndComp
-$Comp
-L GNDA #PWR18
-U 1 1 56A23340
-P 4500 4700
-AR Path="/56888583/56A2193A/56A23340" Ref="#PWR18"  Part="1"
-AR Path="/56888583/56A25341/56A23340" Ref="#PWR25"  Part="1"
-F 0 "#PWR25" H 4500 4450 50  0001 C CNN
-F 1 "GNDA" H 4500 4550 50  0000 C CNN
-F 2 "" H 4500 4700 50  0000 C CNN
-F 3 "" H 4500 4700 50  0000 C CNN
-	1    4500 4700
 	1    0    0    -1
 $EndComp
@@
 Connection ~ 7050 4400
 $Comp
-L +12VA #PWR20
+L +12VA #PWR019
 U 1 1 56A62B13
 P 5350 3500
-AR Path="/56888583/56A2193A/56A62B13" Ref="#PWR20"  Part="1"
-AR Path="/56888583/56A25341/56A62B13" Ref="#PWR27"  Part="1"
-F 0 "#PWR27" H 5350 3350 50  0001 C CNN
+AR Path="/56888583/56A2193A/56A62B13" Ref="#PWR019"  Part="1"
+AR Path="/56888583/56A25341/56A62B13" Ref="#PWR026"  Part="1"
+F 0 "#PWR026" H 5350 3350 50  0001 C CNN
 F 1 "+12VA" H 5350 3640 50  0000 C CNN
 F 2 "" H 5350 3500 50  0000 C CNN
@@
 $EndComp
 $Comp
-L -12VA #PWR19
+L -12VA #PWR020
 U 1 1 56A62B54
 P 5350 2700
-AR Path="/56888583/56A2193A/56A62B54" Ref="#PWR19"  Part="1"
-AR Path="/56888583/56A25341/56A62B54" Ref="#PWR26"  Part="1"
-F 0 "#PWR26" H 5350 2550 50  0001 C CNN
+AR Path="/56888583/56A2193A/56A62B54" Ref="#PWR020"  Part="1"
+AR Path="/56888583/56A25341/56A62B54" Ref="#PWR027"  Part="1"
+F 0 "#PWR027" H 5350 2550 50  0001 C CNN
 F 1 "-12VA" H 5350 2840 50  0000 C CNN
 F 2 "" H 5350 2700 50  0000 C CNN
@@
 	0    1    1    0
 $EndComp
-$Comp
-L GNDA #PWR23
-U 1 1 56A63494
+Wire Wire Line
+	5850 3750 6000 3750
+Wire Wire Line
+	5350 2700 5350 2800
+Wire Wire Line
+	5350 3400 5350 3500
+Wire Wire Line
+	5350 4000 5350 4100
+Wire Wire Line
+	5350 4700 5350 4800
+$Comp
+L GND #PWR021
+U 1 1 57170EC5
 P 6000 3750
-AR Path="/56888583/56A2193A/56A63494" Ref="#PWR23"  Part="1"
-AR Path="/56888583/56A25341/56A63494" Ref="#PWR30"  Part="1"
-F 0 "#PWR30" H 6000 3500 50  0001 C CNN
-F 1 "GNDA" H 6000 3600 50  0000 C CNN
+AR Path="/56888583/56A2193A/57170EC5" Ref="#PWR021"  Part="1"
+AR Path="/56888583/56A25341/57170EC5" Ref="#PWR028"  Part="1"
+F 0 "#PWR028" H 6000 3500 50  0001 C CNN
+F 1 "GND" H 6000 3600 50  0000 C CNN
 F 2 "" H 6000 3750 50  0000 C CNN
 F 3 "" H 6000 3750 50  0000 C CNN
@@
 	1    0    0    -1
 $EndComp
-Wire Wire Line
-	5850 3750 6000 3750
-Wire Wire Line
-	5350 2700 5350 2800
-Wire Wire Line
-	5350 3400 5350 3500
-Wire Wire Line
-	5350 4000 5350 4100
-Wire Wire Line
-	5350 4700 5350 4800
+$Comp
+L GND #PWR022
+U 1 1 57170EFF
+P 4500 3700
+AR Path="/56888583/56A2193A/57170EFF" Ref="#PWR022"  Part="1"
+AR Path="/56888583/56A25341/57170EFF" Ref="#PWR029"  Part="1"
+F 0 "#PWR029" H 4500 3450 50  0001 C CNN
+F 1 "GND" H 4500 3550 50  0000 C CNN
+F 2 "" H 4500 3700 50  0000 C CNN
+F 3 "" H 4500 3700 50  0000 C CNN
+	1    4500 3700
+	1    0    0    -1
+$EndComp
+$Comp
+L GND #PWR023
+U 1 1 57170F39
+P 4500 4700
+AR Path="/56888583/56A2193A/57170F39" Ref="#PWR023"  Part="1"
+AR Path="/56888583/56A25341/57170F39" Ref="#PWR030"  Part="1"
+F 0 "#PWR030" H 4500 4450 50  0001 C CNN
+F 1 "GND" H 4500 4550 50  0000 C CNN
+F 2 "" H 4500 4700 50  0000 C CNN
+F 3 "" H 4500 4700 50  0000 C CNN
+	1    4500 4700
+	1    0    0    -1
+$EndComp
 $EndSCHEMATC

Commit message: Latest work on footprints and BOM
Parts:
- C11, C12: footprint (none) -> Capacitors_ThroughHole:C_Radial_D5_L11_P2; Manufacturer (none) -> Panasonic; Manufacturer Part Number (none) -> P13478-ND
- C13, C14: footprint (none) -> Capacitors_SMD:C_0603; Manufacturer (none) -> Murata; Manufacturer Part Number (none) -> GRM1885C1H471JA01
- C15: footprint (none) -> Capacitors_SMD:C_0603; Manufacturer (none) -> Murata; Manufacturer Part Number (none) -> GRM188R61C104KA01
- C16: footprint (none) -> Capacitors_SMD:C_0603; Manufacturer (none) -> Murata; Manufacturer Part Number (none) -> GRM1885C1H272JA01
- R10, R9: footprint (none) -> Resistors_SMD:R_0603; Manufacturer (none) -> Panasonic; Manufacturer Part Number (none) -> ERJ-3EKF6340V
- R11, R12: footprint (none) -> Resistors_SMD:R_0603; Manufacturer (none) -> Panasonic; Manufacturer Part Number (none) -> ERJ-3EKF91R0V
- R13, R14, R15: footprint (none) -> Resistors_SMD:R_0603; Manufacturer (none) -> Panasonic; Manufacturer Part Number (none) -> ERJ-3EKF2000V
- R5, R6: footprint (none) -> Resistors_SMD:R_0603; Manufacturer (none) -> Panasonic; Manufacturer Part Number (none) -> ERJ-3GEYJ104V
- R7, R8: footprint (none) -> Resistors_SMD:R_0603; Manufacturer (none) -> Panasonic; Manufacturer Part Number (none) -> ERJ-3GEYJ103V
- U2: footprint (none) -> Housings_SOIC:SOIC-8_3.9x4.9mm_Pitch1.27mm; Manufacturer (none) -> Texas Instruments; Manufacturer Part Number (none) -> OPA1642
