File: pcb/analog_input_buffer.sch (KiCad schematic (older format))
At the start: 18 parts, among them U2 OP1642

Commit message: Fixing up USB connector
- Had to go back through and re-annotate all the 0603 caps and
  resistors to the hand-solderding versions since those changes didn't
  make it back into the schematics the last time I tried.

- Added a new footprint for the USB connector to connect to all the
  shield pins.
Parts:
- C13, C14, C15, C16: footprint Capacitors_SMD:C_0603 -> Capacitors_SMD:C_0603_HandSoldering
- R10, R11, R12, R13, R14, R15, R5, R6, R7, R8, R9: footprint Resistors_SMD:R_0603 -> Resistors_SMD:R_0603_HandSoldering
Changed lines of the file:
@@
 F 0 "R20" V 5480 1950 50  0000 C CNN
 F 1 "634" V 5400 1950 50  0000 C CNN
-F 2 "Resistors_SMD:R_0603" V 5330 1950 50  0001 C CNN
+F 2 "Resistors_SMD:R_0603_HandSoldering" V 5330 1950 50  0001 C CNN
 F 3 "" H 5400 1950 50  0000 C CNN
 F 4 "Panasonic" V 5400 1950 60  0001 C CNN "Manufacturer"
@@
 F 0 "R22" V 6130 3100 50  0000 C CNN
 F 1 "91" V 6050 3100 50  0000 C CNN
-F 2 "Resistors_SMD:R_0603" V 5980 3100 50  0001 C CNN
+F 2 "Resistors_SMD:R_0603_HandSoldering" V 5980 3100 50  0001 C CNN
 F 3 "" H 6050 3100 50  0000 C CNN
 F 4 "Panasonic" V 6050 3100 60  0001 C CNN "Manufacturer"
@@
 F 0 "C22" H 7075 3850 50  0000 L CNN
 F 1 "2700pF C0G" H 7075 3650 50  0000 L CNN
-F 2 "Capacitors_SMD:C_0603" H 7088 3600 50  0001 C CNN
+F 2 "Capacitors_SMD:C_0603_HandSoldering" H 7088 3600 50  0001 C CNN
 F 3 "" H 7050 3750 50  0000 C CNN
 F 4 "Murata" H 7050 3750 60  0001 C CNN "Manufacturer"
@@
 F 0 "R18" V 5130 3550 50  0000 C CNN
 F 1 "10K" V 5050 3550 50  0000 C CNN
-F 2 "Resistors_SMD:R_0603" V 4980 3550 50  0001 C CNN
+F 2 "Resistors_SMD:R_0603_HandSoldering" V 4980 3550 50  0001 C CNN
 F 3 "" H 5050 3550 50  0000 C CNN
 F 4 "Panasonic" V 5050 3550 60  0001 C CNN "Manufacturer"
@@
 F 0 "C19" H 5425 2300 50  0000 L CNN
 F 1 "470pF C0G" V 5600 2000 50  0000 L CNN
-F 2 "Capacitors_SMD:C_0603" H 5438 2050 50  0001 C CNN
+F 2 "Capacitors_SMD:C_0603_HandSoldering" H 5438 2050 50  0001 C CNN
 F 3 "" H 5400 2200 50  0000 C CNN
 F 4 "Murata" H 5400 2200 60  0001 C CNN "Manufacturer"
@@
 F 0 "R16" V 4580 3550 50  0000 C CNN
 F 1 "100K" V 4500 3550 50  0000 C CNN
-F 2 "Resistors_SMD:R_0603" V 4430 3550 50  0001 C CNN
+F 2 "Resistors_SMD:R_0603_HandSoldering" V 4430 3550 50  0001 C CNN
 F 3 "" H 4500 3550 50  0000 C CNN
 F 4 "Panasonic" V 4500 3550 60  0001 C CNN "Manufacturer"
@@
 F 0 "R24" V 6630 3100 50  0000 C CNN
 F 1 "200" V 6550 3100 50  0000 C CNN
-F 2 "Resistors_SMD:R_0603" V 6480 3100 50  0001 C CNN
+F 2 "Resistors_SMD:R_0603_HandSoldering" V 6480 3100 50  0001 C CNN
 F 3 "" H 6550 3100 50  0000 C CNN
 F 4 "Panasonic" V 6550 3100 60  0001 C CNN "Manufacturer"
@@
 F 0 "C21" H 5725 3850 50  0000 L CNN
 F 1 "0.1uF" H 5725 3650 50  0000 L CNN
-F 2 "Capacitors_SMD:C_0603" H 5738 3600 50  0001 C CNN
+F 2 "Capacitors_SMD:C_0603_HandSoldering" H 5738 3600 50  0001 C CNN
 F 3 "" H 5700 3750 50  0000 C CNN
 F 4 "Murata" H 5700 3750 60  0001 C CNN "Manufacturer"
@@
 F 0 "R17" V 4580 4550 50  0000 C CNN
 F 1 "100K" V 4500 4550 50  0000 C CNN
-F 2 "Resistors_SMD:R_0603" V 4430 4550 50  0001 C CNN
+F 2 "Resistors_SMD:R_0603_HandSoldering" V 4430 4550 50  0001 C CNN
 F 3 "" H 4500 4550 50  0000 C CNN
 F 4 "Panasonic" V 4500 4550 60  0001 C CNN "Manufacturer"
@@
 F 0 "R19" V 5130 3950 50  0000 C CNN
 F 1 "10K" V 5050 3950 50  0000 C CNN
-F 2 "Resistors_SMD:R_0603" V 4980 3950 50  0001 C CNN
+F 2 "Resistors_SMD:R_0603_HandSoldering" V 4980 3950 50  0001 C CNN
 F 3 "" H 5050 3950 50  0000 C CNN
 F 4 "Panasonic" V 5050 3950 60  0001 C CNN "Manufacturer"
@@
 F 0 "R21" V 5480 5650 50  0000 C CNN
 F 1 "634" V 5400 5650 50  0000 C CNN
-F 2 "Resistors_SMD:R_0603" V 5330 5650 50  0001 C CNN
+F 2 "Resistors_SMD:R_0603_HandSoldering" V 5330 5650 50  0001 C CNN
 F 3 "" H 5400 5650 50  0000 C CNN
 F 4 "Panasonic" V 5400 5650 60  0001 C CNN "Manufacturer"
@@
 F 0 "R23" V 6130 4400 50  0000 C CNN
 F 1 "91" V 6050 4400 50  0000 C CNN
-F 2 "Resistors_SMD:R_0603" V 5980 4400 50  0001 C CNN
+F 2 "Resistors_SMD:R_0603_HandSoldering" V 5980 4400 50  0001 C CNN
 F 3 "" H 6050 4400 50  0000 C CNN
 F 4 "Panasonic" V 6050 4400 60  0001 C CNN "Manufacturer"
@@
 F 0 "R25" V 6630 4400 50  0000 C CNN
 F 1 "200" V 6550 4400 50  0000 C CNN
-F 2 "Resistors_SMD:R_0603" V 6480 4400 50  0001 C CNN
+F 2 "Resistors_SMD:R_0603_HandSoldering" V 6480 4400 50  0001 C CNN
 F 3 "" H 6550 4400 50  0000 C CNN
 F 4 "Panasonic" V 6550 4400 60  0001 C CNN "Manufacturer"
@@
 F 0 "R26" V 6880 3750 50  0000 C CNN
 F 1 "200" V 6800 3750 50  0000 C CNN
-F 2 "Resistors_SMD:R_0603" V 6730 3750 50  0001 C CNN
+F 2 "Resistors_SMD:R_0603_HandSoldering" V 6730 3750 50  0001 C CNN
 F 3 "" H 6800 3750 50  0000 C CNN
 F 4 "Panasonic" V 6800 3750 60  0001 C CNN "Manufacturer"
@@
 F 0 "C20" H 5425 5350 50  0000 L CNN
 F 1 "470pF C0G" V 5600 5050 50  0000 L CNN
-F 2 "Capacitors_SMD:C_0603" H 5438 5100 50  0001 C CNN
+F 2 "Capacitors_SMD:C_0603_HandSoldering" H 5438 5100 50  0001 C CNN
 F 3 "" H 5400 5250 50  0000 C CNN
 F 4 "Murata" H 5400 5250 60  0001 C CNN "Manufacturer"

Commit message: Added sense resistors everywhere
Parts:
- added C111, C114: 10uF, Capacitors_ThroughHole:C_Radial_D5_L11_P2, symbol CP
- added C112, C113: 0.1uF, Capacitors_SMD:C_0603_HandSoldering, symbol C
- added R106, R107: 0.01, symbol R
Connections:
- wire segments 41 -> 57

Commit message: Still need to route all the new resistors
Parts:
- R106, R107: footprint (none) -> Resistors_SMD:R_0603_HandSoldering
Changed lines of the file:
@@
 AR Path="/56888583/56A2193A/56A21F1B" Ref="C11"  Part="1"
 AR Path="/56888583/56A25341/56A21F1B" Ref="C17"  Part="1"
-F 0 "C11" H 4825 3300 50  0000 L CNN
+F 0 "C17" H 4825 3300 50  0000 L CNN
 F 1 "10uF" H 4825 3100 50  0000 L CNN
 F 2 "Capacitors_ThroughHole:C_Radial_D5_L11_P2" H 4838 3050 50  0001 C CNN
@@
 AR Path="/56888583/56A2193A/56A21F4F" Ref="R9"  Part="1"
 AR Path="/56888583/56A25341/56A21F4F" Ref="R20"  Part="1"
-F 0 "R9" V 5480 1950 50  0000 C CNN
+F 0 "R20" V 5480 1950 50  0000 C CNN
 F 1 "634" V 5400 1950 50  0000 C CNN
 F 2 "Resistors_SMD:R_0603_HandSoldering" V 5330 1950 50  0001 C CNN
@@
 AR Path="/56888583/56A2193A/56A21F56" Ref="R11"  Part="1"
 AR Path="/56888583/56A25341/56A21F56" Ref="R22"  Part="1"
-F 0 "R11" V 6130 3100 50  0000 C CNN
+F 0 "R22" V 6130 3100 50  0000 C CNN
 F 1 "91" V 6050 3100 50  0000 C CNN
 F 2 "Resistors_SMD:R_0603_HandSoldering" V 5980 3100 50  0001 C CNN
@@
 AR Path="/56888583/56A2193A/56A21F7F" Ref="C16"  Part="1"
 AR Path="/56888583/56A25341/56A21F7F" Ref="C22"  Part="1"
-F 0 "C16" H 7075 3850 50  0000 L CNN
+F 0 "C22" H 7075 3850 50  0000 L CNN
 F 1 "2700pF C0G" H 7075 3650 50  0000 L CNN
 F 2 "Capacitors_SMD:C_0603_HandSoldering" H 7088 3600 50  0001 C CNN
@@
 AR Path="/56888583/56A2193A/56A21F90" Ref="R7"  Part="1"
 AR Path="/56888583/56A25341/56A21F90" Ref="R18"  Part="1"
-F 0 "R7" V 5130 3550 50  0000 C CNN
+F 0 "R18" V 5130 3550 50  0000 C CNN
 F 1 "10K" V 5050 3550 50  0000 C CNN
 F 2 "Resistors_SMD:R_0603_HandSoldering" V 4980 3550 50  0001 C CNN
@@
 AR Path="/56888583/56A2193A/56A21F89" Ref="C13"  Part="1"
 AR Path="/56888583/56A25341/56A21F89" Ref="C19"  Part="1"
-F 0 "C13" H 5425 2300 50  0000 L CNN
+F 0 "C19" H 5425 2300 50  0000 L CNN
 F 1 "470pF C0G" V 5600 2000 50  0000 L CNN
 F 2 "Capacitors_SMD:C_0603_HandSoldering" H 5438 2050 50  0001 C CNN
@@
 AR Path="/56888583/56A2193A/56A21F0E" Ref="R5"  Part="1"
 AR Path="/56888583/56A25341/56A21F0E" Ref="R16"  Part="1"
-F 0 "R5" V 4580 3550 50  0000 C CNN
+F 0 "R16" V 4580 3550 50  0000 C CNN
 F 1 "100K" V 4500 3550 50  0000 C CNN
 F 2 "Resistors_SMD:R_0603_HandSoldering" V 4430 3550 50  0001 C CNN
@@
 AR Path="/56888583/56A2193A/56A60AB3" Ref="U2"  Part="1"
 AR Path="/56888583/56A25341/56A60AB3" Ref="U3"  Part="1"
-F 0 "U2" H 5400 3300 50  0000 L CNN
+F 0 "U3" H 5400 3300 50  0000 L CNN
 F 1 "OP1642" H 5400 2850 50  0000 L CNN
 F 2 "Housings_SOIC:SOIC-8_3.9x4.9mm_Pitch1.27mm" H 5450 3100 50  0001 C CNN
@@
 AR Path="/56888583/56A2193A/56A61EC6" Ref="R13"  Part="1"
 AR Path="/56888583/56A25341/56A61EC6" Ref="R24"  Part="1"
-F 0 "R13" V 6630 3100 50  0000 C CNN
+F 0 "R24" V 6630 3100 50  0000 C CNN
 F 1 "200" V 6550 3100 50  0000 C CNN
 F 2 "Resistors_SMD:R_0603_HandSoldering" V 6480 3100 50  0001 C CNN
@@
 AR Path="/56888583/56A2193A/56A62F06" Ref="U2"  Part="2"
 AR Path="/56888583/56A25341/56A62F06" Ref="U3"  Part="2"
-F 0 "U2" H 5400 4600 50  0000 L CNN
+F 0 "U3" H 5400 4600 50  0000 L CNN
 F 1 "OP1642" H 5400 4150 50  0000 L CNN
 F 2 "Housings_SOIC:SOIC-8_3.9x4.9mm_Pitch1.27mm" H 5450 4400 50  0001 C CNN
@@
 AR Path="/56888583/56A2193A/56A63424" Ref="C15"  Part="1"
 AR Path="/56888583/56A25341/56A63424" Ref="C21"  Part="1"
-F 0 "C15" H 5725 3850 50  0000 L CNN
+F 0 "C21" H 5725 3850 50  0000 L CNN
 F 1 "0.1uF" H 5725 3650 50  0000 L CNN
 F 2 "Capacitors_SMD:C_0603_HandSoldering" H 5738 3600 50  0001 C CNN
@@
 AR Path="/56888583/56A2193A/5714F51E" Ref="R6"  Part="1"
 AR Path="/56888583/56A25341/5714F51E" Ref="R17"  Part="1"
-F 0 "R6" V 4580 4550 50  0000 C CNN
+F 0 "R17" V 4580 4550 50  0000 C CNN
 F 1 "100K" V 4500 4550 50  0000 C CNN
 F 2 "Resistors_SMD:R_0603_HandSoldering" V 4430 4550 50  0001 C CNN
@@
 AR Path="/56888583/56A2193A/5714FC91" Ref="R8"  Part="1"
 AR Path="/56888583/56A25341/5714FC91" Ref="R19"  Part="1"
-F 0 "R8" V 5130 3950 50  0000 C CNN
+F 0 "R19" V 5130 3950 50  0000 C CNN
 F 1 "10K" V 5050 3950 50  0000 C CNN
 F 2 "Resistors_SMD:R_0603_HandSoldering" V 4980 3950 50  0001 C CNN
@@
 AR Path="/56888583/56A2193A/57150BC8" Ref="C12"  Part="1"
 AR Path="/56888583/56A25341/57150BC8" Ref="C18"  Part="1"
-F 0 "C12" H 4825 4400 50  0000 L CNN
+F 0 "C18" H 4825 4400 50  0000 L CNN
 F 1 "10uF" H 4825 4200 50  0000 L CNN
 F 2 "Capacitors_ThroughHole:C_Radial_D5_L11_P2" H 4838 4150 50  0001 C CNN
@@
 AR Path="/56888583/56A2193A/5715440C" Ref="R10"  Part="1"
 AR Path="/56888583/56A25341/5715440C" Ref="R21"  Part="1"
-F 0 "R10" V 5480 5650 50  0000 C CNN
+F 0 "R21" V 5480 5650 50  0000 C CNN
 F 1 "634" V 5400 5650 50  0000 C CNN
 F 2 "Resistors_SMD:R_0603_HandSoldering" V 5330 5650 50  0001 C CNN
@@
 AR Path="/56888583/56A2193A/57154E49" Ref="R12"  Part="1"
 AR Path="/56888583/56A25341/57154E49" Ref="R23"  Part="1"
-F 0 "R12" V 6130 4400 50  0000 C CNN
+F 0 "R23" V 6130 4400 50  0000 C CNN
 F 1 "91" V 6050 4400 50  0000 C CNN
 F 2 "Resistors_SMD:R_0603_HandSoldering" V 5980 4400 50  0001 C CNN
@@
 AR Path="/56888583/56A2193A/571552FC" Ref="R14"  Part="1"
 AR Path="/56888583/56A25341/571552FC" Ref="R25"  Part="1"
-F 0 "R14" V 6630 4400 50  0000 C CNN
+F 0 "R25" V 6630 4400 50  0000 C CNN
 F 1 "200" V 6550 4400 50  0000 C CNN
 F 2 "Resistors_SMD:R_0603_HandSoldering" V 6480 4400 50  0001 C CNN
@@
 AR Path="/56888583/56A2193A/57155733" Ref="R15"  Part="1"
 AR Path="/56888583/56A25341/57155733" Ref="R26"  Part="1"
-F 0 "R15" V 6880 3750 50  0000 C CNN
+F 0 "R26" V 6880 3750 50  0000 C CNN
 F 1 "200" V 6800 3750 50  0000 C CNN
 F 2 "Resistors_SMD:R_0603_HandSoldering" V 6730 3750 50  0001 C CNN
@@
 AR Path="/56888583/56A2193A/5715776A" Ref="C14"  Part="1"
 AR Path="/56888583/56A25341/5715776A" Ref="C20"  Part="1"
-F 0 "C14" H 5425 5350 50  0000 L CNN
+F 0 "C20" H 5425 5350 50  0000 L CNN
 F 1 "470pF C0G" V 5600 5050 50  0000 L CNN
 F 2 "Capacitors_SMD:C_0603_HandSoldering" H 5438 5100 50  0001 C CNN
@@
 AR Path="/56888583/56A2193A/57AC2185" Ref="C111"  Part="1"
 AR Path="/56888583/56A25341/57AC2185" Ref="C115"  Part="1"
-F 0 "C111" H 2675 2500 50  0000 L CNN
+F 0 "C115" H 2675 2500 50  0000 L CNN
 F 1 "10uF" H 2675 2300 50  0000 L CNN
 F 2 "Capacitors_ThroughHole:C_Radial_D5_L11_P2" H 2688 2250 50  0001 C CNN
@@
 AR Path="/56888583/56A2193A/57AC218E" Ref="C114"  Part="1"
 AR Path="/56888583/56A25341/57AC218E" Ref="C118"  Part="1"
-F 0 "C114" H 3675 2500 50  0000 L CNN
+F 0 "C118" H 3675 2500 50  0000 L CNN
 F 1 "10uF" H 3675 2300 50  0000 L CNN
 F 2 "Capacitors_ThroughHole:C_Radial_D5_L11_P2" H 3688 2250 50  0001 C CNN
@@
 AR Path="/56888583/56A2193A/57AC2197" Ref="C112"  Part="1"
 AR Path="/56888583/56A25341/57AC2197" Ref="C116"  Part="1"
-F 0 "C112" H 2975 2500 50  0000 L CNN
+F 0 "C116" H 2975 2500 50  0000 L CNN
 F 1 "0.1uF" H 2975 2300 50  0000 L CNN
 F 2 "Capacitors_SMD:C_0603_HandSoldering" H 2988 2250 50  0001 C CNN
@@
 AR Path="/56888583/56A2193A/57AC21A0" Ref="C113"  Part="1"
 AR Path="/56888583/56A25341/57AC21A0" Ref="C117"  Part="1"
-F 0 "C113" H 3375 2500 50  0000 L CNN
+F 0 "C117" H 3375 2500 50  0000 L CNN
 F 1 "0.1uF" H 3375 2300 50  0000 L CNN
 F 2 "Capacitors_SMD:C_0603_HandSoldering" H 3388 2250 50  0001 C CNN
@@
 AR Path="/56888583/56A2193A/57AC3BC1" Ref="R106"  Part="1"
 AR Path="/56888583/56A25341/57AC3BC1" Ref="R108"  Part="1"
-F 0 "R106" V 2430 2200 50  0000 C CNN
+F 0 "R108" V 2430 2200 50  0000 C CNN
 F 1 "0.01" V 2350 2200 50  0000 C CNN
-F 2 "" V 2280 2200 50  0000 C CNN
+F 2 "Resistors_SMD:R_0603_HandSoldering" V 2280 2200 50  0001 C CNN
 F 3 "" H 2350 2200 50  0000 C CNN
 	1    2350 2200
@@
 AR Path="/56888583/56A2193A/57AC3C63" Ref="R107"  Part="1"
 AR Path="/56888583/56A25341/57AC3C63" Ref="R109"  Part="1"
-F 0 "R107" V 4030 2200 50  0000 C CNN
+F 0 "R109" V 4030 2200 50  0000 C CNN
 F 1 "0.01" V 3950 2200 50  0000 C CNN
-F 2 "" V 3880 2200 50  0000 C CNN
+F 2 "Resistors_SMD:R_0603_HandSoldering" V 3880 2200 50  0001 C CNN
 F 3 "" H 3950 2200 50  0000 C CNN
 	1    3950 2200

Commit message: Moving sense resistors into place
Connections:
- net labels added: +12L, -12L
- wire segments 57 -> 63
