File: pcb/analog_input_buffer.sch (KiCad schematic (older format))
At the start: 24 parts, among them U2 OP1642

Commit message: More cleanup and switched sense resistors
Increased the resistance of the current sense resistors up to 0.1 ohm.
Parts:
- R106, R107: value 0.01 -> 0.1
Changed lines of the file:
@@
 AR Path="/56888583/56A25341/57AC3BC1" Ref="R108"  Part="1"
 F 0 "R106" V 2430 2200 50  0000 C CNN
-F 1 "0.01" V 2350 2200 50  0000 C CNN
+F 1 "0.1" V 2350 2200 50  0000 C CNN
 F 2 "Resistors_SMD:R_0603_HandSoldering" V 2280 2200 50  0001 C CNN
 F 3 "" H 2350 2200 50  0000 C CNN
@@
 AR Path="/56888583/56A25341/57AC3C63" Ref="R109"  Part="1"
 F 0 "R107" V 4030 2200 50  0000 C CNN
-F 1 "0.01" V 3950 2200 50  0000 C CNN
+F 1 "0.1" V 3950 2200 50  0000 C CNN
 F 2 "Resistors_SMD:R_0603_HandSoldering" V 3880 2200 50  0001 C CNN
 F 3 "" H 3950 2200 50  0000 C CNN
