File: pcb/ft2232d.sch (KiCad schematic (older format))
At the start: 26 parts, among them U4 93CxxA, U5 FT2232D, X1 6MHz

Commit message: Began cleaning up ERC errors
Connections:
- no-connect marks 2 -> 19
Changed lines of the file:
@@
 $Descr A4 11693 8268
 encoding utf-8
-Sheet 9 9
+Sheet 5 9
 Title "USB FGPA Programming Interface"
 Date ""
@@
 $EndComp
 $Comp
-L GND #PWR44
+L GND #PWR031
 U 1 1 56A42CE2
 P 4400 4250
-F 0 "#PWR44" H 4400 4000 50  0001 C CNN
+F 0 "#PWR031" H 4400 4000 50  0001 C CNN
 F 1 "GND" H 4400 4100 50  0000 C CNN
 F 2 "" H 4400 4250 50  0000 C CNN
@@
 NoConn ~ 4450 5650
 $Comp
-L GND #PWR42
+L GND #PWR032
 U 1 1 56A43CD0
 P 3800 5700
-F 0 "#PWR42" H 3800 5450 50  0001 C CNN
+F 0 "#PWR032" H 3800 5450 50  0001 C CNN
 F 1 "GND" H 3800 5550 50  0000 C CNN
 F 2 "" H 3800 5700 50  0000 C CNN
@@
 $EndComp
 $Comp
-L GND #PWR47
+L GND #PWR033
 U 1 1 56A43CF4
 P 5100 5200
-F 0 "#PWR47" H 5100 4950 50  0001 C CNN
+F 0 "#PWR033" H 5100 4950 50  0001 C CNN
 F 1 "GND" H 5100 5050 50  0000 C CNN
 F 2 "" H 5100 5200 50  0000 C CNN
@@
 $EndComp
 $Comp
-L GND #PWR53
+L GND #PWR034
 U 1 1 56A43D18
 P 6050 5800
-F 0 "#PWR53" H 6050 5550 50  0001 C CNN
+F 0 "#PWR034" H 6050 5550 50  0001 C CNN
 F 1 "GND" H 6050 5650 50  0000 C CNN
 F 2 "" H 6050 5800 50  0000 C CNN
@@
 $EndComp
 $Comp
-L GND #PWR45
+L GND #PWR035
 U 1 1 56A45799
 P 4850 2750
-F 0 "#PWR45" H 4850 2500 50  0001 C CNN
+F 0 "#PWR035" H 4850 2500 50  0001 C CNN
 F 1 "GND" H 4850 2600 50  0000 C CNN
 F 2 "" H 4850 2750 50  0000 C CNN
@@
 	8000 5100 8000 5000
 $Comp
-L +3.3V #PWR54
+L +3.3V #PWR036
 U 1 1 56A48B0E
 P 6400 1200
-F 0 "#PWR54" H 6400 1050 50  0001 C CNN
+F 0 "#PWR036" H 6400 1050 50  0001 C CNN
 F 1 "+3.3V" H 6400 1340 50  0000 C CNN
 F 2 "" H 6400 1200 50  0000 C CNN
@@
 $EndComp
 $Comp
-L +3.3V #PWR59
+L +3.3V #PWR037
 U 1 1 56A4AC53
 P 8200 5200
-F 0 "#PWR59" H 8200 5050 50  0001 C CNN
+F 0 "#PWR037" H 8200 5050 50  0001 C CNN
 F 1 "+3.3V" H 8200 5340 50  0000 C CNN
 F 2 "" H 8200 5200 50  0000 C CNN
@@
 	7000 5200 8200 5200
 $Comp
-L +3.3V #PWR57
+L +3.3V #PWR038
 U 1 1 56A4B585
 P 7700 4600
-F 0 "#PWR57" H 7700 4450 50  0001 C CNN
+F 0 "#PWR038" H 7700 4450 50  0001 C CNN
 F 1 "+3.3V" H 7700 4740 50  0000 C CNN
 F 2 "" H 7700 4600 50  0000 C CNN
@@
 $EndComp
 $Comp
-L +3.3V #PWR58
+L +3.3V #PWR039
 U 1 1 56A4B6FF
 P 8000 4600
-F 0 "#PWR58" H 8000 4450 50  0001 C CNN
+F 0 "#PWR039" H 8000 4450 50  0001 C CNN
 F 1 "+3.3V" H 8000 4740 50  0000 C CNN
 F 2 "" H 8000 4600 50  0000 C CNN
@@
 $EndComp
 $Comp
-L +3.3V #PWR56
+L +3.3V #PWR040
 U 1 1 56A4C262
 P 7200 3700
-F 0 "#PWR56" H 7200 3550 50  0001 C CNN
+F 0 "#PWR040" H 7200 3550 50  0001 C CNN
 F 1 "+3.3V" H 7200 3840 50  0000 C CNN
 F 2 "" H 7200 3700 50  0000 C CNN
@@
 $EndComp
 $Comp
-L GND #PWR49
+L GND #PWR041
 U 1 1 56A4C939
 P 5150 2200
-F 0 "#PWR49" H 5150 1950 50  0001 C CNN
+F 0 "#PWR041" H 5150 1950 50  0001 C CNN
 F 1 "GND" H 5150 2050 50  0000 C CNN
 F 2 "" H 5150 2200 50  0000 C CNN
@@
 Connection ~ 3850 3800
 $Comp
-L GND #PWR43
+L GND #PWR042
 U 1 1 56A50E44
 P 3850 4200
-F 0 "#PWR43" H 3850 3950 50  0001 C CNN
+F 0 "#PWR042" H 3850 3950 50  0001 C CNN
 F 1 "GND" H 3850 4050 50  0000 C CNN
 F 2 "" H 3850 4200 50  0000 C CNN
@@
 $EndComp
 $Comp
-L +5V #PWR52
+L +5V #PWR043
 U 1 1 56A51073
 P 6050 1200
-F 0 "#PWR52" H 6050 1050 50  0001 C CNN
+F 0 "#PWR043" H 6050 1050 50  0001 C CNN
 F 1 "+5V" H 6050 1340 50  0000 C CNN
 F 2 "" H 6050 1200 50  0000 C CNN
@@
 $EndComp
 $Comp
-L +5V #PWR41
+L +5V #PWR044
 U 1 1 56A514D9
 P 3800 5300
-F 0 "#PWR41" H 3800 5150 50  0001 C CNN
+F 0 "#PWR044" H 3800 5150 50  0001 C CNN
 F 1 "+5V" H 3800 5440 50  0000 C CNN
 F 2 "" H 3800 5300 50  0000 C CNN
@@
 $EndComp
 $Comp
-L +5V #PWR46
+L +5V #PWR045
 U 1 1 56A5151B
 P 4850 5650
-F 0 "#PWR46" H 4850 5500 50  0001 C CNN
+F 0 "#PWR045" H 4850 5500 50  0001 C CNN
 F 1 "+5V" H 4850 5790 50  0000 C CNN
 F 2 "" H 4850 5650 50  0000 C CNN
@@
 $EndComp
 $Comp
-L GND #PWR48
+L GND #PWR046
 U 1 1 56A550EE
 P 5150 1600
-F 0 "#PWR48" H 5150 1350 50  0001 C CNN
+F 0 "#PWR046" H 5150 1350 50  0001 C CNN
 F 1 "GND" H 5150 1450 50  0000 C CNN
 F 2 "" H 5150 1600 50  0000 C CNN
@@
 $EndComp
 $Comp
-L GND #PWR50
+L GND #PWR047
 U 1 1 56A55147
 P 5450 1600
-F 0 "#PWR50" H 5450 1350 50  0001 C CNN
+F 0 "#PWR047" H 5450 1350 50  0001 C CNN
 F 1 "GND" H 5450 1450 50  0000 C CNN
 F 2 "" H 5450 1600 50  0000 C CNN
@@
 $EndComp
 $Comp
-L GND #PWR51
+L GND #PWR048
 U 1 1 56A551A0
 P 5750 1600
-F 0 "#PWR51" H 5750 1350 50  0001 C CNN
+F 0 "#PWR048" H 5750 1350 50  0001 C CNN
 F 1 "GND" H 5750 1450 50  0000 C CNN
 F 2 "" H 5750 1600 50  0000 C CNN
@@
 $EndComp
 $Comp
-L GND #PWR55
+L GND #PWR049
 U 1 1 56A56EFD
 P 6400 1600
-F 0 "#PWR55" H 6400 1350 50  0001 C CNN
+F 0 "#PWR049" H 6400 1350 50  0001 C CNN
 F 1 "GND" H 6400 1450 50  0000 C CNN
 F 2 "" H 6400 1600 50  0000 C CNN
@@
 	6250 2050 6250 2100
 Connection ~ 6150 2050
-$Comp
-L +3.3V #PWR61
-U 1 1 56A57FC6
-P 9150 1150
-F 0 "#PWR61" H 9150 1000 50  0001 C CNN
-F 1 "+3.3V" H 9150 1290 50  0000 C CNN
-F 2 "" H 9150 1150 50  0000 C CNN
-F 3 "" H 9150 1150 50  0000 C CNN
-	1    9150 1150
-	1    0    0    -1
-$EndComp
-$Comp
-L +5V #PWR62
-U 1 1 56A58022
-P 9550 1150
-F 0 "#PWR62" H 9550 1000 50  0001 C CNN
-F 1 "+5V" H 9550 1290 50  0000 C CNN
-F 2 "" H 9550 1150 50  0000 C CNN
-F 3 "" H 9550 1150 50  0000 C CNN
-	1    9550 1150
-	1    0    0    -1
-$EndComp
-$Comp
-L GND #PWR60
-U 1 1 56A5807E
-P 8800 1200
-F 0 "#PWR60" H 8800 950 50  0001 C CNN
-F 1 "GND" H 8800 1050 50  0000 C CNN
-F 2 "" H 8800 1200 50  0000 C CNN
-F 3 "" H 8800 1200 50  0000 C CNN
-	1    8800 1200
-	1    0    0    -1
-$EndComp
-$Comp
-L PWR_FLAG #FLG11
-U 1 1 56A580C1
-P 8800 1200
-F 0 "#FLG11" H 8800 1295 50  0001 C CNN
-F 1 "PWR_FLAG" H 8800 1380 50  0000 C CNN
-F 2 "" H 8800 1200 50  0000 C CNN
-F 3 "" H 8800 1200 50  0000 C CNN
-	1    8800 1200
-	1    0    0    -1
-$EndComp
-$Comp
-L PWR_FLAG #FLG12
-U 1 1 56A5813F
-P 9150 1150
-F 0 "#FLG12" H 9150 1245 50  0001 C CNN
-F 1 "PWR_FLAG" H 9150 1330 50  0000 C CNN
-F 2 "" H 9150 1150 50  0000 C CNN
-F 3 "" H 9150 1150 50  0000 C CNN
-	1    9150 1150
-	-1   0    0    1
-$EndComp
-$Comp
-L PWR_FLAG #FLG13
-U 1 1 56A5819B
-P 9550 1150
-F 0 "#FLG13" H 9550 1245 50  0001 C CNN
-F 1 "PWR_FLAG" H 9550 1330 50  0000 C CNN
-F 2 "" H 9550 1150 50  0000 C CNN
-F 3 "" H 9550 1150 50  0000 C CNN
-	1    9550 1150
-	-1   0    0    1
-$EndComp
 Text HLabel 4400 3300 0    60   BiDi ~ 0
 D+
@@
 Wire Wire Line
 	3850 3300 3850 3400
+NoConn ~ 7000 5400
+NoConn ~ 7000 2800
+NoConn ~ 7000 2900
+NoConn ~ 7000 3000
+NoConn ~ 7000 3100
+NoConn ~ 7000 3300
+NoConn ~ 7000 3400
+NoConn ~ 7000 3500
+NoConn ~ 7000 3600
+NoConn ~ 7000 4100
+NoConn ~ 7000 4200
+NoConn ~ 7000 4300
+NoConn ~ 7000 4400
+NoConn ~ 7000 4500
+NoConn ~ 7000 4600
+NoConn ~ 7000 4800
+NoConn ~ 7000 4900
 $EndSCHEMATC

Commit message: Cleaned up ERC
Changed lines of the file:
@@
 $EndComp
 $Comp
-L GND #PWR34
+L GND #PWR031
 U 1 1 56A42CE2
 P 4400 4250
-F 0 "#PWR34" H 4400 4000 50  0001 C CNN
+F 0 "#PWR031" H 4400 4000 50  0001 C CNN
 F 1 "GND" H 4400 4100 50  0000 C CNN
 F 2 "" H 4400 4250 50  0000 C CNN
@@
 NoConn ~ 4450 5650
 $Comp
-L GND #PWR32
+L GND #PWR032
 U 1 1 56A43CD0
 P 3800 5700
-F 0 "#PWR32" H 3800 5450 50  0001 C CNN
+F 0 "#PWR032" H 3800 5450 50  0001 C CNN
 F 1 "GND" H 3800 5550 50  0000 C CNN
 F 2 "" H 3800 5700 50  0000 C CNN
@@
 $EndComp
 $Comp
-L GND #PWR37
+L GND #PWR033
 U 1 1 56A43CF4
 P 5100 5200
-F 0 "#PWR37" H 5100 4950 50  0001 C CNN
+F 0 "#PWR033" H 5100 4950 50  0001 C CNN
 F 1 "GND" H 5100 5050 50  0000 C CNN
 F 2 "" H 5100 5200 50  0000 C CNN
@@
 $EndComp
 $Comp
-L GND #PWR43
+L GND #PWR034
 U 1 1 56A43D18
 P 6050 5800
-F 0 "#PWR43" H 6050 5550 50  0001 C CNN
+F 0 "#PWR034" H 6050 5550 50  0001 C CNN
 F 1 "GND" H 6050 5650 50  0000 C CNN
 F 2 "" H 6050 5800 50  0000 C CNN
@@
 $EndComp
 $Comp
-L GND #PWR35
+L GND #PWR035
 U 1 1 56A45799
 P 4850 2750
-F 0 "#PWR35" H 4850 2500 50  0001 C CNN
+F 0 "#PWR035" H 4850 2500 50  0001 C CNN
 F 1 "GND" H 4850 2600 50  0000 C CNN
 F 2 "" H 4850 2750 50  0000 C CNN
@@
 	8000 5100 8000 5000
 $Comp
-L +3.3V #PWR44
+L +3.3V #PWR036
 U 1 1 56A48B0E
 P 6400 1200
-F 0 "#PWR44" H 6400 1050 50  0001 C CNN
+F 0 "#PWR036" H 6400 1050 50  0001 C CNN
 F 1 "+3.3V" H 6400 1340 50  0000 C CNN
 F 2 "" H 6400 1200 50  0000 C CNN
@@
 $EndComp
 $Comp
-L +3.3V #PWR49
+L +3.3V #PWR037
 U 1 1 56A4AC53
 P 8200 5200
-F 0 "#PWR49" H 8200 5050 50  0001 C CNN
+F 0 "#PWR037" H 8200 5050 50  0001 C CNN
 F 1 "+3.3V" H 8200 5340 50  0000 C CNN
 F 2 "" H 8200 5200 50  0000 C CNN
@@
 	7000 5200 8200 5200
 $Comp
-L +3.3V #PWR47
+L +3.3V #PWR038
 U 1 1 56A4B585
 P 7700 4600
-F 0 "#PWR47" H 7700 4450 50  0001 C CNN
+F 0 "#PWR038" H 7700 4450 50  0001 C CNN
 F 1 "+3.3V" H 7700 4740 50  0000 C CNN
 F 2 "" H 7700 4600 50  0000 C CNN
@@
 $EndComp
 $Comp
-L +3.3V #PWR48
+L +3.3V #PWR039
 U 1 1 56A4B6FF
 P 8000 4600
-F 0 "#PWR48" H 8000 4450 50  0001 C CNN
+F 0 "#PWR039" H 8000 4450 50  0001 C CNN
 F 1 "+3.3V" H 8000 4740 50  0000 C CNN
 F 2 "" H 8000 4600 50  0000 C CNN
@@
 $EndComp
 $Comp
-L +3.3V #PWR46
+L +3.3V #PWR040
 U 1 1 56A4C262
 P 7200 3700
-F 0 "#PWR46" H 7200 3550 50  0001 C CNN
+F 0 "#PWR040" H 7200 3550 50  0001 C CNN
 F 1 "+3.3V" H 7200 3840 50  0000 C CNN
 F 2 "" H 7200 3700 50  0000 C CNN
@@
 $EndComp
 $Comp
-L GND #PWR39
+L GND #PWR041
 U 1 1 56A4C939
 P 5150 2200
-F 0 "#PWR39" H 5150 1950 50  0001 C CNN
+F 0 "#PWR041" H 5150 1950 50  0001 C CNN
 F 1 "GND" H 5150 2050 50  0000 C CNN
 F 2 "" H 5150 2200 50  0000 C CNN
@@
 $EndComp
 Wire Wire Line
-	5150 1900 5700 1900
+	5100 1900 5700 1900
 Wire Wire Line
 	6050 1900 6000 1900
@@
 Connection ~ 3850 3800
 $Comp
-L GND #PWR33
+L GND #PWR042
 U 1 1 56A50E44
 P 3850 4200
-F 0 "#PWR33" H 3850 3950 50  0001 C CNN
+F 0 "#PWR042" H 3850 3950 50  0001 C CNN
 F 1 "GND" H 3850 4050 50  0000 C CNN
 F 2 "" H 3850 4200 50  0000 C CNN
@@
 $EndComp
 $Comp
-L +5V #PWR42
+L +5V #PWR043
 U 1 1 56A51073
 P 6050 1200
-F 0 "#PWR42" H 6050 1050 50  0001 C CNN
+F 0 "#PWR043" H 6050 1050 50  0001 C CNN
 F 1 "+5V" H 6050 1340 50  0000 C CNN
 F 2 "" H 6050 1200 50  0000 C CNN
@@
 $EndComp
 $Comp
-L +5V #PWR31
+L +5V #PWR044
 U 1 1 56A514D9
 P 3800 5300
-F 0 "#PWR31" H 3800 5150 50  0001 C CNN
+F 0 "#PWR044" H 3800 5150 50  0001 C CNN
 F 1 "+5V" H 3800 5440 50  0000 C CNN
 F 2 "" H 3800 5300 50  0000 C CNN
@@
 $EndComp
 $Comp
-L +5V #PWR36
+L +5V #PWR045
 U 1 1 56A5151B
 P 4850 5650
-F 0 "#PWR36" H 4850 5500 50  0001 C CNN
+F 0 "#PWR045" H 4850 5500 50  0001 C CNN
 F 1 "+5V" H 4850 5790 50  0000 C CNN
 F 2 "" H 4850 5650 50  0000 C CNN
@@
 $EndComp
 $Comp
-L GND #PWR38
+L GND #PWR046
 U 1 1 56A550EE
 P 5150 1600
-F 0 "#PWR38" H 5150 1350 50  0001 C CNN
+F 0 "#PWR046" H 5150 1350 50  0001 C CNN
 F 1 "GND" H 5150 1450 50  0000 C CNN
 F 2 "" H 5150 1600 50  0000 C CNN
@@
 $EndComp
 $Comp
-L GND #PWR40
+L GND #PWR047
 U 1 1 56A55147
 P 5450 1600
-F 0 "#PWR40" H 5450 1350 50  0001 C CNN
+F 0 "#PWR047" H 5450 1350 50  0001 C CNN
 F 1 "GND" H 5450 1450 50  0000 C CNN
 F 2 "" H 5450 1600 50  0000 C CNN
@@
 $EndComp
 $Comp
-L GND #PWR41
+L GND #PWR048
 U 1 1 56A551A0
 P 5750 1600
-F 0 "#PWR41" H 5750 1350 50  0001 C CNN
+F 0 "#PWR048" H 5750 1350 50  0001 C CNN
 F 1 "GND" H 5750 1450 50  0000 C CNN
 F 2 "" H 5750 1600 50  0000 C CNN
@@
 $EndComp
 $Comp
-L GND #PWR45
+L GND #PWR049
 U 1 1 56A56EFD
 P 6400 1600
-F 0 "#PWR45" H 6400 1350 50  0001 C CNN
+F 0 "#PWR049" H 6400 1350 50  0001 C CNN
 F 1 "GND" H 6400 1450 50  0000 C CNN
 F 2 "" H 6400 1600 50  0000 C CNN
@@
 NoConn ~ 7000 4800
 NoConn ~ 7000 4900
+$Comp
+L PWR_FLAG #FLG050
+U 1 1 57151F2A
+P 5100 1900
+F 0 "#FLG050" H 5100 1995 50  0001 C CNN
+F 1 "PWR_FLAG" H 5100 2080 50  0000 C CNN
+F 2 "" H 5100 1900 50  0000 C CNN
+F 3 "" H 5100 1900 50  0000 C CNN
+	1    5100 1900
+	0    -1   -1   0
+$EndComp
+Connection ~ 5150 1900
 $EndSCHEMATC

Commit message: Latest work on footprints and BOM
Parts:
- removed R28, R32: 10K, symbol R
- removed R30: 27, symbol R
- removed R37, R38, R39: 68, symbol R
- added R? (x3): 68, Resistors_SMD:R_0603, symbol R
- added R?: 27, Resistors_SMD:R_0603, symbol R
- added R? (x2): 10K, Resistors_SMD:R_0603, symbol R
- C23: footprint (none) -> Capacitors_SMD:C_0603; Manufacturer (none) -> Murata; Manufacturer Part Number (none) -> GRM188R71E333KA01
- C24, C25, C26, C28: footprint (none) -> Capacitors_SMD:C_0603; Manufacturer (none) -> Murata; Manufacturer Part Number (none) -> GRM188R61C104KA01
- C27: footprint (none) -> Capacitors_SMD:C_0603; Manufacturer (none) -> Murata; Manufacturer Part Number (none) -> GRM188R61A106KE69
- R27: footprint (none) -> Resistors_SMD:R_0603; Manufacturer (none) -> Panasonic; Manufacturer Part Number (none) -> ERJ-3GEYJ472V
- R29: footprint (none) -> Resistors_SMD:R_0603; Manufacturer (none) -> Panasonic; Manufacturer Part Number (none) -> ERJ-3EKF27R0V
- R34: footprint (none) -> Resistors_SMD:R_0603; Manufacturer (none) -> Panasonic; Manufacturer Part Number (none) -> ERJ-3EKF1501V
- R35: footprint (none) -> Resistors_SMD:R_0603; Manufacturer (none) -> Panasonic; Manufacturer Part Number (none) -> ERJ-3EKF1004V
- R36: footprint (none) -> Resistors_SMD:R_0603; Manufacturer (none) -> Panasonic; Manufacturer Part Number (none) -> ERJ-3EKF4700V
- X1: Manufacturer (none) -> Murata; Manufacturer Part Number (none) -> CSTCR6M00G55-R0
Changed lines of the file:
@@
 F 0 "R34" V 5030 3450 50  0000 C CNN
 F 1 "1.5K" V 4950 3450 50  0000 C CNN
-F 2 "" V 4880 3450 50  0000 C CNN
+F 2 "Resistors_SMD:R_0603" V 4880 3450 50  0001 C CNN
 F 3 "" H 4950 3450 50  0000 C CNN
+F 4 "Panasonic" V 4950 3450 60  0001 C CNN "Manufacturer"
+F 5 "ERJ-3EKF1501V" V 4950 3450 60  0001 C CNN "Manufacturer Part Number"
 	1    4950 3450
 	1    0    0    -1
@@
 F 0 "R35" V 5030 4250 50  0000 C CNN
 F 1 "1M" V 4950 4250 50  0000 C CNN
-F 2 "" V 4880 4250 50  0000 C CNN
+F 2 "Resistors_SMD:R_0603" V 4880 4250 50  0001 C CNN
 F 3 "" H 4950 4250 50  0000 C CNN
+F 4 "Panasonic" V 4950 4250 60  0001 C CNN "Manufacturer"
+F 5 "ERJ-3EKF1004V" V 4950 4250 60  0001 C CNN "Manufacturer Part Number"
 	1    4950 4250
 	1    0    0    -1
@@
 F 2 "" H 4700 4250 50  0000 C CNN
 F 3 "" H 4700 4250 50  0000 C CNN
+F 4 "Murata" H 4700 4250 60  0001 C CNN "Manufacturer"
+F 5 "CSTCR6M00G55-R0" H 4700 4250 60  0001 C CNN "Manufacturer Part Number"
 	1    4700 4250
 	0    1    1    0
@@
 	4650 5100 4650 5000
 Connection ~ 4650 5000
-$Comp
-L R R32
-U 1 1 56A43C4A
-P 4650 5650
-F 0 "R32" V 4730 5650 50  0000 C CNN
-F 1 "10K" V 4650 5650 50  0000 C CNN
-F 2 "" V 4580 5650 50  0000 C CNN
-F 3 "" H 4650 5650 50  0000 C CNN
-	1    4650 5650
-	1    0    0    -1
-$EndComp
 Connection ~ 4650 5450
 NoConn ~ 4450 5550
@@
 F 0 "C23" H 4875 2700 50  0000 L CNN
 F 1 "33nF" H 4875 2500 50  0000 L CNN
-F 2 "" H 4888 2450 50  0000 C CNN
+F 2 "Capacitors_SMD:C_0603" H 4888 2450 50  0001 C CNN
 F 3 "" H 4850 2600 50  0000 C CNN
+F 4 "Murata" H 4850 2600 60  0001 C CNN "Manufacturer"
+F 5 "GRM188R71E333KA01" H 4850 2600 60  0001 C CNN "Manufacturer Part Number"
 	1    4850 2600
 	1    0    0    -1
@@
 Text HLabel 7700 2700 2    60   Output ~ 0
 TMS
-$Comp
-L R R37
-U 1 1 56A462EE
-P 7300 2400
-F 0 "R37" V 7350 2200 50  0000 C CNN
-F 1 "68" V 7300 2400 50  0000 C CNN
-F 2 "" V 7230 2400 50  0000 C CNN
-F 3 "" H 7300 2400 50  0000 C CNN
-	1    7300 2400
-	0    -1   -1   0
-$EndComp
-$Comp
-L R R38
-U 1 1 56A4641A
-P 7300 2500
-F 0 "R38" V 7350 2300 50  0000 C CNN
-F 1 "68" V 7300 2500 50  0000 C CNN
-F 2 "" V 7230 2500 50  0000 C CNN
-F 3 "" H 7300 2500 50  0000 C CNN
-	1    7300 2500
-	0    -1   -1   0
-$EndComp
-$Comp
-L R R39
-U 1 1 56A46452
-P 7300 2700
-F 0 "R39" V 7350 2500 50  0000 C CNN
-F 1 "68" V 7300 2700 50  0000 C CNN
-F 2 "" V 7230 2700 50  0000 C CNN
-F 3 "" H 7300 2700 50  0000 C CNN
-	1    7300 2700
-	0    -1   -1   0
-$EndComp
 Wire Wire Line
 	7000 2400 7150 2400
@@
 F 0 "R36" V 5930 1900 50  0000 C CNN
 F 1 "470" V 5850 1900 50  0000 C CNN
-F 2 "" V 5780 1900 50  0000 C CNN
+F 2 "Resistors_SMD:R_0603" V 5780 1900 50  0001 C CNN
 F 3 "" H 5850 1900 50  0000 C CNN
+F 4 "Panasonic" V 5850 1900 60  0001 C CNN "Manufacturer"
+F 5 "ERJ-3EKF4700V" V 5850 1900 60  0001 C CNN "Manufacturer Part Number"
 	1    5850 1900
 	0    1    1    0
-$EndComp
-$Comp
-L C C25
-U 1 1 56A4C8B8
-P 5150 2050
-F 0 "C25" H 5175 2150 50  0000 L CNN
-F 1 "0.1uF" H 5175 1950 50  0000 L CNN
-F 2 "" H 5188 1900 50  0000 C CNN
-F 3 "" H 5150 2050 50  0000 C CNN
-	1    5150 2050
-	1    0    0    -1
 $EndComp
 $Comp
@@
 F 0 "R29" V 4730 3000 50  0000 C CNN
 F 1 "27" V 4650 3000 50  0000 C CNN
-F 2 "" V 4580 3000 50  0000 C CNN
+F 2 "Resistors_SMD:R_0603" V 4580 3000 50  0001 C CNN
 F 3 "" H 4650 3000 50  0000 C CNN
+F 4 "Panasonic" V 4650 3000 60  0001 C CNN "Manufacturer"
+F 5 "ERJ-3EKF27R0V" V 4650 3000 60  0001 C CNN "Manufacturer Part Number"
 	1    4650 3000
-	0    1    1    0
-$EndComp
-$Comp
-L R R30
-U 1 1 56A4D2BC
-P 4650 3300
-F 0 "R30" V 4730 3300 50  0000 C CNN
-F 1 "27" V 4650 3300 50  0000 C CNN
-F 2 "" V 4580 3300 50  0000 C CNN
-F 3 "" H 4650 3300 50  0000 C CNN
-	1    4650 3300
 	0    1    1    0
 $EndComp
@@
 F 0 "R27" V 3930 3550 50  0000 C CNN
 F 1 "4.7K" V 3850 3550 50  0000 C CNN
-F 2 "" V 3780 3550 50  0000 C CNN
+F 2 "Resistors_SMD:R_0603" V 3780 3550 50  0001 C CNN
 F 3 "" H 3850 3550 50  0000 C CNN
+F 4 "Panasonic" V 3850 3550 60  0001 C CNN "Manufacturer"
+F 5 "ERJ-3GEYJ472V" V 3850 3550 60  0001 C CNN "Manufacturer Part Number"
 	1    3850 3550
-	1    0    0    -1
-$EndComp
-$Comp
-L R R28
-U 1 1 56A50C74
-P 3850 4050
-F 0 "R28" V 3930 4050 50  0000 C CNN
-F 1 "10K" V 3850 4050 50  0000 C CNN
-F 2 "" V 3780 4050 50  0000 C CNN
-F 3 "" H 3850 4050 50  0000 C CNN
-	1    3850 4050
-	1    0    0    -1
+	-1   0    0    1
 $EndComp
 Wire Wire Line
@@
 F 0 "C27" H 5775 1550 50  0000 L CNN
 F 1 "10uF" H 5775 1350 50  0000 L CNN
-F 2 "" H 5788 1300 50  0000 C CNN
+F 2 "Capacitors_SMD:C_0603" H 5788 1300 50  0001 C CNN
 F 3 "" H 5750 1450 50  0000 C CNN
+F 4 "Murata" H 5750 1450 60  0001 C CNN "Manufacturer"
+F 5 "GRM188R61A106KE69" H 5750 1450 60  0001 C CNN "Manufacturer Part Number"
 	1    5750 1450
-	1    0    0    -1
-$EndComp
-$Comp
-L C C26
-U 1 1 56A54EB1
-P 5450 1450
-F 0 "C26" H 5475 1550 50  0000 L CNN
-F 1 "0.1uF" H 5475 1350 50  0000 L CNN
-F 2 "" H 5488 1300 50  0000 C CNN
-F 3 "" H 5450 1450 50  0000 C CNN
-	1    5450 1450
-	1    0    0    -1
-$EndComp
-$Comp
-L C C24
-U 1 1 56A5501C
-P 5150 1450
-F 0 "C24" H 5175 1550 50  0000 L CNN
-F 1 "0.1uF" H 5175 1350 50  0000 L CNN
-F 2 "" H 5188 1300 50  0000 C CNN
-F 3 "" H 5150 1450 50  0000 C CNN
-	1    5150 1450
 	1    0    0    -1
 $EndComp
@@
 	5750 1300 5750 1250
 Connection ~ 5750 1250
-$Comp
-L C C28
-U 1 1 56A56EF7
-P 6400 1450
-F 0 "C28" H 6425 1550 50  0000 L CNN
-F 1 "0.1uF" H 6425 1350 50  0000 L CNN
-F 2 "" H 6438 1300 50  0000 C CNN
-F 3 "" H 6400 1450 50  0000 C CNN
-	1    6400 1450
-	1    0    0    -1
-$EndComp
 $Comp
 L GND #PWR049
@@
 $EndComp
 Connection ~ 5150 1900
+$Comp
+L C C24
+U 1 1 5715BBFF
+P 5150 1450
+F 0 "C24" H 5175 1550 50  0000 L CNN
+F 1 "0.1uF" H 5175 1350 50  0000 L CNN
+F 2 "Capacitors_SMD:C_0603" H 5188 1300 50  0001 C CNN
+F 3 "" H 5150 1450 50  0000 C CNN
+F 4 "Murata" H 5150 1450 60  0001 C CNN "Manufacturer"
+F 5 "GRM188R61C104KA01" H 5150 1450 60  0001 C CNN "Manufacturer Part Number"
+	1    5150 1450
+	1    0    0    -1
+$EndComp
+$Comp
+L C C26
+U 1 1 5715BCAE
+P 5450 1450
+F 0 "C26" H 5475 1550 50  0000 L CNN
+F 1 "0.1uF" H 5475 1350 50  0000 L CNN
+F 2 "Capacitors_SMD:C_0603" H 5488 1300 50  0001 C CNN
+F 3 "" H 5450 1450 50  0000 C CNN
+F 4 "Murata" H 5450 1450 60  0001 C CNN "Manufacturer"
+F 5 "GRM188R61C104KA01" H 5450 1450 60  0001 C CNN "Manufacturer Part Number"
+	1    5450 1450
+	1    0    0    -1
+$EndComp
+$Comp
+L C C28
+U 1 1 5715BD1C
+P 6400 1450
+F 0 "C28" H 6425 1550 50  0000 L CNN
+F 1 "0.1uF" H 6425 1350 50  0000 L CNN
+F 2 "Capacitors_SMD:C_0603" H 6438 1300 50  0001 C CNN
+F 3 "" H 6400 1450 50  0000 C CNN
+F 4 "Murata" H 6400 1450 60  0001 C CNN "Manufacturer"
+F 5 "GRM188R61C104KA01" H 6400 1450 60  0001 C CNN "Manufacturer Part Number"
+	1    6400 1450
+	1    0    0    -1
+$EndComp
+$Comp
+L C C25
+U 1 1 5715BDBB
+P 5150 2050
+F 0 "C25" H 5175 2150 50  0000 L CNN
+F 1 "0.1uF" H 5175 1950 50  0000 L CNN
+F 2 "Capacitors_SMD:C_0603" H 5188 1900 50  0001 C CNN
+F 3 "" H 5150 2050 50  0000 C CNN
+F 4 "Murata" H 5150 2050 60  0001 C CNN "Manufacturer"
+F 5 "GRM188R61C104KA01" H 5150 2050 60  0001 C CNN "Manufacturer Part Number"
+	1    5150 2050
+	1    0    0    -1
+$EndComp
+$Comp
+L R R?
+U 1 1 57145DF4
+P 7300 2400
+F 0 "R?" V 7250 2200 50  0000 C CNN
+F 1 "68" V 7300 2400 50  0000 C CNN
+F 2 "Resistors_SMD:R_0603" V 7230 2400 50  0001 C CNN
+F 3 "" H 7300 2400 50  0000 C CNN
+F 4 "Panasonic" V 7300 2400 60  0001 C CNN "Manufacturer"
+F 5 "ERJ-3EKF68R0V" V 7300 2400 60  0001 C CNN "Manufacturer Part Number"
+	1    7300 2400
+	0    1    1    0
+$EndComp
+$Comp
+L R R?
+U 1 1 57145E79
+P 7300 2500
+F 0 "R?" V 7250 2300 50  0000 C CNN
+F 1 "68" V 7300 2500 50  0000 C CNN
+F 2 "Resistors_SMD:R_0603" V 7230 2500 50  0001 C CNN
+F 3 "" H 7300 2500 50  0000 C CNN
+F 4 "Panasonic" V 7300 2500 60  0001 C CNN "Manufacturer"
+F 5 "ERJ-3EKF68R0V" V 7300 2500 60  0001 C CNN "Manufacturer Part Number"
+	1    7300 2500
+	0    1    1    0
+$EndComp
+$Comp
+L R R?
+U 1 1 57145EFD
+P 7300 2700
+F 0 "R?" V 7250 2500 50  0000 C CNN
+F 1 "68" V 7300 2700 50  0000 C CNN
+F 2 "Resistors_SMD:R_0603" V 7230 2700 50  0001 C CNN
+F 3 "" H 7300 2700 50  0000 C CNN
+F 4 "Panasonic" V 7300 2700 60  0001 C CNN "Manufacturer"
+F 5 "ERJ-3EKF68R0V" V 7300 2700 60  0001 C CNN "Manufacturer Part Number"
+	1    7300 2700
+	0    1    1    0
+$EndComp
+$Comp
+L R R?
+U 1 1 571476DF
+P 4650 3300
+F 0 "R?" V 4730 3300 50  0000 C CNN
+F 1 "27" V 4650 3300 50  0000 C CNN
+F 2 "Resistors_SMD:R_0603" V 4580 3300 50  0001 C CNN
+F 3 "" H 4650 3300 50  0000 C CNN
+F 4 "Panasonic" V 4650 3300 60  0001 C CNN "Manufacturer"
+F 5 "ERJ-3EKF27R0V" V 4650 3300 60  0001 C CNN "Manufacturer Part Number"
+	1    4650 3300
+	0    1    1    0
+$EndComp
+$Comp
+L R R?
+U 1 1 571495CF
+P 3850 4050
+F 0 "R?" V 3950 4100 50  0000 C CNN
+F 1 "10K" V 3850 4050 50  0000 C CNN
+F 2 "Resistors_SMD:R_0603" V 3780 4050 50  0001 C CNN
+F 3 "" H 3850 4050 50  0000 C CNN
+F 4 "Panasonic" V 3850 4050 60  0001 C CNN "Manufacturer"
+F 5 "ERJ-3GEYJ103V" V 3850 4050 60  0001 C CNN "Manufacturer Part Number"
+	1    3850 4050
+	-1   0    0    1
+$EndComp
+$Comp
+L R R?
+U 1 1 5714C2A1
+P 4650 5650
+F 0 "R?" V 4750 5700 50  0000 C CNN
+F 1 "10K" V 4650 5650 50  0000 C CNN
+F 2 "Resistors_SMD:R_0603" V 4580 5650 50  0001 C CNN
+F 3 "" H 4650 5650 50  0000 C CNN
+F 4 "Panasonic" V 4650 5650 60  0001 C CNN "Manufacturer"
+F 5 "ERJ-3GEYJ103V" V 4650 5650 60  0001 C CNN "Manufacturer Part Number"
+	1    4650 5650
+	-1   0    0    1
+$EndComp
 $EndSCHEMATC
