File: pcb/ft2232d.sch (KiCad schematic (older format))
At the start: 26 parts, among them U4 93CxxA, U5 FT2232D, X1 6MHz

Commit message: Added more BOM info
Parts:
- removed X1: 6MHz, symbol CRYSTAL_SMD
- added X1: 6MHz, headphones:CSCTR_G, symbol CRYSTAL_CSCTR_G
- R31: footprint (none) -> Resistors_SMD:R_0603; Manufacturer (none) -> Panasonic; Manufacturer Part Number (none) -> ERJ-3EKF2201V
- R33: footprint (none) -> Resistors_SMD:R_0603; Manufacturer (none) -> Panasonic; Manufacturer Part Number (none) -> ERJ-3EKF30R0V
- R40, R41: footprint (none) -> Resistors_SMD:R_0603; Manufacturer (none) -> Panasonic; Manufacturer Part Number (none) -> ERJ-3EKF2200V
- U4: footprint (none) -> Housings_SOIC:SOIC-8_3.9x4.9mm_Pitch1.27mm; Manufacturer (none) -> Microchip; Manufacturer Part Number (none) -> 93C46A-I/SN
- U5: footprint (none) -> Housings_QFP:LQFP-48_7x7mm_Pitch0.5mm; Manufacturer (none) -> FTDI; Manufacturer Part Number (none) -> FT2232D
- gave numbers to parts that had none: 6
Connections:
- wire segments 75 -> 76

Commit message: Started filling out FPGA sheet BOM
Parts:
- D1: footprint (none) -> LEDs:LED_0603; Manufacturer (none) -> Lite-On; Manufacturer Part Number (none) -> LTST-C191KRKT
- D2: footprint (none) -> LEDs:LED_0603; Manufacturer (none) -> Lite-On; Manufacturer Part Number (none) -> LTST-C191KGKT
Other:
- note added: "Green"
- note added: "Red"
Changed lines of the file:
@@
 Connection ~ 4950 4400
 $Comp
-L GND #PWR34
+L GND #PWR031
 U 1 1 56A42CE2
 P 4400 4300
-F 0 "#PWR34" H 4400 4050 50  0001 C CNN
+F 0 "#PWR031" H 4400 4050 50  0001 C CNN
 F 1 "GND" H 4400 4150 50  0000 C CNN
 F 2 "" H 4400 4300 50  0000 C CNN
@@
 NoConn ~ 4450 5650
 $Comp
-L GND #PWR32
+L GND #PWR032
 U 1 1 56A43CD0
 P 3800 5700
-F 0 "#PWR32" H 3800 5450 50  0001 C CNN
+F 0 "#PWR032" H 3800 5450 50  0001 C CNN
 F 1 "GND" H 3800 5550 50  0000 C CNN
 F 2 "" H 3800 5700 50  0000 C CNN
@@
 $EndComp
 $Comp
-L GND #PWR37
+L GND #PWR033
 U 1 1 56A43CF4
 P 5100 5200
-F 0 "#PWR37" H 5100 4950 50  0001 C CNN
+F 0 "#PWR033" H 5100 4950 50  0001 C CNN
 F 1 "GND" H 5100 5050 50  0000 C CNN
 F 2 "" H 5100 5200 50  0000 C CNN
@@
 $EndComp
 $Comp
-L GND #PWR43
+L GND #PWR034
 U 1 1 56A43D18
 P 6050 5800
-F 0 "#PWR43" H 6050 5550 50  0001 C CNN
+F 0 "#PWR034" H 6050 5550 50  0001 C CNN
 F 1 "GND" H 6050 5650 50  0000 C CNN
 F 2 "" H 6050 5800 50  0000 C CNN
@@
 $EndComp
 $Comp
-L GND #PWR35
+L GND #PWR035
 U 1 1 56A45799
 P 4850 2750
-F 0 "#PWR35" H 4850 2500 50  0001 C CNN
+F 0 "#PWR035" H 4850 2500 50  0001 C CNN
 F 1 "GND" H 4850 2600 50  0000 C CNN
 F 2 "" H 4850 2750 50  0000 C CNN
@@
 F 0 "D1" H 7700 4900 50  0000 C CNN
 F 1 "RX" H 7700 4700 50  0000 C CNN
-F 2 "" H 7700 4800 50  0000 C CNN
+F 2 "LEDs:LED_0603" H 7700 4800 50  0001 C CNN
 F 3 "" H 7700 4800 50  0000 C CNN
+F 4 "Lite-On" H 7700 4800 60  0001 C CNN "Manufacturer"
+F 5 "LTST-C191KRKT" H 7700 4800 60  0001 C CNN "Manufacturer Part Number"
 	1    7700 4800
 	0    -1   -1   0
@@
 F 0 "D2" H 8000 4900 50  0000 C CNN
 F 1 "TX" H 8000 4700 50  0000 C CNN
-F 2 "" H 8000 4800 50  0000 C CNN
+F 2 "LEDs:LED_0603" H 8000 4800 50  0001 C CNN
 F 3 "" H 8000 4800 50  0000 C CNN
+F 4 "Lite-On" H 8000 4800 60  0001 C CNN "Manufacturer"
+F 5 "LTST-C191KGKT" H 8000 4800 60  0001 C CNN "Manufacturer Part Number"
 	1    8000 4800
 	0    -1   -1   0
@@
 	8000 5100 8000 5000
 $Comp
-L +3.3V #PWR44
+L +3.3V #PWR036
 U 1 1 56A48B0E
 P 6400 1200
-F 0 "#PWR44" H 6400 1050 50  0001 C CNN
+F 0 "#PWR036" H 6400 1050 50  0001 C CNN
 F 1 "+3.3V" H 6400 1340 50  0000 C CNN
 F 2 "" H 6400 1200 50  0000 C CNN
@@
 $EndComp
 $Comp
-L +3.3V #PWR49
+L +3.3V #PWR037
 U 1 1 56A4AC53
 P 8200 5200
-F 0 "#PWR49" H 8200 5050 50  0001 C CNN
+F 0 "#PWR037" H 8200 5050 50  0001 C CNN
 F 1 "+3.3V" H 8200 5340 50  0000 C CNN
 F 2 "" H 8200 5200 50  0000 C CNN
@@
 	7000 5200 8200 5200
 $Comp
-L +3.3V #PWR47
+L +3.3V #PWR038
 U 1 1 56A4B585
 P 7700 4600
-F 0 "#PWR47" H 7700 4450 50  0001 C CNN
+F 0 "#PWR038" H 7700 4450 50  0001 C CNN
 F 1 "+3.3V" H 7700 4740 50  0000 C CNN
 F 2 "" H 7700 4600 50  0000 C CNN
@@
 $EndComp
 $Comp
-L +3.3V #PWR48
+L +3.3V #PWR039
 U 1 1 56A4B6FF
 P 8000 4600
-F 0 "#PWR48" H 8000 4450 50  0001 C CNN
+F 0 "#PWR039" H 8000 4450 50  0001 C CNN
 F 1 "+3.3V" H 8000 4740 50  0000 C CNN
 F 2 "" H 8000 4600 50  0000 C CNN
@@
 $EndComp
 $Comp
-L +3.3V #PWR46
+L +3.3V #PWR040
 U 1 1 56A4C262
 P 7200 3700
-F 0 "#PWR46" H 7200 3550 50  0001 C CNN
+F 0 "#PWR040" H 7200 3550 50  0001 C CNN
 F 1 "+3.3V" H 7200 3840 50  0000 C CNN
 F 2 "" H 7200 3700 50  0000 C CNN
@@
 $EndComp
 $Comp
-L GND #PWR39
+L GND #PWR041
 U 1 1 56A4C939
 P 5150 2200
-F 0 "#PWR39" H 5150 1950 50  0001 C CNN
+F 0 "#PWR041" H 5150 1950 50  0001 C CNN
 F 1 "GND" H 5150 2050 50  0000 C CNN
 F 2 "" H 5150 2200 50  0000 C CNN
@@
 Connection ~ 3850 3800
 $Comp
-L GND #PWR33
+L GND #PWR042
 U 1 1 56A50E44
 P 3850 4200
-F 0 "#PWR33" H 3850 3950 50  0001 C CNN
+F 0 "#PWR042" H 3850 3950 50  0001 C CNN
 F 1 "GND" H 3850 4050 50  0000 C CNN
 F 2 "" H 3850 4200 50  0000 C CNN
@@
 $EndComp
 $Comp
-L +5V #PWR42
+L +5V #PWR043
 U 1 1 56A51073
 P 6050 1200
-F 0 "#PWR42" H 6050 1050 50  0001 C CNN
+F 0 "#PWR043" H 6050 1050 50  0001 C CNN
 F 1 "+5V" H 6050 1340 50  0000 C CNN
 F 2 "" H 6050 1200 50  0000 C CNN
@@
 $EndComp
 $Comp
-L +5V #PWR31
+L +5V #PWR044
 U 1 1 56A514D9
 P 3800 5300
-F 0 "#PWR31" H 3800 5150 50  0001 C CNN
+F 0 "#PWR044" H 3800 5150 50  0001 C CNN
 F 1 "+5V" H 3800 5440 50  0000 C CNN
 F 2 "" H 3800 5300 50  0000 C CNN
@@
 $EndComp
 $Comp
-L +5V #PWR36
+L +5V #PWR045
 U 1 1 56A5151B
 P 4850 5650
-F 0 "#PWR36" H 4850 5500 50  0001 C CNN
+F 0 "#PWR045" H 4850 5500 50  0001 C CNN
 F 1 "+5V" H 4850 5790 50  0000 C CNN
 F 2 "" H 4850 5650 50  0000 C CNN
@@
 $EndComp
 $Comp
-L GND #PWR38
+L GND #PWR046
 U 1 1 56A550EE
 P 5150 1600
-F 0 "#PWR38" H 5150 1350 50  0001 C CNN
+F 0 "#PWR046" H 5150 1350 50  0001 C CNN
 F 1 "GND" H 5150 1450 50  0000 C CNN
 F 2 "" H 5150 1600 50  0000 C CNN
@@
 $EndComp
 $Comp
-L GND #PWR40
+L GND #PWR047
 U 1 1 56A55147
 P 5450 1600
-F 0 "#PWR40" H 5450 1350 50  0001 C CNN
+F 0 "#PWR047" H 5450 1350 50  0001 C CNN
 F 1 "GND" H 5450 1450 50  0000 C CNN
 F 2 "" H 5450 1600 50  0000 C CNN
@@
 $EndComp
 $Comp
-L GND #PWR41
+L GND #PWR048
 U 1 1 56A551A0
 P 5750 1600
-F 0 "#PWR41" H 5750 1350 50  0001 C CNN
+F 0 "#PWR048" H 5750 1350 50  0001 C CNN
 F 1 "GND" H 5750 1450 50  0000 C CNN
 F 2 "" H 5750 1600 50  0000 C CNN
@@
 Connection ~ 5750 1250
 $Comp
-L GND #PWR45
+L GND #PWR049
 U 1 1 56A56EFD
 P 6400 1600
-F 0 "#PWR45" H 6400 1350 50  0001 C CNN
+F 0 "#PWR049" H 6400 1350 50  0001 C CNN
 F 1 "GND" H 6400 1450 50  0000 C CNN
 F 2 "" H 6400 1600 50  0000 C CNN
@@
 NoConn ~ 7000 4900
 $Comp
-L PWR_FLAG #FLG1
+L PWR_FLAG #FLG050
 U 1 1 57151F2A
 P 5100 1900
-F 0 "#FLG1" H 5100 1995 50  0001 C CNN
+F 0 "#FLG050" H 5100 1995 50  0001 C CNN
 F 1 "PWR_FLAG" H 5100 2080 50  0000 C CNN
 F 2 "" H 5100 1900 50  0000 C CNN
@@
 	0    1    1    0
 $EndComp
+Text Notes 7900 4350 0    60   ~ 0
+Green
+Text Notes 7650 4350 0    60   ~ 0
+Red
 $EndSCHEMATC
