File: pcb/ft2232d.sch (KiCad schematic (older format))
At the start: 26 parts, among them U4 93CxxA, U5 FT2232D, X1 6MHz

Commit message: Started laying out FPGA
Connections:
- net labels added: USBD+, USBD-
Changed lines of the file:
@@
 L C C23
 U 1 1 56A45754
-P 4850 2600
-F 0 "C23" H 4875 2700 50  0000 L CNN
-F 1 "33nF" H 4875 2500 50  0000 L CNN
-F 2 "Capacitors_SMD:C_0603" H 4888 2450 50  0001 C CNN
-F 3 "" H 4850 2600 50  0000 C CNN
-F 4 "Murata" H 4850 2600 60  0001 C CNN "Manufacturer"
-F 5 "GRM188R71E333KA01" H 4850 2600 60  0001 C CNN "Manufacturer Part Number"
-	1    4850 2600
+P 4850 2550
+F 0 "C23" H 4875 2650 50  0000 L CNN
+F 1 "33nF" H 4875 2450 50  0000 L CNN
+F 2 "Capacitors_SMD:C_0603" H 4888 2400 50  0001 C CNN
+F 3 "" H 4850 2550 50  0000 C CNN
+F 4 "Murata" H 4850 2550 60  0001 C CNN "Manufacturer"
+F 5 "GRM188R71E333KA01" H 4850 2550 60  0001 C CNN "Manufacturer Part Number"
+	1    4850 2550
 	1    0    0    -1
 $EndComp
@@
 L GND #PWR035
 U 1 1 56A45799
-P 4850 2750
-F 0 "#PWR035" H 4850 2500 50  0001 C CNN
-F 1 "GND" H 4850 2600 50  0000 C CNN
-F 2 "" H 4850 2750 50  0000 C CNN
-F 3 "" H 4850 2750 50  0000 C CNN
-	1    4850 2750
-	1    0    0    -1
-$EndComp
-Wire Wire Line
-	4850 2450 5100 2450
-Wire Wire Line
-	5100 2450 5100 2700
+P 4850 2700
+F 0 "#PWR035" H 4850 2450 50  0001 C CNN
+F 1 "GND" H 4850 2550 50  0000 C CNN
+F 2 "" H 4850 2700 50  0000 C CNN
+F 3 "" H 4850 2700 50  0000 C CNN
+	1    4850 2700
+	1    0    0    -1
+$EndComp
+Wire Wire Line
+	4850 2400 5100 2400
+Wire Wire Line
+	5100 2400 5100 2700
 Text HLabel 7700 2400 2    60   Output ~ 0
 TCK
@@
 L R R29
 U 1 1 56A4D226
-P 4650 3000
-F 0 "R29" V 4730 3000 50  0000 C CNN
-F 1 "27" V 4650 3000 50  0000 C CNN
-F 2 "Resistors_SMD:R_0603" V 4580 3000 50  0001 C CNN
-F 3 "" H 4650 3000 50  0000 C CNN
-F 4 "Panasonic" V 4650 3000 60  0001 C CNN "Manufacturer"
-F 5 "ERJ-3EKF27R0V" V 4650 3000 60  0001 C CNN "Manufacturer Part Number"
-	1    4650 3000
-	0    1    1    0
-$EndComp
-Wire Wire Line
-	4400 3300 4500 3300
-Wire Wire Line
-	4800 3300 5100 3300
-Wire Wire Line
-	5100 3000 4800 3000
-Wire Wire Line
-	4400 3000 4500 3000
+P 4550 3000
+F 0 "R29" V 4630 3000 50  0000 C CNN
+F 1 "27" V 4550 3000 50  0000 C CNN
+F 2 "Resistors_SMD:R_0603" V 4480 3000 50  0001 C CNN
+F 3 "" H 4550 3000 50  0000 C CNN
+F 4 "Panasonic" V 4550 3000 60  0001 C CNN "Manufacturer"
+F 5 "ERJ-3EKF27R0V" V 4550 3000 60  0001 C CNN "Manufacturer Part Number"
+	1    4550 3000
+	0    1    1    0
+$EndComp
+Wire Wire Line
+	4300 3300 4400 3300
+Wire Wire Line
+	4700 3300 5100 3300
+Wire Wire Line
+	5100 3000 4700 3000
+Wire Wire Line
+	4300 3000 4400 3000
 Wire Wire Line
 	5650 2050 5850 2050
@@
 	6250 2050 6250 2100
 Connection ~ 6150 2050
-Text HLabel 4400 3300 0    60   BiDi ~ 0
+Text HLabel 4300 3300 0    60   BiDi ~ 0
 D+
-Text HLabel 4400 3000 0    60   BiDi ~ 0
+Text HLabel 4300 3000 0    60   BiDi ~ 0
 D-
 Text HLabel 3850 3300 1    60   UnSpc ~ 0
@@
 L R R30
 U 1 1 571476DF
-P 4650 3300
-F 0 "R30" V 4730 3300 50  0000 C CNN
-F 1 "27" V 4650 3300 50  0000 C CNN
-F 2 "Resistors_SMD:R_0603" V 4580 3300 50  0001 C CNN
-F 3 "" H 4650 3300 50  0000 C CNN
-F 4 "Panasonic" V 4650 3300 60  0001 C CNN "Manufacturer"
-F 5 "ERJ-3EKF27R0V" V 4650 3300 60  0001 C CNN "Manufacturer Part Number"
-	1    4650 3300
+P 4550 3300
+F 0 "R30" V 4630 3300 50  0000 C CNN
+F 1 "27" V 4550 3300 50  0000 C CNN
+F 2 "Resistors_SMD:R_0603" V 4480 3300 50  0001 C CNN
+F 3 "" H 4550 3300 50  0000 C CNN
+F 4 "Panasonic" V 4550 3300 60  0001 C CNN "Manufacturer"
+F 5 "ERJ-3EKF27R0V" V 4550 3300 60  0001 C CNN "Manufacturer Part Number"
+	1    4550 3300
 	0    1    1    0
 $EndComp
@@
 Text Notes 7650 4350 0    60   ~ 0
 Red
+Text Label 4700 3300 0    60   ~ 0
+USBD+
+Text Label 4700 3000 0    60   ~ 0
+USBD-
 $EndSCHEMATC

Commit message: Cleaned up a lot of the FT2232D->FPGA connections
Moved the series termination resistors into the right spots and
cleaned up and aligned all the traces to the FPGA.
Parts:
- removed R38, R39: 68, Resistors_SMD:R_0603, symbol R
Connections:
- wire segments 76 -> 74
Changed lines of the file:
@@
 Connection ~ 4950 4400
 $Comp
-L GND #PWR034
+L GND #PWR37
 U 1 1 56A42CE2
 P 4400 4300
-F 0 "#PWR034" H 4400 4050 50  0001 C CNN
+F 0 "#PWR37" H 4400 4050 50  0001 C CNN
 F 1 "GND" H 4400 4150 50  0000 C CNN
 F 2 "" H 4400 4300 50  0000 C CNN
@@
 NoConn ~ 4450 5650
 $Comp
-L GND #PWR035
+L GND #PWR35
 U 1 1 56A43CD0
 P 3800 5700
-F 0 "#PWR035" H 3800 5450 50  0001 C CNN
+F 0 "#PWR35" H 3800 5450 50  0001 C CNN
 F 1 "GND" H 3800 5550 50  0000 C CNN
 F 2 "" H 3800 5700 50  0000 C CNN
@@
 $EndComp
 $Comp
-L GND #PWR036
+L GND #PWR40
 U 1 1 56A43CF4
 P 5100 5200
-F 0 "#PWR036" H 5100 4950 50  0001 C CNN
+F 0 "#PWR40" H 5100 4950 50  0001 C CNN
 F 1 "GND" H 5100 5050 50  0000 C CNN
 F 2 "" H 5100 5200 50  0000 C CNN
@@
 $EndComp
 $Comp
-L GND #PWR037
+L GND #PWR46
 U 1 1 56A43D18
 P 6050 5800
-F 0 "#PWR037" H 6050 5550 50  0001 C CNN
+F 0 "#PWR46" H 6050 5550 50  0001 C CNN
 F 1 "GND" H 6050 5650 50  0000 C CNN
 F 2 "" H 6050 5800 50  0000 C CNN
@@
 $EndComp
 $Comp
-L GND #PWR038
+L GND #PWR38
 U 1 1 56A45799
 P 4850 2700
-F 0 "#PWR038" H 4850 2450 50  0001 C CNN
+F 0 "#PWR38" H 4850 2450 50  0001 C CNN
 F 1 "GND" H 4850 2550 50  0000 C CNN
 F 2 "" H 4850 2700 50  0000 C CNN
@@
 TMS
 Wire Wire Line
-	7000 2400 7150 2400
-Wire Wire Line
-	7000 2500 7150 2500
-Wire Wire Line
-	7000 2700 7150 2700
-Wire Wire Line
-	7000 2600 7700 2600
-Wire Wire Line
-	7450 2700 7700 2700
-Wire Wire Line
-	7450 2500 7700 2500
-Wire Wire Line
-	7450 2400 7700 2400
+	7000 2400 7700 2400
+Wire Wire Line
+	7000 2500 7700 2500
+Wire Wire Line
+	7000 2700 7700 2700
 Text HLabel 7700 3900 2    60   Output ~ 0
 USB_TXD
@@
 	8000 5100 8000 5000
 $Comp
-L +3.3V #PWR039
+L +3.3V #PWR47
 U 1 1 56A48B0E
 P 6400 1200
-F 0 "#PWR039" H 6400 1050 50  0001 C CNN
+F 0 "#PWR47" H 6400 1050 50  0001 C CNN
 F 1 "+3.3V" H 6400 1340 50  0000 C CNN
 F 2 "" H 6400 1200 50  0000 C CNN
@@
 $EndComp
 $Comp
-L +3.3V #PWR040
+L +3.3V #PWR52
 U 1 1 56A4AC53
 P 8200 5200
-F 0 "#PWR040" H 8200 5050 50  0001 C CNN
+F 0 "#PWR52" H 8200 5050 50  0001 C CNN
 F 1 "+3.3V" H 8200 5340 50  0000 C CNN
 F 2 "" H 8200 5200 50  0000 C CNN
@@
 	7000 5200 8200 5200
 $Comp
-L +3.3V #PWR041
+L +3.3V #PWR50
 U 1 1 56A4B585
 P 7700 4600
-F 0 "#PWR041" H 7700 4450 50  0001 C CNN
+F 0 "#PWR50" H 7700 4450 50  0001 C CNN
 F 1 "+3.3V" H 7700 4740 50  0000 C CNN
 F 2 "" H 7700 4600 50  0000 C CNN
@@
 $EndComp
 $Comp
-L +3.3V #PWR042
+L +3.3V #PWR51
 U 1 1 56A4B6FF
 P 8000 4600
-F 0 "#PWR042" H 8000 4450 50  0001 C CNN
+F 0 "#PWR51" H 8000 4450 50  0001 C CNN
 F 1 "+3.3V" H 8000 4740 50  0000 C CNN
 F 2 "" H 8000 4600 50  0000 C CNN
@@
 $EndComp
 $Comp
-L +3.3V #PWR043
+L +3.3V #PWR49
 U 1 1 56A4C262
 P 7200 3700
-F 0 "#PWR043" H 7200 3550 50  0001 C CNN
+F 0 "#PWR49" H 7200 3550 50  0001 C CNN
 F 1 "+3.3V" H 7200 3840 50  0000 C CNN
 F 2 "" H 7200 3700 50  0000 C CNN
@@
 $EndComp
 $Comp
-L GND #PWR044
+L GND #PWR42
 U 1 1 56A4C939
 P 5150 2200
-F 0 "#PWR044" H 5150 1950 50  0001 C CNN
+F 0 "#PWR42" H 5150 1950 50  0001 C CNN
 F 1 "GND" H 5150 2050 50  0000 C CNN
 F 2 "" H 5150 2200 50  0000 C CNN
@@
 Connection ~ 3850 3800
 $Comp
-L GND #PWR045
+L GND #PWR36
 U 1 1 56A50E44
 P 3850 4200
-F 0 "#PWR045" H 3850 3950 50  0001 C CNN
+F 0 "#PWR36" H 3850 3950 50  0001 C CNN
 F 1 "GND" H 3850 4050 50  0000 C CNN
 F 2 "" H 3850 4200 50  0000 C CNN
@@
 $EndComp
 $Comp
-L +5V #PWR046
+L +5V #PWR45
 U 1 1 56A51073
 P 6050 1200
-F 0 "#PWR046" H 6050 1050 50  0001 C CNN
+F 0 "#PWR45" H 6050 1050 50  0001 C CNN
 F 1 "+5V" H 6050 1340 50  0000 C CNN
 F 2 "" H 6050 1200 50  0000 C CNN
@@
 $EndComp
 $Comp
-L +5V #PWR047
+L +5V #PWR34
 U 1 1 56A514D9
 P 3800 5300
-F 0 "#PWR047" H 3800 5150 50  0001 C CNN
+F 0 "#PWR34" H 3800 5150 50  0001 C CNN
 F 1 "+5V" H 3800 5440 50  0000 C CNN
 F 2 "" H 3800 5300 50  0000 C CNN
@@
 $EndComp
 $Comp
-L +5V #PWR048
+L +5V #PWR39
 U 1 1 56A5151B
 P 4850 5650
-F 0 "#PWR048" H 4850 5500 50  0001 C CNN
+F 0 "#PWR39" H 4850 5500 50  0001 C CNN
 F 1 "+5V" H 4850 5790 50  0000 C CNN
 F 2 "" H 4850 5650 50  0000 C CNN
@@
 $EndComp
 $Comp
-L GND #PWR049
+L GND #PWR41
 U 1 1 56A550EE
 P 5150 1600
-F 0 "#PWR049" H 5150 1350 50  0001 C CNN
+F 0 "#PWR41" H 5150 1350 50  0001 C CNN
 F 1 "GND" H 5150 1450 50  0000 C CNN
 F 2 "" H 5150 1600 50  0000 C CNN
@@
 $EndComp
 $Comp
-L GND #PWR050
+L GND #PWR43
 U 1 1 56A55147
 P 5450 1600
-F 0 "#PWR050" H 5450 1350 50  0001 C CNN
+F 0 "#PWR43" H 5450 1350 50  0001 C CNN
 F 1 "GND" H 5450 1450 50  0000 C CNN
 F 2 "" H 5450 1600 50  0000 C CNN
@@
 $EndComp
 $Comp
-L GND #PWR051
+L GND #PWR44
 U 1 1 56A551A0
 P 5750 1600
-F 0 "#PWR051" H 5750 1350 50  0001 C CNN
+F 0 "#PWR44" H 5750 1350 50  0001 C CNN
 F 1 "GND" H 5750 1450 50  0000 C CNN
 F 2 "" H 5750 1600 50  0000 C CNN
@@
 Connection ~ 5750 1250
 $Comp
-L GND #PWR052
+L GND #PWR48
 U 1 1 56A56EFD
 P 6400 1600
-F 0 "#PWR052" H 6400 1350 50  0001 C CNN
+F 0 "#PWR48" H 6400 1350 50  0001 C CNN
 F 1 "GND" H 6400 1450 50  0000 C CNN
 F 2 "" H 6400 1600 50  0000 C CNN
@@
 NoConn ~ 7000 4900
 $Comp
-L PWR_FLAG #FLG053
+L PWR_FLAG #FLG1
 U 1 1 57151F2A
 P 5100 1900
-F 0 "#FLG053" H 5100 1995 50  0001 C CNN
+F 0 "#FLG1" H 5100 1995 50  0001 C CNN
 F 1 "PWR_FLAG" H 5100 2080 50  0000 C CNN
 F 2 "" H 5100 1900 50  0000 C CNN
@@
 	1    5150 2050
 	1    0    0    -1
-$EndComp
-$Comp
-L R R37
-U 1 1 57145DF4
-P 7300 2400
-F 0 "R37" V 7250 2200 50  0000 C CNN
-F 1 "68" V 7300 2400 50  0000 C CNN
-F 2 "Resistors_SMD:R_0603" V 7230 2400 50  0001 C CNN
-F 3 "" H 7300 2400 50  0000 C CNN
-F 4 "Panasonic" V 7300 2400 60  0001 C CNN "Manufacturer"
-F 5 "ERJ-3EKF68R0V" V 7300 2400 60  0001 C CNN "Manufacturer Part Number"
-	1    7300 2400
-	0    1    1    0
-$EndComp
-$Comp
-L R R38
-U 1 1 57145E79
-P 7300 2500
-F 0 "R38" V 7250 2300 50  0000 C CNN
-F 1 "68" V 7300 2500 50  0000 C CNN
-F 2 "Resistors_SMD:R_0603" V 7230 2500 50  0001 C CNN
-F 3 "" H 7300 2500 50  0000 C CNN
-F 4 "Panasonic" V 7300 2500 60  0001 C CNN "Manufacturer"
-F 5 "ERJ-3EKF68R0V" V 7300 2500 60  0001 C CNN "Manufacturer Part Number"
-	1    7300 2500
-	0    1    1    0
-$EndComp
-$Comp
-L R R39
-U 1 1 57145EFD
-P 7300 2700
-F 0 "R39" V 7250 2500 50  0000 C CNN
-F 1 "68" V 7300 2700 50  0000 C CNN
-F 2 "Resistors_SMD:R_0603" V 7230 2700 50  0001 C CNN
-F 3 "" H 7300 2700 50  0000 C CNN
-F 4 "Panasonic" V 7300 2700 60  0001 C CNN "Manufacturer"
-F 5 "ERJ-3EKF68R0V" V 7300 2700 60  0001 C CNN "Manufacturer Part Number"
-	1    7300 2700
-	0    1    1    0
 $EndComp
 $Comp
@@
 Text Label 4700 3000 0    60   ~ 0
 USBD-
+$Comp
+L R R37
+U 1 1 574CB91C
+P 7300 2600
+F 0 "R37" V 7350 2800 50  0000 C CNN
+F 1 "68" V 7300 2600 50  0000 C CNN
+F 2 "Resistors_SMD:R_0603" V 7230 2600 50  0001 C CNN
+F 3 "" H 7300 2600 50  0000 C CNN
+F 4 "Panasonic" V 7300 2600 60  0001 C CNN "Manufacturer"
+F 5 "ERJ-3EKF68R0V" V 7300 2600 60  0001 C CNN "Manufacturer Part Number"
+	1    7300 2600
+	0    -1   -1   0
+$EndComp
+Wire Wire Line
+	7000 2600 7150 2600
+Wire Wire Line
+	7450 2600 7700 2600
 $EndSCHEMATC

Commit message: Fixing up USB connector
- Had to go back through and re-annotate all the 0603 caps and
  resistors to the hand-solderding versions since those changes didn't
  make it back into the schematics the last time I tried.

- Added a new footprint for the USB connector to connect to all the
  shield pins.
Parts:
- C23, C24, C25, C26, C27, C28: footprint Capacitors_SMD:C_0603 -> Capacitors_SMD:C_0603_HandSoldering
- R27, R28, R29, R30, R31, R32, R33, R34, R35, R36, R37, R40, R41: footprint Resistors_SMD:R_0603 -> Resistors_SMD:R_0603_HandSoldering
Changed lines of the file:
@@
 F 0 "R34" V 5030 3450 50  0000 C CNN
 F 1 "1.5K" V 4950 3450 50  0000 C CNN
-F 2 "Resistors_SMD:R_0603" V 4880 3450 50  0001 C CNN
+F 2 "Resistors_SMD:R_0603_HandSoldering" V 4880 3450 50  0001 C CNN
 F 3 "" H 4950 3450 50  0000 C CNN
 F 4 "Panasonic" V 4950 3450 60  0001 C CNN "Manufacturer"
@@
 F 0 "R35" V 5030 4250 50  0000 C CNN
 F 1 "1M" V 4950 4250 50  0000 C CNN
-F 2 "Resistors_SMD:R_0603" V 4880 4250 50  0001 C CNN
+F 2 "Resistors_SMD:R_0603_HandSoldering" V 4880 4250 50  0001 C CNN
 F 3 "" H 4950 4250 50  0000 C CNN
 F 4 "Panasonic" V 4950 4250 60  0001 C CNN "Manufacturer"
@@
 F 0 "R33" V 4930 4800 50  0000 C CNN
 F 1 "30" V 4850 4800 50  0000 C CNN
-F 2 "Resistors_SMD:R_0603" V 4780 4800 50  0001 C CNN
+F 2 "Resistors_SMD:R_0603_HandSoldering" V 4780 4800 50  0001 C CNN
 F 3 "" H 4850 4800 50  0000 C CNN
 F 4 "Panasonic" V 4850 4800 60  0001 C CNN "Manufacturer"
@@
 F 0 "R31" V 4730 5250 50  0000 C CNN
 F 1 "2.2K" V 4650 5250 50  0000 C CNN
-F 2 "Resistors_SMD:R_0603" V 4580 5250 50  0001 C CNN
+F 2 "Resistors_SMD:R_0603_HandSoldering" V 4580 5250 50  0001 C CNN
 F 3 "" H 4650 5250 50  0000 C CNN
 F 4 "Panasonic" V 4650 5250 60  0001 C CNN "Manufacturer"
@@
 F 0 "C23" H 4875 2650 50  0000 L CNN
 F 1 "33nF" H 4875 2450 50  0000 L CNN
-F 2 "Capacitors_SMD:C_0603" H 4888 2400 50  0001 C CNN
+F 2 "Capacitors_SMD:C_0603_HandSoldering" H 4888 2400 50  0001 C CNN
 F 3 "" H 4850 2550 50  0000 C CNN
 F 4 "Murata" H 4850 2550 60  0001 C CNN "Manufacturer"
@@
 F 0 "R41" V 7300 5300 50  0000 C CNN
 F 1 "220" V 7350 5100 50  0000 C CNN
-F 2 "Resistors_SMD:R_0603" V 7280 5100 50  0001 C CNN
+F 2 "Resistors_SMD:R_0603_HandSoldering" V 7280 5100 50  0001 C CNN
 F 3 "" H 7350 5100 50  0000 C CNN
 F 4 "Panasonic" V 7350 5100 60  0001 C CNN "Manufacturer"
@@
 F 0 "R36" V 5930 1900 50  0000 C CNN
 F 1 "470" V 5850 1900 50  0000 C CNN
-F 2 "Resistors_SMD:R_0603" V 5780 1900 50  0001 C CNN
+F 2 "Resistors_SMD:R_0603_HandSoldering" V 5780 1900 50  0001 C CNN
 F 3 "" H 5850 1900 50  0000 C CNN
 F 4 "Panasonic" V 5850 1900 60  0001 C CNN "Manufacturer"
@@
 F 0 "R29" V 4630 3000 50  0000 C CNN
 F 1 "27" V 4550 3000 50  0000 C CNN
-F 2 "Resistors_SMD:R_0603" V 4480 3000 50  0001 C CNN
+F 2 "Resistors_SMD:R_0603_HandSoldering" V 4480 3000 50  0001 C CNN
 F 3 "" H 4550 3000 50  0000 C CNN
 F 4 "Panasonic" V 4550 3000 60  0001 C CNN "Manufacturer"
@@
 F 0 "R27" V 3930 3550 50  0000 C CNN
 F 1 "4.7K" V 3850 3550 50  0000 C CNN
-F 2 "Resistors_SMD:R_0603" V 3780 3550 50  0001 C CNN
+F 2 "Resistors_SMD:R_0603_HandSoldering" V 3780 3550 50  0001 C CNN
 F 3 "" H 3850 3550 50  0000 C CNN
 F 4 "Panasonic" V 3850 3550 60  0001 C CNN "Manufacturer"
@@
 F 0 "C27" H 5775 1550 50  0000 L CNN
 F 1 "10uF" H 5775 1350 50  0000 L CNN
-F 2 "Capacitors_SMD:C_0603" H 5788 1300 50  0001 C CNN
+F 2 "Capacitors_SMD:C_0603_HandSoldering" H 5788 1300 50  0001 C CNN
 F 3 "" H 5750 1450 50  0000 C CNN
 F 4 "Murata" H 5750 1450 60  0001 C CNN "Manufacturer"
@@
 F 0 "C24" H 5175 1550 50  0000 L CNN
 F 1 "0.1uF" H 5175 1350 50  0000 L CNN
-F 2 "Capacitors_SMD:C_0603" H 5188 1300 50  0001 C CNN
+F 2 "Capacitors_SMD:C_0603_HandSoldering" H 5188 1300 50  0001 C CNN
 F 3 "" H 5150 1450 50  0000 C CNN
 F 4 "Murata" H 5150 1450 60  0001 C CNN "Manufacturer"
@@
 F 0 "C26" H 5475 1550 50  0000 L CNN
 F 1 "0.1uF" H 5475 1350 50  0000 L CNN
-F 2 "Capacitors_SMD:C_0603" H 5488 1300 50  0001 C CNN
+F 2 "Capacitors_SMD:C_0603_HandSoldering" H 5488 1300 50  0001 C CNN
 F 3 "" H 5450 1450 50  0000 C CNN
 F 4 "Murata" H 5450 1450 60  0001 C CNN "Manufacturer"
@@
 F 0 "C28" H 6425 1550 50  0000 L CNN
 F 1 "0.1uF" H 6425 1350 50  0000 L CNN
-F 2 "Capacitors_SMD:C_0603" H 6438 1300 50  0001 C CNN
+F 2 "Capacitors_SMD:C_0603_HandSoldering" H 6438 1300 50  0001 C CNN
 F 3 "" H 6400 1450 50  0000 C CNN
 F 4 "Murata" H 6400 1450 60  0001 C CNN "Manufacturer"
@@
 F 0 "C25" H 5175 2150 50  0000 L CNN
 F 1 "0.1uF" H 5175 1950 50  0000 L CNN
-F 2 "Capacitors_SMD:C_0603" H 5188 1900 50  0001 C CNN
+F 2 "Capacitors_SMD:C_0603_HandSoldering" H 5188 1900 50  0001 C CNN
 F 3 "" H 5150 2050 50  0000 C CNN
 F 4 "Murata" H 5150 2050 60  0001 C CNN "Manufacturer"
@@
 F 0 "R30" V 4630 3300 50  0000 C CNN
 F 1 "27" V 4550 3300 50  0000 C CNN
-F 2 "Resistors_SMD:R_0603" V 4480 3300 50  0001 C CNN
+F 2 "Resistors_SMD:R_0603_HandSoldering" V 4480 3300 50  0001 C CNN
 F 3 "" H 4550 3300 50  0000 C CNN
 F 4 "Panasonic" V 4550 3300 60  0001 C CNN "Manufacturer"
@@
 F 0 "R28" V 3950 4100 50  0000 C CNN
 F 1 "10K" V 3850 4050 50  0000 C CNN
-F 2 "Resistors_SMD:R_0603" V 3780 4050 50  0001 C CNN
+F 2 "Resistors_SMD:R_0603_HandSoldering" V 3780 4050 50  0001 C CNN
 F 3 "" H 3850 4050 50  0000 C CNN
 F 4 "Panasonic" V 3850 4050 60  0001 C CNN "Manufacturer"
@@
 F 0 "R32" V 4750 5700 50  0000 C CNN
 F 1 "10K" V 4650 5650 50  0000 C CNN
-F 2 "Resistors_SMD:R_0603" V 4580 5650 50  0001 C CNN
+F 2 "Resistors_SMD:R_0603_HandSoldering" V 4580 5650 50  0001 C CNN
 F 3 "" H 4650 5650 50  0000 C CNN
 F 4 "Panasonic" V 4650 5650 60  0001 C CNN "Manufacturer"
@@
 F 0 "R40" V 7300 5200 50  0000 C CNN
 F 1 "220" V 7350 5000 50  0000 C CNN
-F 2 "Resistors_SMD:R_0603" V 7280 5000 50  0001 C CNN
+F 2 "Resistors_SMD:R_0603_HandSoldering" V 7280 5000 50  0001 C CNN
 F 3 "" H 7350 5000 50  0000 C CNN
 F 4 "Panasonic" V 7350 5000 60  0001 C CNN "Manufacturer"
@@
 F 0 "R37" V 7350 2800 50  0000 C CNN
 F 1 "68" V 7300 2600 50  0000 C CNN
-F 2 "Resistors_SMD:R_0603" V 7230 2600 50  0001 C CNN
+F 2 "Resistors_SMD:R_0603_HandSoldering" V 7230 2600 50  0001 C CNN
 F 3 "" H 7300 2600 50  0000 C CNN
 F 4 "Panasonic" V 7300 2600 60  0001 C CNN "Manufacturer"
