File: pcb/ft2232d.sch (KiCad schematic (older format))
At the start: 27 parts, among them U4 93CxxA, U5 FT2232D, X1 6MHz

Commit message: More cleanup and switched sense resistors
Increased the resistance of the current sense resistors up to 0.1 ohm.
Parts:
- R110, R111, R129: value 0.01 -> 0.1
Changed lines of the file:
@@
 P 6750 1250
 F 0 "R111" V 6830 1250 50  0000 C CNN
-F 1 "0.01" V 6750 1250 50  0000 C CNN
+F 1 "0.1" V 6750 1250 50  0000 C CNN
 F 2 "Resistors_SMD:R_0603_HandSoldering" V 6680 1250 50  0001 C CNN
 F 3 "" H 6750 1250 50  0000 C CNN
@@
 P 4900 1250
 F 0 "R110" V 4980 1250 50  0000 C CNN
-F 1 "0.01" V 4900 1250 50  0000 C CNN
+F 1 "0.1" V 4900 1250 50  0000 C CNN
 F 2 "Resistors_SMD:R_0603_HandSoldering" V 4830 1250 50  0001 C CNN
 F 3 "" H 4900 1250 50  0000 C CNN
@@
 P 3100 5150
 F 0 "R129" V 3180 5150 50  0000 C CNN
-F 1 "0.01" V 3100 5150 50  0000 C CNN
+F 1 "0.1" V 3100 5150 50  0000 C CNN
 F 2 "Resistors_SMD:R_0603_HandSoldering" V 3030 5150 50  0001 C CNN
 F 3 "" H 3100 5150 50  0000 C CNN

Commit message: Traces on a plane
- Finished placing testpoints and got footprints for them
- Cleaned up the last of the unconnected tracks
- Switched up supply rails for PWRGOOD LEDs
Parts:
- D1, D2: symbol LED -> LED-RESCUE-NYCDB-01
Changed lines of the file:
@@
 EESchema Schematic File Version 2
+LIBS:NYCDB-01-rescue
 LIBS:power
 LIBS:device
@@
 LIBS:valves
 LIBS:my
+LIBS:NYCDB-01-cache
 EELAYER 25 0
 EELAYER END
@@
 $EndComp
 $Comp
-L LED D1
+L LED-RESCUE-NYCDB-01 D1
 U 1 1 56A47794
 P 7700 4800
+AR Path="/56A47794" Ref="D1"  Part="1"
+AR Path="/56A409F6/56A47794" Ref="D1"  Part="1"
 F 0 "D1" H 7700 4900 50  0000 C CNN
 F 1 "RX" H 7700 4700 50  0000 C CNN
@@
 $EndComp
 $Comp
-L LED D2
+L LED-RESCUE-NYCDB-01 D2
 U 1 1 56A477F3
 P 8000 4800
+AR Path="/56A477F3" Ref="D2"  Part="1"
+AR Path="/56A409F6/56A477F3" Ref="D2"  Part="1"
 F 0 "D2" H 8000 4900 50  0000 C CNN
 F 1 "TX" H 8000 4700 50  0000 C CNN
