File: pcb/power_supplies.sch (KiCad schematic (older format))
At the start: 46 parts, among them U6 bq2409x, U7 LTC3521, U8 LT1617

Commit message: Began cleaning up ERC errors
Connections:
- wire segments 110 -> 111

Commit message: Cleaned up power supplies
- Finished the FAULT LED driver
- Annotated the schematics
- Started updating the power consumption spreadsheet
Parts:
- removed D10, D11, D8, D9: MBR0530, symbol D_Schottky
- removed U8: LT1617, symbol LT1617
- added C100, C101, C102, C103, C96, C97, C98, C99: 10uF, symbol C
- added C104, C105, C106, C107: 10uF TANT, symbol C
- added D10, D11, D14, D15, D8: D, symbol D
- added D9: FAULT15V, symbol LED
- added Q1: Q_PNP_BCE, symbol Q_PNP_BCE
- added R94: 422, symbol R
- added R95: 34K, symbol R
- added R96: 165K, symbol R
- added U15: LT1086CT-12, symbol LT1086CT-12
- added U16: LT1086CT-5, symbol LT1086CT-5
- added U17: LT3015ET-12, symbol LT3015ET-12
- added U18: LT3015ET-5, symbol LT3015ET-5
- added U8: LT3579, symbol LT3579
- C37: value 4.7uF -> 10uF
- C38: value 1uF -> 0.1uF
- C39: value 1uF -> 4.7uF
- C40: value 100pF -> 4.7uF
- C41: value 1uF -> 27pF
- C42: value 1uF -> 1nF
- L4: value 10uH -> 4.7uH
- R48, R52, R53: value R -> 294
- R56: value 210K -> 86.6K
- R57: value 24.9K -> 100K
Connections:
- net labels added: +15V, +5VA, -15V, -5VA
- wire segments 111 -> 225
- no-connect marks 0 -> 2

Commit message: Cleaned up ERC
Connections:
- wire segments 225 -> 161

Commit message: Working through the power supplies sheet
Parts:
- C29, C34, C36, C37, C96, C97, C98, C99: footprint (none) -> Capacitors_SMD:C_0603; Manufacturer (none) -> Murata; Manufacturer Part Number (none) -> GRM188R61A106KE69
- C30, C39, C40: footprint (none) -> Capacitors_SMD:C_0603; Manufacturer (none) -> Murata; Manufacturer Part Number (none) -> GRM188R61A475KE15
- C31, C33: footprint (none) -> Capacitors_SMD:C_0603; Manufacturer (none) -> Murata; Manufacturer Part Number (none) -> GRM188R61A105KA61
- C32: footprint (none) -> Capacitors_SMD:C_0603; Manufacturer (none) -> Murata; Manufacturer Part Number (none) -> GQM1885C1H220GB01
- C35: footprint (none) -> Capacitors_SMD:C_0603; Manufacturer (none) -> Murata; Manufacturer Part Number (none) -> GQM1885C1H330GB01
- C38: footprint (none) -> Capacitors_SMD:C_0603; Manufacturer (none) -> Murata; Manufacturer Part Number (none) -> GRM188R61C104KA01
- C41: footprint (none) -> Capacitors_SMD:C_0603; Manufacturer (none) -> Murata; Manufacturer Part Number (none) -> GRM1885C1H270JA01
- C42: footprint (none) -> Capacitors_SMD:C_0603; Manufacturer (none) -> Murata; Manufacturer Part Number (none) -> GRM1885C1E102JA01
- D10, D11, D14, D15, D8: footprint (none) -> headphones:POWERDI_123; Manufacturer (none) -> Diodes Incorporated; Manufacturer Part Number (none) -> SBR2A40P1-7
- D3: footprint (none) -> LEDs:LED_0603; Manufacturer (none) -> Lite-On; Manufacturer Part Number (none) -> LTST-C191KGKT
- D4: footprint (none) -> LEDs:LED_0603; Manufacturer (none) -> Lite-On; Manufacturer Part Number (none) -> LTST-C191KRKT
- L1, L2, L3, L4: footprint (none) -> headphones:IHLP-2525CZ-01; Manufacturer (none) -> Vishay Dale; Manufacturer Part Number (none) -> IHLP2525CZER4R7M01
- R42: value 1M -> 121K; footprint (none) -> Resistors_SMD:R_0603; Manufacturer (none) -> Panasonic; Manufacturer Part Number (none) -> ERJ-3EKF1213V
- R43: value 136K -> 16.5K; footprint (none) -> Resistors_SMD:R_0603; Manufacturer (none) -> Panasonic; Manufacturer Part Number (none) -> ERJ-3EKF1652V
- R44, R45: footprint (none) -> Resistors_SMD:R_0603; Manufacturer (none) -> Panasonic; Manufacturer Part Number (none) -> ERJ-3EKF1001V
- R46, R49: footprint (none) -> Resistors_SMD:R_0603; Manufacturer (none) -> Panasonic; Manufacturer Part Number (none) -> ERJ-3EKF1501V
- R48, R52, R53: footprint (none) -> Resistors_SMD:R_0603; Manufacturer (none) -> Panasonic; Manufacturer Part Number (none) -> ERJ-3EKF2940V
- R50: footprint (none) -> Resistors_SMD:R_0603; Manufacturer (none) -> Panasonic; Manufacturer Part Number (none) -> ERJ-3EKF1023V
- R51, R57: footprint (none) -> Resistors_SMD:R_0603; Manufacturer (none) -> Panasonic; Manufacturer Part Number (none) -> ERJ-3GEYJ104V
- R54: footprint (none) -> Resistors_SMD:R_0603; Manufacturer (none) -> Panasonic; Manufacturer Part Number (none) -> ERJ-3EKF2743V
- R55: footprint (none) -> Resistors_SMD:R_0603; Manufacturer (none) -> Panasonic; Manufacturer Part Number (none) -> ERJ-3EKF6042V
- R56: footprint (none) -> Resistors_SMD:R_0603; Manufacturer (none) -> Panasonic; Manufacturer Part Number (none) -> ERJ-3EKF8662V
- R95: footprint (none) -> Resistors_SMD:R_0603; Manufacturer (none) -> Panasonic; Manufacturer Part Number (none) -> ERJ-3EKF3402V
- R96: footprint (none) -> Resistors_SMD:R_0603; Manufacturer (none) -> Panasonic; Manufacturer Part Number (none) -> ERJ-3EKF1653V
- U6: footprint (none) -> Housings_SSOP:MSOP-10-1EP_3x3mm_Pitch0.5mm; Manufacturer (none) -> Texas Instruments; Manufacturer Part Number (none) -> BQ24092DGQR
- U7: footprint (none) -> Housings_SSOP:TSSOP-20_4.4x6.5mm_Pitch0.65mm; Manufacturer (none) -> Linear Technology; Manufacturer Part Number (none) -> LTC3521IFE
- U8: footprint (none) -> Housings_SSOP:TSSOP-20_4.4x6.5mm_Pitch0.65mm; Manufacturer (none) -> Linear Technology; Manufacturer Part Number (none) -> LT3579EFE#PBF
Other:
- note added: "GREEN"
- note added: "RED"

Commit message: More progress on power supply sheet
Parts:
- removed C100, C101, C102, C103: 10uF, symbol C
- removed C104, C105, C106, C107: 10uF TANT, symbol C
- removed D5: PG1V2, symbol LED
- removed D6: PG3V3, symbol LED
- removed D7: PG5V, symbol LED
- removed D9: FAULT15V, symbol LED
- removed Q1: Q_PNP_BCE, symbol Q_PNP_BCE
- added C? (x4): 10uF, Capacitors_SMD:C_0603, symbol C
- added C? (x4): 10uF TANT, Capacitors_Tantalum_SMD:TantalC_SizeS_EIA-3216, symbol CP
- added D?: PG1V2, LEDs:LED_0603, symbol LED
- added D?: PG3V3, LEDs:LED_0603, symbol LED
- added D?: PG5V0, LEDs:LED_0603, symbol LED
- added D?: FAULT15V, LEDs:LED_0603, symbol LED
- added Q?: Q_PMOS_GSD, TO_SOT_Packages_SMD:SOT-23, symbol Q_PMOS_GSD
- R94: footprint (none) -> Resistors_SMD:R_0603; Manufacturer (none) -> Panasonic; Manufacturer Part Number (none) -> ERJ-3EKF4220V
- U15: footprint (none) -> TO_SOT_Packages_THT:TO-220_Neutral123_Horizontal; Manufacturer (none) -> Linear Technology; Manufacturer Part Number (none) -> LT1086CT-12
- U16: footprint (none) -> TO_SOT_Packages_THT:TO-220_Neutral123_Horizontal; Manufacturer (none) -> Linear Technology; Manufacturer Part Number (none) -> LT1086CT-5
- U17: footprint (none) -> TO_SOT_Packages_THT:Pentawatt_Neutral_Staggered_Verical_TO220-5-T05D
Connections:
- wire segments 161 -> 226

Commit message: Picked a footprint for the inverting LDOs
Parts:
- U17: footprint TO_SOT_Packages_THT:Pentawatt_Neutral_Staggered_Verical_TO220-5-T05D -> headphones:LT3015_DD_PAK; Manufacturer (none) -> Linear Technology; Manufacturer Part Number (none) -> LT3015EQ-12
- U18: footprint (none) -> headphones:LT3015_DD_PAK; Manufacturer (none) -> Linear Technology; Manufacturer Part Number (none) -> LT3015EQ-5
Connections:
- wire segments 226 -> 161
Changed lines of the file:
@@
 	2100 3100 2100 3150
 Wire Wire Line
-	1250 3100 2100 3100
-Wire Wire Line
-	2100 3100 3700 3100
-Wire Wire Line
-	3700 3100 3800 3100
-Wire Wire Line
-	3800 3100 3900 3100
-Wire Wire Line
-	3900 3100 5900 3100
-Wire Wire Line
-	5900 3100 7800 3100
-Wire Wire Line
-	7800 3100 8200 3100
-Wire Wire Line
-	8200 3100 8750 3100
+	1250 3100 8750 3100
 Wire Wire Line
 	3800 3100 3800 3150
@@
 $EndComp
 Wire Wire Line
-	1800 3800 2100 3800
-Wire Wire Line
-	2100 3800 3050 3800
+	1800 3800 3050 3800
 Connection ~ 2100 3800
 Wire Wire Line
-	2100 4150 2100 4200
-Wire Wire Line
-	2100 4200 2100 4250
+	2100 4150 2100 4250
 Wire Wire Line
 	2350 4200 2100 4200
@@
 	2100 3800 2100 3850
 Wire Wire Line
-	1800 3750 1800 3800
-Wire Wire Line
-	1800 3800 1800 3850
+	1800 3750 1800 3850
 Connection ~ 1800 3800
 Wire Wire Line
@@
 $EndComp
 Wire Wire Line
-	5150 3600 6350 3600
-Wire Wire Line
-	6350 3600 6650 3600
-Wire Wire Line
-	6650 3600 7000 3600
-Wire Wire Line
-	7000 3550 7000 3600
-Wire Wire Line
-	7000 3600 7000 3650
+	5150 3600 7000 3600
+Wire Wire Line
+	7000 3550 7000 3650
 Connection ~ 7000 3600
 Wire Wire Line
@@
 	6150 3700 6150 4000
 Wire Wire Line
-	6150 4000 6350 4000
-Wire Wire Line
-	6350 4000 6650 4000
-Wire Wire Line
-	6350 3950 6350 4000
-Wire Wire Line
-	6350 4000 6350 4050
+	6150 4000 6650 4000
+Wire Wire Line
+	6350 3950 6350 4050
 Connection ~ 6350 4000
 Wire Wire Line
@@
 $EndComp
 Wire Wire Line
-	5900 3950 5900 4000
-Wire Wire Line
-	5900 4000 5900 4050
+	5900 3950 5900 4050
 $Comp
 L GND #PWR70
@@
 	4600 3700 6150 3700
 Wire Wire Line
-	5150 4000 5250 4000
-Wire Wire Line
-	5250 4000 5550 4000
-Wire Wire Line
-	5550 4000 5900 4000
+	5150 4000 5900 4000
 Connection ~ 5900 4000
 Wire Wire Line
@@
 	5550 4400 5550 4350
 Wire Wire Line
-	5050 4400 5250 4400
-Wire Wire Line
-	5250 4400 5550 4400
-Wire Wire Line
-	5250 4350 5250 4400
-Wire Wire Line
-	5250 4400 5250 4450
+	5050 4400 5550 4400
+Wire Wire Line
+	5250 4350 5250 4450
 Connection ~ 5250 4400
 Wire Wire Line
@@
 	3750 5050 3750 5100
 Wire Wire Line
-	3750 5100 3800 5100
-Wire Wire Line
-	3800 5100 3850 5100
+	3750 5100 3850 5100
 Wire Wire Line
 	3800 5100 3800 5150
@@
 $EndComp
 Wire Wire Line
-	4950 5500 4950 5650
-Wire Wire Line
-	4950 5650 4950 5700
-Wire Wire Line
-	5250 5500 5250 5600
-Wire Wire Line
-	5250 5600 5250 5700
-Wire Wire Line
-	5550 5500 5550 5550
-Wire Wire Line
-	5550 5550 5550 5700
+	4950 5500 4950 5700
+Wire Wire Line
+	5250 5500 5250 5700
+Wire Wire Line
+	5550 5500 5550 5700
 Wire Wire Line
 	4550 4600 4600 4600
@@
 PWR_SW
 Wire Wire Line
-	1250 6400 2800 6400
-Wire Wire Line
-	2800 6400 8100 6400
-Wire Wire Line
-	2800 4400 2800 4500
-Wire Wire Line
-	2800 4500 2800 4600
-Wire Wire Line
-	2800 4600 2800 6400
+	1250 6400 8100 6400
+Wire Wire Line
+	2800 4400 2800 6400
 Wire Wire Line
 	2800 4400 3050 4400
@@
 $EndComp
 Wire Wire Line
-	1250 1550 2200 1550
-Wire Wire Line
-	2200 1550 3200 1550
+	1250 1550 3200 1550
 Wire Wire Line
 	2200 1550 2200 2050
@@
 	3100 950  3450 950
 Wire Wire Line
-	4400 1550 4500 1550
-Wire Wire Line
-	4500 1550 5400 1550
-Wire Wire Line
-	5400 1550 5650 1550
-Wire Wire Line
-	5650 1550 5900 1550
+	4400 1550 5900 1550
 Wire Wire Line
 	4500 1550 4500 950
@@
 F 0 "U17" H 13600 3250 60  0000 C CNN
 F 1 "LT3015ET-12" H 14050 3250 60  0000 C CNN
-F 2 "TO_SOT_Packages_THT:Pentawatt_Neutral_Staggered_Verical_TO220-5-T05D" H 13900 3250 60  0001 C CNN
+F 2 "headphones:LT3015_DD_PAK" H 13900 3250 60  0001 C CNN
 F 3 "" H 13900 3250 60  0000 C CNN
+F 4 "Linear Technology" H 13900 3200 60  0001 C CNN "Manufacturer"
+F 5 "LT3015EQ-12" H 13900 3200 60  0001 C CNN "Manufacturer Part Number"
 	1    13900 3200
 	1    0    0    -1
@@
 F 0 "U18" H 13600 4300 60  0000 C CNN
 F 1 "LT3015ET-5" H 14050 4300 60  0000 C CNN
-F 2 "" H 13900 4300 60  0000 C CNN
+F 2 "headphones:LT3015_DD_PAK" H 13900 4300 60  0001 C CNN
 F 3 "" H 13900 4300 60  0000 C CNN
+F 4 "Linear Technology" H 13900 4250 60  0001 C CNN "Manufacturer"
+F 5 "LT3015EQ-5" H 13900 4250 60  0001 C CNN "Manufacturer Part Number"
 	1    13900 4250
 	1    0    0    -1
@@
 	13450 1200 13250 1200
 Wire Wire Line
-	13250 1150 13250 1200
-Wire Wire Line
-	13250 1200 13250 1250
+	13250 1150 13250 1250
 Connection ~ 13250 1200
 Wire Wire Line
 	14350 1200 14700 1200
 Wire Wire Line
-	14700 1150 14700 1200
-Wire Wire Line
-	14700 1200 14700 1250
+	14700 1150 14700 1250
 $Comp
 L GND #PWR104
@@
 $EndComp
 Wire Wire Line
-	13250 2100 13250 2150
-Wire Wire Line
-	13250 2150 13250 2200
+	13250 2100 13250 2200
 Wire Wire Line
 	13250 2150 13450 2150
@@
 	14350 2150 14700 2150
 Wire Wire Line
-	14700 2100 14700 2150
-Wire Wire Line
-	14700 2150 14700 2200
+	14700 2100 14700 2200
 Connection ~ 14700 2150
 $Comp
@@
 $EndComp
 Wire Wire Line
-	13050 3250 13050 3300
-Wire Wire Line
-	13050 3300 13050 3350
-Wire Wire Line
-	13050 3300 13300 3300
-Wire Wire Line
-	13300 3300 13350 3300
+	13050 3250 13050 3350
+Wire Wire Line
+	13050 3300 13350 3300
 Connection ~ 13050 3300
 Wire Wire Line
@@
 Connection ~ 13300 3300
 Wire Wire Line
-	14450 3300 14500 3300
-Wire Wire Line
-	14500 3300 14700 3300
-Wire Wire Line
-	14700 3250 14700 3300
-Wire Wire Line
-	14700 3300 14700 3350
+	14450 3300 14700 3300
+Wire Wire Line
+	14700 3250 14700 3350
 Connection ~ 14700 3300
 Wire Wire Line
@@
 $EndComp
 Wire Wire Line
-	13050 4300 13050 4350
-Wire Wire Line
-	13050 4350 13050 4400
-Wire Wire Line
-	13050 4350 13300 4350
-Wire Wire Line
-	13300 4350 13350 4350
+	13050 4300 13050 4400
+Wire Wire Line
+	13050 4350 13350 4350
 Connection ~ 13050 4350
 Wire Wire Line
@@
 $EndComp
 Wire Wire Line
-	14450 4350 14500 4350
-Wire Wire Line
-	14500 4350 14700 4350
-Wire Wire Line
-	14700 4300 14700 4350
-Wire Wire Line
-	14700 4350 14700 4400
+	14450 4350 14700 4350
+Wire Wire Line
+	14700 4300 14700 4400
 Connection ~ 14700 4350
 Wire Wire Line
@@
 $EndComp
 Wire Wire Line
-	10050 3400 10500 3400
-Wire Wire Line
-	10500 3400 10900 3400
+	10050 3400 10900 3400
 Wire Wire Line
 	10500 3400 10500 3550
@@
 $EndComp
 Wire Wire Line
-	8650 3400 8700 3400
-Wire Wire Line
-	8700 3400 8750 3400
+	8650 3400 8750 3400
 Wire Wire Line
 	8200 3100 8200 3400
@@
 $EndComp
 Wire Wire Line
-	7800 2050 7800 3100
-Wire Wire Line
-	7800 3100 7800 3200
+	7800 2050 7800 3200
 Connection ~ 7800 3100
 $Comp
@@
 	8700 2900 8750 2900
 Wire Wire Line
-	8700 2050 8700 2500
-Wire Wire Line
-	8700 2500 8700 2600
-Wire Wire Line
-	8700 2600 8700 2700
-Wire Wire Line
-	8700 2700 8700 2800
-Wire Wire Line
-	8700 2800 8700 2900
-Wire Wire Line
-	8600 2050 8700 2050
-Wire Wire Line
-	8700 2050 9250 2050
+	8700 2050 8700 2900
+Wire Wire Line
+	8600 2050 9250 2050
 Wire Wire Line
 	8750 2800 8700 2800
@@
 	10100 2900 10050 2900
 Wire Wire Line
-	10100 1200 10100 2050
-Wire Wire Line
-	10100 2050 10100 2500
-Wire Wire Line
-	10100 2500 10100 2600
-Wire Wire Line
-	10100 2600 10100 2700
-Wire Wire Line
-	10100 2700 10100 2800
-Wire Wire Line
-	10100 2800 10100 2900
-Wire Wire Line
-	9550 2050 10100 2050
-Wire Wire Line
-	10100 2050 10300 2050
+	10100 1200 10100 2900
+Wire Wire Line
+	9550 2050 10300 2050
 Wire Wire Line
 	10050 2500 10100 2500
@@
 Connection ~ 10100 2050
 Wire Wire Line
-	10600 1200 10700 1200
-Wire Wire Line
-	10700 1200 10800 1200
+	10600 1200 10800 1200
 Wire Wire Line
 	10700 1300 10700 1200
 Connection ~ 10700 1200
 Wire Wire Line
-	10600 2050 10700 2050
-Wire Wire Line
-	10700 2050 10800 2050
+	10600 2050 10800 2050
 Wire Wire Line
 	10700 2150 10700 2050
@@
 	11250 2550 11250 2050
 Wire Wire Line
-	11100 2050 11250 2050
-Wire Wire Line
-	11250 2050 11550 2050
-Wire Wire Line
-	11550 2050 11900 2050
-Wire Wire Line
-	11900 2000 11900 2050
-Wire Wire Line
-	11900 2050 11900 2100
+	11100 2050 11900 2050
+Wire Wire Line
+	11900 2000 11900 2100
 Connection ~ 11250 2050
 Wire Wire Line
@@
 $EndComp
 Wire Wire Line
-	11100 1200 11250 1200
-Wire Wire Line
-	11250 1200 11550 1200
-Wire Wire Line
-	11550 1200 11900 1200
-Wire Wire Line
-	11900 1150 11900 1200
-Wire Wire Line
-	11900 1200 11900 1250
+	11100 1200 11900 1200
+Wire Wire Line
+	11900 1150 11900 1250
 Wire Wire Line
 	11550 1250 11550 1200

Commit message: Finished up BOM for power supplies
Parts:
- removed U17: LT3015ET-12, headphones:LT3015_DD_PAK, symbol LT3015ET-12
- removed U18: LT3015ET-5, headphones:LT3015_DD_PAK, symbol LT3015ET-5
- added R100: 107K, Resistors_SMD:R_0603, symbol R
- added R101, R103: 12.1K, Resistors_SMD:R_0603, symbol R
- added R102: 37.4K, Resistors_SMD:R_0603, symbol R
- added U17, U18: LT3015ET-ADJ, TO_SOT_Packages_THT:Pentawatt_Neutral_Staggered-Typ1_Horizontal_TO220-5-TA05B, symbol LT3015ET-ADJ
- R47: value R -> 10K; footprint (none) -> Resistors_SMD:R_0603; Manufacturer (none) -> Panasonic; Manufacturer Part Number (none) -> ERJ-3GEYJ103V
- gave numbers to parts that had none: 13
Connections:
- wire segments 161 -> 167
