File: pcb/power_supplies.sch (KiCad schematic (older format))
At the start: 72 parts, among them Q1 Q_PMOS_GSD, U15 LT1086CT-12, U16 LT1086CT-5, U17 LT3015ET-ADJ, U18 LT3015ET-ADJ, U6 bq2409x, U7 LTC3521, U8 LT3579

Commit message: Began layout on board
Parts:
- U8: footprint Housings_SSOP:TSSOP-20_4.4x6.5mm_Pitch0.65mm -> headphones:TSSOP-20_4.4x6.5mm_Pitch0.65mm_Pad
Changed lines of the file:
@@
 F 0 "U8" H 9000 2450 60  0000 C CNN
 F 1 "LT3579" H 9700 2450 60  0000 C CNN
-F 2 "Housings_SSOP:TSSOP-20_4.4x6.5mm_Pitch0.65mm" H 10050 1800 60  0001 C CNN
+F 2 "headphones:TSSOP-20_4.4x6.5mm_Pitch0.65mm_Pad" H 10050 1800 60  0001 C CNN
 F 3 "" H 10050 1800 60  0000 C CNN
 F 4 "Linear Technology" H 9400 2400 60  0001 C CNN "Manufacturer"

Commit message: Laid out most of the power supplies
Parts:
- added C108, C109: 4.7uF, Capacitors_SMD:C_0603, symbol C
Connections:
- wire segments 167 -> 169
Changed lines of the file:
@@
 L +5V #PWR052
 U 1 1 56A76440
-P 1800 3750
-F 0 "#PWR052" H 1800 3600 50  0001 C CNN
-F 1 "+5V" H 1800 3890 50  0000 C CNN
-F 2 "" H 1800 3750 50  0000 C CNN
-F 3 "" H 1800 3750 50  0000 C CNN
-	1    1800 3750
-	1    0    0    -1
-$EndComp
-Wire Wire Line
-	1800 3800 3050 3800
+P 1250 3750
+F 0 "#PWR052" H 1250 3600 50  0001 C CNN
+F 1 "+5V" H 1250 3890 50  0000 C CNN
+F 2 "" H 1250 3750 50  0000 C CNN
+F 3 "" H 1250 3750 50  0000 C CNN
+	1    1250 3750
+	1    0    0    -1
+$EndComp
+Wire Wire Line
+	1250 3800 3050 3800
 Connection ~ 2100 3800
 Wire Wire Line
@@
 L GND #PWR053
 U 1 1 56A7651D
-P 1800 4150
-F 0 "#PWR053" H 1800 3900 50  0001 C CNN
-F 1 "GND" H 1800 4000 50  0000 C CNN
-F 2 "" H 1800 4150 50  0000 C CNN
-F 3 "" H 1800 4150 50  0000 C CNN
-	1    1800 4150
+P 1250 4150
+F 0 "#PWR053" H 1250 3900 50  0001 C CNN
+F 1 "GND" H 1250 4000 50  0000 C CNN
+F 2 "" H 1250 4150 50  0000 C CNN
+F 3 "" H 1250 4150 50  0000 C CNN
+	1    1250 4150
 	1    0    0    -1
 $EndComp
@@
 	2100 3800 2100 3850
 Wire Wire Line
-	1800 3750 1800 3850
-Connection ~ 1800 3800
+	1250 3750 1250 3850
+Connection ~ 1250 3800
 Wire Wire Line
 	4550 3600 4650 3600
@@
 $EndComp
 $Comp
-L -15V #PWR90
+L -15V #PWR92
 U 1 1 57085091
 P 13050 3250
-F 0 "#PWR90" H 13050 3350 50  0001 C CNN
+F 0 "#PWR92" H 13050 3350 50  0001 C CNN
 F 1 "-15V" H 13050 3400 50  0000 C CNN
 F 2 "" H 13050 3250 50  0000 C CNN
@@
 $EndComp
 $Comp
-L -15V #PWR92
+L -15V #PWR94
 U 1 1 570850F5
 P 13050 4650
-F 0 "#PWR92" H 13050 4750 50  0001 C CNN
+F 0 "#PWR94" H 13050 4750 50  0001 C CNN
 F 1 "-15V" H 13050 4800 50  0000 C CNN
 F 2 "" H 13050 4650 50  0000 C CNN
@@
 $EndComp
 $Comp
-L -15V #PWR86
+L -15V #PWR88
 U 1 1 570A676D
 P 11900 1150
-F 0 "#PWR86" H 11900 1250 50  0001 C CNN
+F 0 "#PWR88" H 11900 1250 50  0001 C CNN
 F 1 "-15V" H 11900 1300 50  0000 C CNN
 F 2 "" H 11900 1150 50  0000 C CNN
@@
 $EndComp
 $Comp
-L -5VA #PWR111
+L -5VA #PWR113
 U 1 1 5715CB67
 P 15050 4650
-F 0 "#PWR111" H 15050 4750 50  0001 C CNN
+F 0 "#PWR113" H 15050 4750 50  0001 C CNN
 F 1 "-5VA" H 15050 4800 50  0000 C CNN
 F 2 "" H 15050 4650 50  0000 C CNN
@@
 L C C29
 U 1 1 572262C0
-P 1800 4000
-F 0 "C29" H 1825 4100 50  0000 L CNN
-F 1 "10uF" H 1825 3900 50  0000 L CNN
-F 2 "Capacitors_SMD:C_0603" H 1838 3850 50  0001 C CNN
-F 3 "" H 1800 4000 50  0000 C CNN
-F 4 "Murata" H 1800 4000 60  0001 C CNN "Manufacturer"
-F 5 "GRM188R61A106KE69" H 1800 4000 60  0001 C CNN "Manufacturer Part Number"
-	1    1800 4000
+P 1250 4000
+F 0 "C29" H 1275 4100 50  0000 L CNN
+F 1 "10uF" H 1275 3900 50  0000 L CNN
+F 2 "Capacitors_SMD:C_0603" H 1288 3850 50  0001 C CNN
+F 3 "" H 1250 4000 50  0000 C CNN
+F 4 "Murata" H 1250 4000 60  0001 C CNN "Manufacturer"
+F 5 "GRM188R61A106KE69" H 1250 4000 60  0001 C CNN "Manufacturer Part Number"
+	1    1250 4000
 	1    0    0    -1
 $EndComp
@@
 	-1   0    0    1
 $EndComp
+$Comp
+L GND #PWR0115
+U 1 1 5738267C
+P 1450 3450
+F 0 "#PWR0115" H 1450 3200 50  0001 C CNN
+F 1 "GND" H 1450 3300 50  0000 C CNN
+F 2 "" H 1450 3450 50  0000 C CNN
+F 3 "" H 1450 3450 50  0000 C CNN
+	1    1450 3450
+	1    0    0    -1
+$EndComp
+$Comp
+L C C108
+U 1 1 57382684
+P 1450 3300
+F 0 "C108" H 1475 3400 50  0000 L CNN
+F 1 "4.7uF" H 1475 3200 50  0000 L CNN
+F 2 "Capacitors_SMD:C_0603" H 1488 3150 50  0001 C CNN
+F 3 "" H 1450 3300 50  0000 C CNN
+F 4 "Murata" H 1450 3300 60  0001 C CNN "Manufacturer"
+F 5 "GRM188R61A475KE15" H 1450 3300 60  0001 C CNN "Manufacturer Part Number"
+	1    1450 3300
+	1    0    0    -1
+$EndComp
+$Comp
+L GND #PWR0116
+U 1 1 573828CB
+P 1800 3450
+F 0 "#PWR0116" H 1800 3200 50  0001 C CNN
+F 1 "GND" H 1800 3300 50  0000 C CNN
+F 2 "" H 1800 3450 50  0000 C CNN
+F 3 "" H 1800 3450 50  0000 C CNN
+	1    1800 3450
+	1    0    0    -1
+$EndComp
+$Comp
+L C C109
+U 1 1 573828D3
+P 1800 3300
+F 0 "C109" H 1825 3400 50  0000 L CNN
+F 1 "4.7uF" H 1825 3200 50  0000 L CNN
+F 2 "Capacitors_SMD:C_0603" H 1838 3150 50  0001 C CNN
+F 3 "" H 1800 3300 50  0000 C CNN
+F 4 "Murata" H 1800 3300 60  0001 C CNN "Manufacturer"
+F 5 "GRM188R61A475KE15" H 1800 3300 60  0001 C CNN "Manufacturer Part Number"
+	1    1800 3300
+	1    0    0    -1
+$EndComp
+Wire Wire Line
+	1450 3150 1450 3100
+Connection ~ 1450 3100
+Wire Wire Line
+	1800 3150 1800 3100
+Connection ~ 1800 3100
 $EndSCHEMATC

Commit message: Fixing up USB connector
- Had to go back through and re-annotate all the 0603 caps and
  resistors to the hand-solderding versions since those changes didn't
  make it back into the schematics the last time I tried.

- Added a new footprint for the USB connector to connect to all the
  shield pins.
Parts:
- C100, C101, C102, C103, C108, C109, C29, C30, C31, C32, C33, C34, C35, C36, C37, C38, C39, C40, C41, C42, C96, C97, C98, C99: footprint Capacitors_SMD:C_0603 -> Capacitors_SMD:C_0603_HandSoldering
- R100, R101, R102, R103, R42, R43, R44, R45, R46, R47, R48, R49, R50, R51, R52, R53, R54, R55, R56, R57, R94, R95, R96: footprint Resistors_SMD:R_0603 -> Resistors_SMD:R_0603_HandSoldering

Commit message: Cleanup and added testpoints
Cleaned up some of the schematic layout without changing any nets.  Also
added testpoints to all the power rails for easy debug.
Parts:
- added W1, W10, W11, W2, W3, W4, W5, W6, W7, W8, W9: TEST_1P, symbol TEST_1P
Other:
- note added: "TODO: Check forward voltages of these LEDs"
