File: pcb/power_supplies.sch (KiCad schematic (older format))
At the start: 85 parts, among them Q1 Q_PMOS_GSD, U15 LT1086CT-12, U16 LT1086CT-5, U17 LT3015ET-ADJ, U18 LT3015ET-ADJ, U6 bq2409x, U7 LTC3521, U8 LT3579

Commit message: Ran DRC and added some more notes
Other:
- note added: "TODO: Model this in spice"

Commit message: Traces on a plane
- Finished placing testpoints and got footprints for them
- Cleaned up the last of the unconnected tracks
- Switched up supply rails for PWRGOOD LEDs
Parts:
- D3, D4, D5, D6, D7, D9: symbol LED -> LED-RESCUE-NYCDB-01
- W1, W10, W11, W2, W3, W4, W5, W6, W7, W8, W9: footprint (none) -> Measurement_Points:Measurement_Point_Square-TH_Small
Connections:
- wire segments 169 -> 172
Changed lines of the file:
@@
 EESchema Schematic File Version 2
+LIBS:NYCDB-01-rescue
 LIBS:power
 LIBS:device
@@
 LIBS:valves
 LIBS:my
+LIBS:NYCDB-01-cache
 EELAYER 25 0
 EELAYER END
@@
 $EndComp
 $Comp
-L LED D3
+L LED-RESCUE-NYCDB-01 D3
 U 1 1 57201246
 P 3850 2800
+AR Path="/57201246" Ref="D3"  Part="1"
+AR Path="/56A7553B/57201246" Ref="D3"  Part="1"
 F 0 "D3" H 3850 2900 50  0000 C CNN
 F 1 "PG" H 3850 2700 50  0000 C CNN
@@
 GREEN
 $Comp
-L LED D4
+L LED-RESCUE-NYCDB-01 D4
 U 1 1 57203029
 P 5000 3600
+AR Path="/57203029" Ref="D4"  Part="1"
+AR Path="/56A7553B/57203029" Ref="D4"  Part="1"
 F 0 "D4" H 5000 3700 50  0000 C CNN
 F 1 "CHG" H 5000 3500 50  0000 C CNN
@@
 $EndComp
 $Comp
-L LED D5
+L LED-RESCUE-NYCDB-01 D5
 U 1 1 5722895E
 P 5150 7750
+AR Path="/5722895E" Ref="D5"  Part="1"
+AR Path="/56A7553B/5722895E" Ref="D5"  Part="1"
 F 0 "D5" H 5150 7850 50  0000 C CNN
 F 1 "PG1V2" H 5150 7650 50  0000 C CNN
@@
 $EndComp
 $Comp
-L LED D6
+L LED-RESCUE-NYCDB-01 D6
 U 1 1 5722A76B
 P 5450 7750
+AR Path="/5722A76B" Ref="D6"  Part="1"
+AR Path="/56A7553B/5722A76B" Ref="D6"  Part="1"
 F 0 "D6" H 5450 7850 50  0000 C CNN
 F 1 "PG3V3" H 5450 7650 50  0000 C CNN
@@
 $EndComp
 $Comp
-L LED D7
+L LED-RESCUE-NYCDB-01 D7
 U 1 1 5722AA5D
 P 5750 7750
+AR Path="/5722AA5D" Ref="D7"  Part="1"
+AR Path="/56A7553B/5722AA5D" Ref="D7"  Part="1"
 F 0 "D7" H 5750 7850 50  0000 C CNN
 F 1 "PG5V0" H 5750 7650 50  0000 C CNN
@@
 $EndComp
 $Comp
-L LED D9
+L LED-RESCUE-NYCDB-01 D9
 U 1 1 57235B19
 P 9600 6950
+AR Path="/57235B19" Ref="D9"  Part="1"
+AR Path="/56A7553B/57235B19" Ref="D9"  Part="1"
 F 0 "D9" H 9600 7050 50  0000 C CNN
 F 1 "FAULT15V" H 9600 6850 50  0000 C CNN
@@
 F 0 "W3" H 6900 3120 50  0000 C CNN
 F 1 "TEST_1P" H 6900 3050 50  0001 C CNN
-F 2 "" H 7100 2850 50  0000 C CNN
+F 2 "Measurement_Points:Measurement_Point_Square-TH_Small" H 7100 2850 50  0001 C CNN
 F 3 "" H 7100 2850 50  0000 C CNN
 	1    6900 2850
@@
 F 0 "W4" H 7200 3120 50  0000 C CNN
 F 1 "TEST_1P" H 7200 3050 50  0001 C CNN
-F 2 "" H 7400 2850 50  0000 C CNN
+F 2 "Measurement_Points:Measurement_Point_Square-TH_Small" H 7400 2850 50  0001 C CNN
 F 3 "" H 7400 2850 50  0000 C CNN
 	1    7200 2850
@@
 F 0 "W5" H 7500 3120 50  0000 C CNN
 F 1 "TEST_1P" H 7500 3050 50  0001 C CNN
-F 2 "" H 7700 2850 50  0000 C CNN
+F 2 "Measurement_Points:Measurement_Point_Square-TH_Small" H 7700 2850 50  0001 C CNN
 F 3 "" H 7700 2850 50  0000 C CNN
 	1    7500 2850
@@
 F 0 "W6" H 7800 3120 50  0000 C CNN
 F 1 "TEST_1P" H 7800 3050 50  0001 C CNN
-F 2 "" H 8000 2850 50  0000 C CNN
+F 2 "Measurement_Points:Measurement_Point_Square-TH_Small" H 8000 2850 50  0001 C CNN
 F 3 "" H 8000 2850 50  0000 C CNN
 	1    7800 2850
@@
 F 0 "W7" H 8100 3120 50  0000 C CNN
 F 1 "TEST_1P" H 8100 3050 50  0001 C CNN
-F 2 "" H 8300 2850 50  0000 C CNN
+F 2 "Measurement_Points:Measurement_Point_Square-TH_Small" H 8300 2850 50  0001 C CNN
 F 3 "" H 8300 2850 50  0000 C CNN
 	1    8100 2850
@@
 F 0 "W8" H 8400 3120 50  0000 C CNN
 F 1 "TEST_1P" H 8400 3050 50  0001 C CNN
-F 2 "" H 8600 2850 50  0000 C CNN
+F 2 "Measurement_Points:Measurement_Point_Square-TH_Small" H 8600 2850 50  0001 C CNN
 F 3 "" H 8600 2850 50  0000 C CNN
 	1    8400 2850
@@
 F 0 "W9" H 8700 3120 50  0000 C CNN
 F 1 "TEST_1P" H 8700 3050 50  0001 C CNN
-F 2 "" H 8900 2850 50  0000 C CNN
+F 2 "Measurement_Points:Measurement_Point_Square-TH_Small" H 8900 2850 50  0001 C CNN
 F 3 "" H 8900 2850 50  0000 C CNN
 	1    8700 2850
@@
 F 0 "W10" H 9000 3120 50  0000 C CNN
 F 1 "TEST_1P" H 9000 3050 50  0001 C CNN
-F 2 "" H 9200 2850 50  0000 C CNN
+F 2 "Measurement_Points:Measurement_Point_Square-TH_Small" H 9200 2850 50  0001 C CNN
 F 3 "" H 9200 2850 50  0000 C CNN
 	1    9000 2850
@@
 F 0 "W11" H 9300 3120 50  0000 C CNN
 F 1 "TEST_1P" H 9300 3050 50  0001 C CNN
-F 2 "" H 9500 2850 50  0000 C CNN
+F 2 "Measurement_Points:Measurement_Point_Square-TH_Small" H 9500 2850 50  0001 C CNN
 F 3 "" H 9500 2850 50  0000 C CNN
 	1    9300 2850
@@
 F 0 "W2" H 1550 5220 50  0000 C CNN
 F 1 "TEST_1P" H 1550 5150 50  0000 C CNN
-F 2 "" H 1750 4950 50  0000 C CNN
+F 2 "Measurement_Points:Measurement_Point_Square-TH_Small" H 1750 4950 50  0001 C CNN
 F 3 "" H 1750 4950 50  0000 C CNN
 	1    1550 4950
@@
 F 0 "W1" H 1550 3670 50  0000 C CNN
 F 1 "TEST_1P" H 1550 3600 50  0000 C CNN
-F 2 "" H 1750 3400 50  0000 C CNN
+F 2 "Measurement_Points:Measurement_Point_Square-TH_Small" H 1750 3400 50  0001 C CNN
 F 3 "" H 1750 3400 50  0000 C CNN
 	1    1550 3400
@@
 Text Notes 9950 6900 0    60   ~ 0
 TODO: Model this in spice
+$Comp
+L GND #PWR0138
+U 1 1 589E8BBB
+P 4350 4200
+F 0 "#PWR0138" H 4350 3950 50  0001 C CNN
+F 1 "GND" H 4350 4050 50  0000 C CNN
+F 2 "" H 4350 4200 50  0000 C CNN
+F 3 "" H 4350 4200 50  0000 C CNN
+	1    4350 4200
+	1    0    0    -1
+$EndComp
+Wire Wire Line
+	4600 3900 4600 4050
+Wire Wire Line
+	4600 4050 4350 4050
+Wire Wire Line
+	4350 4050 4350 4200
 $EndSCHEMATC
