File: pcb/usb_conn.sch (KiCad schematic (older format))
At the start: 8 parts, among them P2 USB_OTG

Commit message: Began cleaning up ERC errors
Other:
- note added: "TODO: ESD protection and ferrite beads on power and ground"
Changed lines of the file:
@@
 $Descr A4 11693 8268
 encoding utf-8
-Sheet 11 9
+Sheet 7 9
 Title "USB Connector and Filtering"
 Date ""
@@
 NoConn ~ 4900 3700
 $Comp
-L GND #PWR101
+L GND #PWR083
 U 1 1 56A8D0DA
 P 5050 3600
-F 0 "#PWR101" H 5050 3350 50  0001 C CNN
+F 0 "#PWR083" H 5050 3350 50  0001 C CNN
 F 1 "GND" H 5050 3450 50  0000 C CNN
 F 2 "" H 5050 3600 50  0000 C CNN
@@
 $EndComp
 $Comp
-L GND #PWR102
+L GND #PWR084
 U 1 1 56A8D148
 P 5050 4350
-F 0 "#PWR102" H 5050 4100 50  0001 C CNN
+F 0 "#PWR084" H 5050 4100 50  0001 C CNN
 F 1 "GND" H 5050 4200 50  0000 C CNN
 F 2 "" H 5050 4350 50  0000 C CNN
@@
 Connection ~ 6150 4000
 $Comp
-L GND #PWR103
+L GND #PWR085
 U 1 1 56A8D2E5
 P 6150 4350
-F 0 "#PWR103" H 6150 4100 50  0001 C CNN
+F 0 "#PWR085" H 6150 4100 50  0001 C CNN
 F 1 "GND" H 6150 4200 50  0000 C CNN
 F 2 "" H 6150 4350 50  0000 C CNN
@@
 $EndComp
 $Comp
-L GND #PWR104
+L GND #PWR086
 U 1 1 56A8D302
 P 6550 4350
-F 0 "#PWR104" H 6550 4100 50  0001 C CNN
+F 0 "#PWR086" H 6550 4100 50  0001 C CNN
 F 1 "GND" H 6550 4200 50  0000 C CNN
 F 2 "" H 6550 4350 50  0000 C CNN
@@
 Wire Wire Line
 	5750 3900 6800 3900
-$Comp
-L PWR_FLAG #FLG20
-U 1 1 56A8EAF8
-P 5050 3350
-F 0 "#FLG20" H 5050 3445 50  0001 C CNN
-F 1 "PWR_FLAG" H 5050 3530 50  0000 C CNN
-F 2 "" H 5050 3350 50  0000 C CNN
-F 3 "" H 5050 3350 50  0000 C CNN
-	1    5050 3350
-	1    0    0    -1
-$EndComp
-Connection ~ 5050 3350
+Text Notes 5300 3450 0    60   ~ 0
+TODO: ESD protection and ferrite beads on power and ground
 $EndSCHEMATC

Commit message: Cleaned up ERC
Changed lines of the file:
@@
 NoConn ~ 4900 3700
 $Comp
-L GND #PWR110
+L GND #PWR0113
 U 1 1 56A8D0DA
 P 5050 3600
-F 0 "#PWR110" H 5050 3350 50  0001 C CNN
+F 0 "#PWR0113" H 5050 3350 50  0001 C CNN
 F 1 "GND" H 5050 3450 50  0000 C CNN
 F 2 "" H 5050 3600 50  0000 C CNN
@@
 $EndComp
 $Comp
-L GND #PWR111
+L GND #PWR0114
 U 1 1 56A8D148
 P 5050 4350
-F 0 "#PWR111" H 5050 4100 50  0001 C CNN
+F 0 "#PWR0114" H 5050 4100 50  0001 C CNN
 F 1 "GND" H 5050 4200 50  0000 C CNN
 F 2 "" H 5050 4350 50  0000 C CNN
@@
 $EndComp
 Wire Wire Line
-	5700 4000 6800 4000
+	5700 4000 7250 4000
 Wire Wire Line
 	6150 4000 6150 4050
@@
 Connection ~ 6150 4000
 $Comp
-L GND #PWR112
+L GND #PWR0115
 U 1 1 56A8D2E5
 P 6150 4350
-F 0 "#PWR112" H 6150 4100 50  0001 C CNN
+F 0 "#PWR0115" H 6150 4100 50  0001 C CNN
 F 1 "GND" H 6150 4200 50  0000 C CNN
 F 2 "" H 6150 4350 50  0000 C CNN
@@
 $EndComp
 $Comp
-L GND #PWR113
+L GND #PWR0116
 U 1 1 56A8D302
 P 6550 4350
-F 0 "#PWR113" H 6550 4100 50  0001 C CNN
+F 0 "#PWR0116" H 6550 4100 50  0001 C CNN
 F 1 "GND" H 6550 4200 50  0000 C CNN
 F 2 "" H 6550 4350 50  0000 C CNN
@@
 	1    0    0    -1
 $EndComp
-Text HLabel 6800 4000 2    60   UnSpc ~ 0
+Text HLabel 7250 4000 2    60   UnSpc ~ 0
 USB5V
 Connection ~ 6550 4000
@@
 Text Notes 5300 3450 0    60   ~ 0
 TODO: ESD protection and ferrite beads on power and ground
+$Comp
+L PWR_FLAG #FLG0117
+U 1 1 571455C7
+P 7000 4000
+F 0 "#FLG0117" H 7000 4095 50  0001 C CNN
+F 1 "PWR_FLAG" H 7000 4180 50  0000 C CNN
+F 2 "" H 7000 4000 50  0000 C CNN
+F 3 "" H 7000 4000 50  0000 C CNN
+	1    7000 4000
+	-1   0    0    1
+$EndComp
+Connection ~ 7000 4000
 $EndSCHEMATC

Commit message: Tweaked USB connector schematic
Parts:
- removed L5: 600@100MHz, symbol L_Small
- added C108: C, symbol C
- added D16, D17, D18: TVS, symbol TVS
Connections:
- net labels added: GNDPWR
- wire segments 14 -> 34
Other:
- note removed: "TODO: ESD protection and ferrite beads on power and ground"

Commit message: Swapped DNS cap for 0-ohm resistor
Parts:
- removed C108: C, symbol C
- added R104: 0, Resistors_SMD:R_0603, symbol R
Changed lines of the file:
@@
 	1    0    0    -1
-$EndComp
-$Comp
-L C C108
-U 1 1 5728E974
-P 4500 4350
-F 0 "C108" H 4525 4450 50  0000 L CNN
-F 1 "C" H 4525 4250 50  0000 L CNN
-F 2 "" H 4538 4200 50  0000 C CNN
-F 3 "" H 4500 4350 50  0000 C CNN
-	1    4500 4350
-	0    1    1    0
 $EndComp
 Wire Wire Line
@@
 	4350 4350 4300 4350
 Connection ~ 4300 4350
+$Comp
+L R R104
+U 1 1 57291A33
+P 4500 4350
+F 0 "R104" V 4580 4350 50  0000 C CNN
+F 1 "0" V 4500 4350 50  0000 C CNN
+F 2 "Resistors_SMD:R_0603" V 4430 4350 50  0001 C CNN
+F 3 "" H 4500 4350 50  0000 C CNN
+F 4 "Panasonic" V 4500 4350 60  0001 C CNN "Manufacturer"
+F 5 "ERJ-3GEY0R00V" V 4500 4350 60  0001 C CNN "Manufacturer Part Number"
+	1    4500 4350
+	0    1    1    0
+$EndComp
 $EndSCHEMATC

Commit message: Finished first pass at BOM
Parts:
- C43: footprint (none) -> Capacitors_SMD:C_0603; Manufacturer (none) -> Murata; Manufacturer Part Number (none) -> GRM188R71E103KA01
- C44: footprint (none) -> Capacitors_SMD:C_0603; Manufacturer (none) -> Murata; Manufacturer Part Number (none) -> GRM188R61C104KA01
- C45: footprint (none) -> Capacitors_ThroughHole:C_Radial_D10_L21_P5; Manufacturer (none) -> Panasonic; Manufacturer Part Number (none) -> ECA-2WHG4R7
- D16, D17, D18: value TVS -> SMAJ5.0CA; footprint (none) -> Diodes_SMD:SMA_Standard; Manufacturer (none) -> Littelfuse; Manufacturer Part Number (none) -> SMAJ5.0CA
- FB1: renamed from L6; footprint (none) -> Resistors_SMD:R_0603; Manufacturer (none) -> Taiyo Yuden; Manufacturer Part Number (none) -> BKP1608HS330-T
- P2: footprint (none) -> headphones:SJ110578; Manufacturer (none) -> JAE Electronics; Manufacturer Part Number (none) -> DX4R005JJ2R1800
- R58, R59: footprint (none) -> Resistors_SMD:R_0603; Manufacturer (none) -> Panasonic; Manufacturer Part Number (none) -> ERJ-3EKF27R0V
Connections:
- wire segments 34 -> 22
Changed lines of the file:
@@
 F 0 "P2" H 4725 3675 50  0000 C CNN
 F 1 "USB_OTG" H 4400 4000 50  0000 C CNN
-F 2 "" V 4350 3700 50  0000 C CNN
+F 2 "headphones:SJ110578" V 4350 3700 50  0001 C CNN
 F 3 "" V 4350 3700 50  0000 C CNN
+F 4 "JAE Electronics" H 4400 3800 60  0001 C CNN "Manufacturer"
+F 5 "DX4R005JJ2R1800" H 4400 3800 60  0001 C CNN "Manufacturer Part Number"
 	1    4400 3800
 	0    -1   1    0
@@
 NoConn ~ 4700 3900
 $Comp
-L GND #PWR114
+L GND #PWR0115
 U 1 1 56A8D0DA
 P 4750 4400
-F 0 "#PWR114" H 4750 4150 50  0001 C CNN
+F 0 "#PWR0115" H 4750 4150 50  0001 C CNN
 F 1 "GND" H 4750 4250 50  0000 C CNN
 F 2 "" H 4750 4400 50  0000 C CNN
@@
 $EndComp
 $Comp
-L C C43
-U 1 1 56A8D101
-P 5300 3200
-F 0 "C43" H 5325 3300 50  0000 L CNN
-F 1 "0.01uF" H 5325 3100 50  0000 L CNN
-F 2 "" H 5338 3050 50  0000 C CNN
-F 3 "" H 5300 3200 50  0000 C CNN
-	1    5300 3200
-	1    0    0    -1
-$EndComp
-$Comp
-L GND #PWR115
+L GND #PWR0116
 U 1 1 56A8D148
 P 5300 3350
-F 0 "#PWR115" H 5300 3100 50  0001 C CNN
+F 0 "#PWR0116" H 5300 3100 50  0001 C CNN
 F 1 "GND" H 5300 3200 50  0000 C CNN
 F 2 "" H 5300 3350 50  0000 C CNN
@@
 $EndComp
 $Comp
-L L_Small L6
+L L_Small FB1
 U 1 1 56A8D181
 P 5850 3000
-F 0 "L6" V 5900 3200 50  0000 L CNN
+F 0 "FB1" V 5900 3200 50  0000 L CNN
 F 1 "BKP1608HS330-T" V 5800 2650 50  0000 L CNN
-F 2 "" H 5850 3000 50  0000 C CNN
+F 2 "Resistors_SMD:R_0603" H 5850 3000 50  0001 C CNN
 F 3 "" H 5850 3000 50  0000 C CNN
+F 4 "Taiyo Yuden" V 5850 3000 60  0001 C CNN "Manufacturer"
+F 5 "BKP1608HS330-T" V 5850 3000 60  0001 C CNN "Manufacturer Part Number"
 	1    5850 3000
 	0    -1   -1   0
-$EndComp
-$Comp
-L C C44
-U 1 1 56A8D248
-P 6400 3200
-F 0 "C44" H 6425 3300 50  0000 L CNN
-F 1 "0.1uF" H 6425 3100 50  0000 L CNN
-F 2 "" H 6438 3050 50  0000 C CNN
-F 3 "" H 6400 3200 50  0000 C CNN
-	1    6400 3200
-	1    0    0    -1
 $EndComp
 $Comp
@@
 F 0 "C45" H 6825 3300 50  0000 L CNN
 F 1 "4.7uF" H 6825 3100 50  0000 L CNN
-F 2 "" H 6838 3050 50  0000 C CNN
+F 2 "Capacitors_ThroughHole:C_Radial_D10_L21_P5" H 6838 3050 50  0001 C CNN
 F 3 "" H 6800 3200 50  0000 C CNN
+F 4 "Panasonic" H 6800 3200 60  0001 C CNN "Manufacturer"
+F 5 " ECA-2WHG4R7" H 6800 3200 60  0001 C CNN "Manufacturer Part Number"
 	1    6800 3200
 	1    0    0    -1
 $EndComp
 $Comp
-L GND #PWR116
+L GND #PWR0117
 U 1 1 56A8D2E5
 P 6400 3350
-F 0 "#PWR116" H 6400 3100 50  0001 C CNN
+F 0 "#PWR0117" H 6400 3100 50  0001 C CNN
 F 1 "GND" H 6400 3200 50  0000 C CNN
 F 2 "" H 6400 3350 50  0000 C CNN
@@
 $EndComp
 $Comp
-L GND #PWR117
+L GND #PWR0118
 U 1 1 56A8D302
 P 6800 3350
-F 0 "#PWR117" H 6800 3100 50  0001 C CNN
+F 0 "#PWR0118" H 6800 3100 50  0001 C CNN
 F 1 "GND" H 6800 3200 50  0000 C CNN
 F 2 "" H 6800 3350 50  0000 C CNN
@@
 F 0 "R58" V 6550 3950 50  0000 C CNN
 F 1 "27" V 6500 3700 50  0000 C CNN
-F 2 "" V 6430 3700 50  0000 C CNN
+F 2 "Resistors_SMD:R_0603" V 6430 3700 50  0001 C CNN
 F 3 "" H 6500 3700 50  0000 C CNN
+F 4 "Panasonic" V 6500 3700 60  0001 C CNN "Manufacturer"
+F 5 "ERJ-3EKF27R0V" V 6500 3700 60  0001 C CNN "Manufacturer Part Number"
 	1    6500 3700
 	0    -1   -1   0
 $EndComp
 $Comp
-L R R59
-U 1 1 56A8E5DD
-P 6500 3800
-F 0 "R59" V 6550 4050 50  0000 C CNN
-F 1 "27" V 6500 3800 50  0000 C CNN
-F 2 "" V 6430 3800 50  0000 C CNN
-F 3 "" H 6500 3800 50  0000 C CNN
-	1    6500 3800
-	0    -1   -1   0
-$EndComp
-$Comp
-L PWR_FLAG #FLG7
+L PWR_FLAG #FLG0119
 U 1 1 571455C7
 P 7250 3000
-F 0 "#FLG7" H 7250 3095 50  0001 C CNN
+F 0 "#FLG0119" H 7250 3095 50  0001 C CNN
 F 1 "PWR_FLAG" H 7250 3180 50  0000 C CNN
 F 2 "" H 7250 3000 50  0000 C CNN
@@
 P 5100 4400
 F 0 "D16" H 5100 4550 50  0000 C CNN
-F 1 "TVS" H 5100 4250 50  0000 C CNN
-F 2 "" H 5100 4400 50  0000 C CNN
+F 1 "SMAJ5.0CA" H 5100 4250 50  0000 C CNN
+F 2 "Diodes_SMD:SMA_Standard" H 5100 4400 50  0001 C CNN
 F 3 "" H 5100 4400 50  0000 C CNN
+F 4 "Littelfuse" H 5100 4400 60  0001 C CNN "Manufacturer"
+F 5 "SMAJ5.0CA" H 5100 4400 60  0001 C CNN "Manufacturer Part Number"
 	1    5100 4400
 	0    1    1    0
 $EndComp
 $Comp
-L TVS D17
-U 1 1 57288357
-P 5550 4400
-F 0 "D17" H 5550 4550 50  0000 C CNN
-F 1 "TVS" H 5550 4250 50  0000 C CNN
-F 2 "" H 5550 4400 50  0000 C CNN
-F 3 "" H 5550 4400 50  0000 C CNN
-	1    5550 4400
-	0    1    1    0
-$EndComp
-$Comp
-L TVS D18
-U 1 1 57288397
-P 6000 4400
-F 0 "D18" H 6000 4550 50  0000 C CNN
-F 1 "TVS" H 6000 4250 50  0000 C CNN
-F 2 "" H 6000 4400 50  0000 C CNN
-F 3 "" H 6000 4400 50  0000 C CNN
-	1    6000 4400
-	0    1    1    0
-$EndComp
-$Comp
-L GNDPWR #PWR113
+L GNDPWR #PWR0120
 U 1 1 57288D16
 P 4300 4800
-F 0 "#PWR113" H 4300 4600 50  0001 C CNN
+F 0 "#PWR0120" H 4300 4600 50  0001 C CNN
 F 1 "GNDPWR" H 4300 4670 50  0000 C CNN
 F 2 "" H 4300 4750 50  0000 C CNN
@@
 $EndComp
 Wire Wire Line
-	5100 3000 5300 3000
-Wire Wire Line
-	5300 3000 5750 3000
+	5100 3000 5750 3000
 Wire Wire Line
 	5300 3000 5300 3050
 Connection ~ 5300 3000
 Wire Wire Line
-	5950 3000 6400 3000
-Wire Wire Line
-	6400 3000 6800 3000
-Wire Wire Line
-	6800 3000 7250 3000
-Wire Wire Line
-	7250 3000 7500 3000
+	5950 3000 7500 3000
 Wire Wire Line
 	6400 3000 6400 3050
@@
 Connection ~ 7250 3000
 Wire Wire Line
-	4300 4200 4300 4350
-Wire Wire Line
-	4300 4350 4300 4750
-Wire Wire Line
-	4300 4750 4300 4800
+	4300 4200 4300 4800
 Wire Wire Line
 	6000 4750 6000 4700
 Wire Wire Line
-	4300 4750 5100 4750
-Wire Wire Line
-	5100 4750 5550 4750
-Wire Wire Line
-	5550 4750 6000 4750
+	4300 4750 6000 4750
 Connection ~ 4300 4750
 Wire Wire Line
@@
 	4700 3600 5100 3600
 Wire Wire Line
-	5100 3000 5100 3600
-Wire Wire Line
-	5100 3600 5100 4100
-Wire Wire Line
-	4700 3700 5550 3700
-Wire Wire Line
-	5550 3700 6350 3700
+	5100 3000 5100 4100
+Wire Wire Line
+	4700 3700 6350 3700
 Wire Wire Line
 	5550 3700 5550 4100
 Wire Wire Line
-	4700 3800 6000 3800
-Wire Wire Line
-	6000 3800 6350 3800
+	4700 3800 6350 3800
 Wire Wire Line
 	6000 3800 6000 4100
@@
 	4700 4000 4750 4000
 Wire Wire Line
-	4750 4000 4750 4350
-Wire Wire Line
-	4750 4350 4750 4400
+	4750 4000 4750 4400
 Wire Wire Line
 	4650 4350 4750 4350
@@
 	0    1    1    0
 $EndComp
+$Comp
+L TVS D17
+U 1 1 57281B4A
+P 5550 4400
+F 0 "D17" H 5550 4550 50  0000 C CNN
+F 1 "SMAJ5.0CA" H 5550 4250 50  0000 C CNN
+F 2 "Diodes_SMD:SMA_Standard" H 5550 4400 50  0001 C CNN
+F 3 "" H 5550 4400 50  0000 C CNN
+F 4 "Littelfuse" H 5550 4400 60  0001 C CNN "Manufacturer"
+F 5 "SMAJ5.0CA" H 5550 4400 60  0001 C CNN "Manufacturer Part Number"
+	1    5550 4400
+	0    1    1    0
+$EndComp
+$Comp
+L TVS D18
+U 1 1 57281BA2
+P 6000 4400
+F 0 "D18" H 6000 4550 50  0000 C CNN
+F 1 "SMAJ5.0CA" H 6000 4250 50  0000 C CNN
+F 2 "Diodes_SMD:SMA_Standard" H 6000 4400 50  0001 C CNN
+F 3 "" H 6000 4400 50  0000 C CNN
+F 4 "Littelfuse" H 6000 4400 60  0001 C CNN "Manufacturer"
+F 5 "SMAJ5.0CA" H 6000 4400 60  0001 C CNN "Manufacturer Part Number"
+	1    6000 4400
+	0    1    1    0
+$EndComp
+$Comp
+L C C43
+U 1 1 572BF9A2
+P 5300 3200
+F 0 "C43" H 5325 3300 50  0000 L CNN
+F 1 "0.01uF" H 5325 3100 50  0000 L CNN
+F 2 "Capacitors_SMD:C_0603" H 5338 3050 50  0001 C CNN
+F 3 "" H 5300 3200 50  0000 C CNN
+F 4 "Murata" H 5300 3200 60  0001 C CNN "Manufacturer"
+F 5 "GRM188R71E103KA01" H 5300 3200 60  0001 C CNN "Manufacturer Part Number"
+	1    5300 3200
+	1    0    0    -1
+$EndComp
+$Comp
+L C C44
+U 1 1 572C0A24
+P 6400 3200
+F 0 "C44" H 6425 3300 50  0000 L CNN
+F 1 "0.1uF" H 6425 3100 50  0000 L CNN
+F 2 "Capacitors_SMD:C_0603" H 6438 3050 50  0001 C CNN
+F 3 "" H 6400 3200 50  0000 C CNN
+F 4 "Murata" H 6400 3200 60  0001 C CNN "Manufacturer"
+F 5 "GRM188R61C104KA01" H 6400 3200 60  0001 C CNN "Manufacturer Part Number"
+	1    6400 3200
+	1    0    0    -1
+$EndComp
+$Comp
+L R R59
+U 1 1 572C16A2
+P 6500 3800
+F 0 "R59" V 6550 4050 50  0000 C CNN
+F 1 "27" V 6500 3800 50  0000 C CNN
+F 2 "Resistors_SMD:R_0603" V 6430 3800 50  0001 C CNN
+F 3 "" H 6500 3800 50  0000 C CNN
+F 4 "Panasonic" V 6500 3800 60  0001 C CNN "Manufacturer"
+F 5 "ERJ-3EKF27R0V" V 6500 3800 60  0001 C CNN "Manufacturer Part Number"
+	1    6500 3800
+	0    -1   -1   0
+$EndComp
 $EndSCHEMATC
