File: pcb/usb_conn.sch (KiCad schematic (older format))
At the start: 11 parts, among them P2 USB_OTG

Commit message: Worked on USB connection
Connections:
- net labels added: CON_D+, CON_D-
Changed lines of the file:
@@
 $EndComp
 Connection ~ 4750 4750
+Text Label 5150 3700 0    60   ~ 0
+CON_D-
+Text Label 5150 3800 0    60   ~ 0
+CON_D+
 $EndSCHEMATC

Commit message: Worked on the USB connection
Parts:
- removed D17, D18: SMAJ5.0CA, Diodes_SMD:SMA_Standard, symbol TVS
- added D17: TVS_SOT23, TO_SOT_Packages_SMD:SOT-23, symbol TVS_SOT23
- added F1: 1206L150, Resistors_SMD:R_1206_HandSoldering, symbol F_Small
- D16: value SMAJ5.0CA -> V5.5MLA0603H; footprint Diodes_SMD:SMA_Standard -> Resistors_SMD:R_0603_HandSoldering; Manufacturer Part Number SMAJ5.0CA -> V5.5MLA0603H
Changed lines of the file:
@@
 L USB_OTG P2
 U 1 1 56A8D0CF
-P 4400 3800
-F 0 "P2" H 4725 3675 50  0000 C CNN
-F 1 "USB_OTG" H 4400 4000 50  0000 C CNN
-F 2 "headphones:SJ110578" V 4350 3700 50  0001 C CNN
-F 3 "" V 4350 3700 50  0000 C CNN
-F 4 "JAE Electronics" H 4400 3800 60  0001 C CNN "Manufacturer"
-F 5 "DX4R005JJ2R1800" H 4400 3800 60  0001 C CNN "Manufacturer Part Number"
-	1    4400 3800
+P 4300 3800
+F 0 "P2" H 4625 3675 50  0000 C CNN
+F 1 "USB_OTG" H 4300 4000 50  0000 C CNN
+F 2 "headphones:SJ110578" V 4250 3700 50  0001 C CNN
+F 3 "" V 4250 3700 50  0000 C CNN
+F 4 "JAE Electronics" H 4300 3800 60  0001 C CNN "Manufacturer"
+F 5 "DX4R005JJ2R1800" H 4300 3800 60  0001 C CNN "Manufacturer Part Number"
+	1    4300 3800
 	0    -1   1    0
 $EndComp
-NoConn ~ 4700 3900
+NoConn ~ 4600 3900
 $Comp
 L GND #PWR0117
 U 1 1 56A8D0DA
-P 4750 4400
-F 0 "#PWR0117" H 4750 4150 50  0001 C CNN
-F 1 "GND" H 4750 4250 50  0000 C CNN
-F 2 "" H 4750 4400 50  0000 C CNN
-F 3 "" H 4750 4400 50  0000 C CNN
-	1    4750 4400
+P 4650 4400
+F 0 "#PWR0117" H 4650 4150 50  0001 C CNN
+F 1 "GND" H 4650 4250 50  0000 C CNN
+F 2 "" H 4650 4400 50  0000 C CNN
+F 3 "" H 4650 4400 50  0000 C CNN
+	1    4650 4400
 	1    0    0    -1
 $EndComp
@@
 F 5 "BKP1608HS330-T" V 5850 3000 60  0001 C CNN "Manufacturer Part Number"
 	1    5850 3000
-	0    -1   -1   0
+	0    1    -1   0
 $EndComp
 $Comp
@@
 P 5100 4400
 F 0 "D16" H 5100 4550 50  0000 C CNN
-F 1 "SMAJ5.0CA" H 5100 4250 50  0000 C CNN
-F 2 "Diodes_SMD:SMA_Standard" H 5100 4400 50  0001 C CNN
+F 1 "V5.5MLA0603H" H 5100 4250 50  0000 C CNN
+F 2 "Resistors_SMD:R_0603_HandSoldering" H 5100 4400 50  0001 C CNN
 F 3 "" H 5100 4400 50  0000 C CNN
 F 4 "Littelfuse" H 5100 4400 60  0001 C CNN "Manufacturer"
-F 5 "SMAJ5.0CA" H 5100 4400 60  0001 C CNN "Manufacturer Part Number"
+F 5 "V5.5MLA0603H" H 5100 4400 60  0001 C CNN "Manufacturer Part Number"
 	1    5100 4400
-	0    1    1    0
+	0    -1   -1   0
 $EndComp
 $Comp
 L GNDPWR #PWR0122
 U 1 1 57288D16
-P 4300 4800
-F 0 "#PWR0122" H 4300 4600 50  0001 C CNN
-F 1 "GNDPWR" H 4300 4670 50  0000 C CNN
-F 2 "" H 4300 4750 50  0000 C CNN
-F 3 "" H 4300 4750 50  0000 C CNN
-	1    4300 4800
+P 4200 4800
+F 0 "#PWR0122" H 4200 4600 50  0001 C CNN
+F 1 "GNDPWR" H 4200 4670 50  0000 C CNN
+F 2 "" H 4200 4750 50  0000 C CNN
+F 3 "" H 4200 4750 50  0000 C CNN
+	1    4200 4800
 	1    0    0    -1
 $EndComp
@@
 Connection ~ 7250 3000
 Wire Wire Line
-	4300 4200 4300 4800
-Wire Wire Line
-	6000 4750 6000 4700
-Wire Wire Line
-	4300 4750 6000 4750
-Connection ~ 4300 4750
+	4200 4200 4200 4800
+Wire Wire Line
+	4200 4750 5900 4750
+Connection ~ 4200 4750
 Wire Wire Line
 	5100 4700 5100 4750
 Connection ~ 5100 4750
 Wire Wire Line
-	5550 4700 5550 4750
-Connection ~ 5550 4750
-Wire Wire Line
-	4700 3600 5100 3600
-Wire Wire Line
 	5100 3000 5100 4100
 Wire Wire Line
-	4700 3700 6350 3700
-Wire Wire Line
-	5550 3700 5550 4100
-Wire Wire Line
-	4700 3800 6350 3800
+	4600 3700 6350 3700
+Wire Wire Line
+	5800 3700 5800 4100
+Wire Wire Line
+	4600 3800 6350 3800
 Wire Wire Line
 	6000 3800 6000 4100
-Connection ~ 5550 3700
+Connection ~ 5800 3700
 Connection ~ 6000 3800
 Connection ~ 5100 3600
 Wire Wire Line
-	4700 4000 4750 4000
-Wire Wire Line
-	4750 4000 4750 4400
-Wire Wire Line
-	4650 4350 4750 4350
-Connection ~ 4750 4350
-Wire Wire Line
-	4350 4350 4300 4350
-Connection ~ 4300 4350
+	4600 4000 4650 4000
+Wire Wire Line
+	4650 4000 4650 4400
+Wire Wire Line
+	4550 4350 4650 4350
+Connection ~ 4650 4350
+Wire Wire Line
+	4250 4350 4200 4350
+Connection ~ 4200 4350
 $Comp
 L R R104
 U 1 1 57291A33
-P 4500 4350
-F 0 "R104" V 4580 4350 50  0000 C CNN
-F 1 "0" V 4500 4350 50  0000 C CNN
-F 2 "Resistors_SMD:R_0603" V 4430 4350 50  0001 C CNN
-F 3 "" H 4500 4350 50  0000 C CNN
-F 4 "Panasonic" V 4500 4350 60  0001 C CNN "Manufacturer"
-F 5 "ERJ-3GEY0R00V" V 4500 4350 60  0001 C CNN "Manufacturer Part Number"
-	1    4500 4350
-	0    1    1    0
-$EndComp
-$Comp
-L TVS D17
-U 1 1 57281B4A
-P 5550 4400
-F 0 "D17" H 5550 4550 50  0000 C CNN
-F 1 "SMAJ5.0CA" H 5550 4250 50  0000 C CNN
-F 2 "Diodes_SMD:SMA_Standard" H 5550 4400 50  0001 C CNN
-F 3 "" H 5550 4400 50  0000 C CNN
-F 4 "Littelfuse" H 5550 4400 60  0001 C CNN "Manufacturer"
-F 5 "SMAJ5.0CA" H 5550 4400 60  0001 C CNN "Manufacturer Part Number"
-	1    5550 4400
-	0    1    1    0
-$EndComp
-$Comp
-L TVS D18
-U 1 1 57281BA2
-P 6000 4400
-F 0 "D18" H 6000 4550 50  0000 C CNN
-F 1 "SMAJ5.0CA" H 6000 4250 50  0000 C CNN
-F 2 "Diodes_SMD:SMA_Standard" H 6000 4400 50  0001 C CNN
-F 3 "" H 6000 4400 50  0000 C CNN
-F 4 "Littelfuse" H 6000 4400 60  0001 C CNN "Manufacturer"
-F 5 "SMAJ5.0CA" H 6000 4400 60  0001 C CNN "Manufacturer Part Number"
-	1    6000 4400
+P 4400 4350
+F 0 "R104" V 4480 4350 50  0000 C CNN
+F 1 "0" V 4400 4350 50  0000 C CNN
+F 2 "Resistors_SMD:R_0603" V 4330 4350 50  0001 C CNN
+F 3 "" H 4400 4350 50  0000 C CNN
+F 4 "Panasonic" V 4400 4350 60  0001 C CNN "Manufacturer"
+F 5 "ERJ-3GEY0R00V" V 4400 4350 60  0001 C CNN "Manufacturer Part Number"
+	1    4400 4350
 	0    1    1    0
 $EndComp
@@
 F 5 "GRM188R61C104KA01" H 6400 3200 60  0001 C CNN "Manufacturer Part Number"
 	1    6400 3200
-	1    0    0    -1
+	1    0    0    1
 $EndComp
 $Comp
@@
 L PWR_FLAG #FLG0123
 U 1 1 572E8DF0
-P 4750 4750
-F 0 "#FLG0123" H 4750 4845 50  0001 C CNN
-F 1 "PWR_FLAG" H 4750 4930 50  0000 C CNN
-F 2 "" H 4750 4750 50  0000 C CNN
-F 3 "" H 4750 4750 50  0000 C CNN
-	1    4750 4750
+P 4650 4750
+F 0 "#FLG0123" H 4650 4845 50  0001 C CNN
+F 1 "PWR_FLAG" H 4650 4930 50  0000 C CNN
+F 2 "" H 4650 4750 50  0000 C CNN
+F 3 "" H 4650 4750 50  0000 C CNN
+	1    4650 4750
 	-1   0    0    1
 $EndComp
-Connection ~ 4750 4750
+Connection ~ 4650 4750
 Text Label 5150 3700 0    60   ~ 0
 CON_D-
 Text Label 5150 3800 0    60   ~ 0
 CON_D+
+$Comp
+L TVS_SOT23 D17
+U 1 1 573FE61B
+P 5900 4500
+F 0 "D17" H 6130 4370 50  0000 C CNN
+F 1 "TVS_SOT23" H 6290 4290 50  0000 C CNN
+F 2 "TO_SOT_Packages_SMD:SOT-23" V 5800 4360 50  0001 C CNN
+F 3 "" V 5800 4360 50  0000 C CNN
+F 4 "Littelfuse" H 5900 4500 60  0001 C CNN "Manufacturer"
+F 5 "PGB102ST23WR" H 5900 4500 60  0001 C CNN "Manufacturer Part Number"
+	1    5900 4500
+	-1   0    0    1
+$EndComp
+Wire Wire Line
+	5900 4750 5900 4700
+$Comp
+L F_Small F1
+U 1 1 573FF331
+P 4800 3600
+F 0 "F1" H 4760 3660 50  0000 L CNN
+F 1 "1206L150" H 4680 3540 50  0000 L CNN
+F 2 "Resistors_SMD:R_1206_HandSoldering" H 4800 3600 50  0001 C CNN
+F 3 "" H 4800 3600 50  0000 C CNN
+F 4 "Littelfuse" H 4800 3600 60  0001 C CNN "Manufacturer"
+F 5 "1206L150THWR" H 4800 3600 60  0001 C CNN "Manufacturer Part Number"
+	1    4800 3600
+	1    0    0    -1
+$EndComp
+Wire Wire Line
+	4600 3600 4700 3600
+Wire Wire Line
+	4900 3600 5100 3600
 $EndSCHEMATC

Commit message: Started laying out FPGA
Parts:
- removed R58, R59: 27, Resistors_SMD:R_0603, symbol R
Connections:
- net labels removed: CON_D+, CON_D-
- wire segments 22 -> 20
Changed lines of the file:
@@
 D-
-$Comp
-L R R58
-U 1 1 56A8E4E2
-P 6500 3700
-F 0 "R58" V 6550 3950 50  0000 C CNN
-F 1 "27" V 6500 3700 50  0000 C CNN
-F 2 "Resistors_SMD:R_0603" V 6430 3700 50  0001 C CNN
-F 3 "" H 6500 3700 50  0000 C CNN
-F 4 "Panasonic" V 6500 3700 60  0001 C CNN "Manufacturer"
-F 5 "ERJ-3EKF27R0V" V 6500 3700 60  0001 C CNN "Manufacturer Part Number"
-	1    6500 3700
-	0    -1   -1   0
-$EndComp
 $Comp
 L PWR_FLAG #FLG0121
@@
 Connection ~ 6800 3000
 Wire Wire Line
-	6650 3800 6900 3800
+	4600 3800 6900 3800
 Wire Wire Line
-	6650 3700 6900 3700
+	4600 3700 6900 3700
 Connection ~ 7250 3000
 Wire Wire Line
@@
 	5100 3000 5100 4100
 Wire Wire Line
-	4600 3700 6350 3700
-Wire Wire Line
 	5800 3700 5800 4100
-Wire Wire Line
-	4600 3800 6350 3800
 Wire Wire Line
 	6000 3800 6000 4100
@@
 $EndComp
 $Comp
-L R R59
-U 1 1 572C16A2
-P 6500 3800
-F 0 "R59" V 6550 4050 50  0000 C CNN
-F 1 "27" V 6500 3800 50  0000 C CNN
-F 2 "Resistors_SMD:R_0603" V 6430 3800 50  0001 C CNN
-F 3 "" H 6500 3800 50  0000 C CNN
-F 4 "Panasonic" V 6500 3800 60  0001 C CNN "Manufacturer"
-F 5 "ERJ-3EKF27R0V" V 6500 3800 60  0001 C CNN "Manufacturer Part Number"
-	1    6500 3800
-	0    -1   -1   0
-$EndComp
-$Comp
 L PWR_FLAG #FLG0123
 U 1 1 572E8DF0
@@
 $EndComp
 Connection ~ 4650 4750
-Text Label 5150 3700 0    60   ~ 0
-CON_D-
-Text Label 5150 3800 0    60   ~ 0
-CON_D+
 $Comp
 L TVS_SOT23 D17

Commit message: Fixing up USB connector
- Had to go back through and re-annotate all the 0603 caps and
  resistors to the hand-solderding versions since those changes didn't
  make it back into the schematics the last time I tried.

- Added a new footprint for the USB connector to connect to all the
  shield pins.
Parts:
- removed P2: USB_OTG, headphones:SJ110578, symbol USB_OTG
- added P2: SJ110578, headphones:SJ110578, symbol SJ110578
- C43, C44: footprint Capacitors_SMD:C_0603 -> Capacitors_SMD:C_0603_HandSoldering
- FB1, R104: footprint Resistors_SMD:R_0603 -> Resistors_SMD:R_0603_HandSoldering
Connections:
- wire segments 20 -> 25
Changed lines of the file:
@@
 Comment4 ""
 $EndDescr
-$Comp
-L USB_OTG P2
-U 1 1 56A8D0CF
-P 4300 3800
-F 0 "P2" H 4625 3675 50  0000 C CNN
-F 1 "USB_OTG" H 4300 4000 50  0000 C CNN
-F 2 "headphones:SJ110578" V 4250 3700 50  0001 C CNN
-F 3 "" V 4250 3700 50  0000 C CNN
-F 4 "JAE Electronics" H 4300 3800 60  0001 C CNN "Manufacturer"
-F 5 "DX4R005JJ2R1800" H 4300 3800 60  0001 C CNN "Manufacturer Part Number"
-	1    4300 3800
-	0    -1   1    0
-$EndComp
 NoConn ~ 4600 3900
 $Comp
@@
 F 0 "FB1" V 5900 3200 50  0000 L CNN
 F 1 "BKP1608HS330-T" V 5800 2650 50  0000 L CNN
-F 2 "Resistors_SMD:R_0603" H 5850 3000 50  0001 C CNN
+F 2 "Resistors_SMD:R_0603_HandSoldering" H 5850 3000 50  0001 C CNN
 F 3 "" H 5850 3000 50  0000 C CNN
 F 4 "Taiyo Yuden" V 5850 3000 60  0001 C CNN "Manufacturer"
@@
 Connection ~ 4650 4350
 Wire Wire Line
-	4250 4350 4200 4350
+	3700 4350 4250 4350
 Connection ~ 4200 4350
 $Comp
@@
 F 0 "R104" V 4480 4350 50  0000 C CNN
 F 1 "0" V 4400 4350 50  0000 C CNN
-F 2 "Resistors_SMD:R_0603" V 4330 4350 50  0001 C CNN
+F 2 "Resistors_SMD:R_0603_HandSoldering" V 4330 4350 50  0001 C CNN
 F 3 "" H 4400 4350 50  0000 C CNN
 F 4 "Panasonic" V 4400 4350 60  0001 C CNN "Manufacturer"
@@
 F 0 "C43" H 5325 3300 50  0000 L CNN
 F 1 "0.01uF" H 5325 3100 50  0000 L CNN
-F 2 "Capacitors_SMD:C_0603" H 5338 3050 50  0001 C CNN
+F 2 "Capacitors_SMD:C_0603_HandSoldering" H 5338 3050 50  0001 C CNN
 F 3 "" H 5300 3200 50  0000 C CNN
 F 4 "Murata" H 5300 3200 60  0001 C CNN "Manufacturer"
@@
 F 0 "C44" H 6425 3300 50  0000 L CNN
 F 1 "0.1uF" H 6425 3100 50  0000 L CNN
-F 2 "Capacitors_SMD:C_0603" H 6438 3050 50  0001 C CNN
+F 2 "Capacitors_SMD:C_0603_HandSoldering" H 6438 3050 50  0001 C CNN
 F 3 "" H 6400 3200 50  0000 C CNN
 F 4 "Murata" H 6400 3200 60  0001 C CNN "Manufacturer"
@@
 Wire Wire Line
 	4900 3600 5100 3600
+$Comp
+L SJ110578 P2
+U 1 1 57692725
+P 4300 3800
+F 0 "P2" H 4625 3675 50  0000 C CNN
+F 1 "SJ110578" H 4300 4500 50  0000 C CNN
+F 2 "headphones:SJ110578" V 4250 3700 50  0001 C CNN
+F 3 "" V 4250 3700 50  0000 C CNN
+F 4 "JAE Electronics" H 4300 3800 60  0001 C CNN "Manufacturer"
+F 5 "DX4R005JJ2R1800" H 4300 3800 60  0001 C CNN "Manufacturer Part Number"
+	1    4300 3800
+	0    -1   1    0
+$EndComp
+Wire Wire Line
+	3700 4200 3700 4350
+Wire Wire Line
+	3800 4200 3800 4350
+Connection ~ 3800 4350
+Wire Wire Line
+	3900 4200 3900 4350
+Connection ~ 3900 4350
+Wire Wire Line
+	4000 4200 4000 4350
+Connection ~ 4000 4350
+Wire Wire Line
+	4100 4200 4100 4350
+Connection ~ 4100 4350
 $EndSCHEMATC
