File: pcb/cs5361.sch (KiCad schematic (older format))
At the start: 15 parts, among them U1 CS5361

Commit message: Began cleaning up ERC errors
Changed lines of the file:
@@
 $EndComp
 $Comp
-L GND #PWR4
+L GND #PWR04
 U 1 1 5688D779
 P 4850 3300
-F 0 "#PWR4" H 4850 3050 50  0001 C CNN
+F 0 "#PWR04" H 4850 3050 50  0001 C CNN
 F 1 "GND" H 4850 3150 50  0000 C CNN
 F 2 "" H 4850 3300 50  0000 C CNN
@@
 $EndComp
 $Comp
-L GND #PWR6
+L GND #PWR05
 U 1 1 5688D8BB
 P 6000 2400
-F 0 "#PWR6" H 6000 2150 50  0001 C CNN
+F 0 "#PWR05" H 6000 2150 50  0001 C CNN
 F 1 "GND" H 6000 2250 50  0000 C CNN
 F 2 "" H 6000 2400 50  0000 C CNN
@@
 $EndComp
 $Comp
-L GND #PWR7
+L GND #PWR06
 U 1 1 5688D8C1
 P 6300 2400
-F 0 "#PWR7" H 6300 2150 50  0001 C CNN
+F 0 "#PWR06" H 6300 2150 50  0001 C CNN
 F 1 "GND" H 6300 2250 50  0000 C CNN
 F 2 "" H 6300 2400 50  0000 C CNN
@@
 $EndComp
 $Comp
-L +5V #PWR5
+L +5V #PWR07
 U 1 1 5688D8C7
 P 6000 2000
-F 0 "#PWR5" H 6000 1850 50  0001 C CNN
+F 0 "#PWR07" H 6000 1850 50  0001 C CNN
 F 1 "+5V" H 6000 2140 50  0000 C CNN
 F 2 "" H 6000 2000 50  0000 C CNN
@@
 $EndComp
 $Comp
-L GND #PWR10
+L GND #PWR08
 U 1 1 5688D8DB
 P 7000 2400
-F 0 "#PWR10" H 7000 2150 50  0001 C CNN
+F 0 "#PWR08" H 7000 2150 50  0001 C CNN
 F 1 "GND" H 7000 2250 50  0000 C CNN
 F 2 "" H 7000 2400 50  0000 C CNN
@@
 $EndComp
 $Comp
-L GND #PWR13
+L GND #PWR09
 U 1 1 5688D8EF
 P 7800 2400
-F 0 "#PWR13" H 7800 2150 50  0001 C CNN
+F 0 "#PWR09" H 7800 2150 50  0001 C CNN
 F 1 "GND" H 7800 2250 50  0000 C CNN
 F 2 "" H 7800 2400 50  0000 C CNN
@@
 $EndComp
 $Comp
-L GND #PWR15
+L GND #PWR010
 U 1 1 5688D8F5
 P 8100 2400
-F 0 "#PWR15" H 8100 2150 50  0001 C CNN
+F 0 "#PWR010" H 8100 2150 50  0001 C CNN
 F 1 "GND" H 8100 2250 50  0000 C CNN
 F 2 "" H 8100 2400 50  0000 C CNN
@@
 $EndComp
 $Comp
-L +3.3V #PWR14
+L +3.3V #PWR011
 U 1 1 5688D8FB
 P 8100 2000
-F 0 "#PWR14" H 8100 1850 50  0001 C CNN
+F 0 "#PWR011" H 8100 1850 50  0001 C CNN
 F 1 "+3.3V" H 8100 2140 50  0000 C CNN
 F 2 "" H 8100 2000 50  0000 C CNN
@@
 	5200 3300 5600 3300
 $Comp
-L +3.3V #PWR16
+L +3.3V #PWR012
 U 1 1 5688D934
 P 8100 3000
-F 0 "#PWR16" H 8100 2850 50  0001 C CNN
+F 0 "#PWR012" H 8100 2850 50  0001 C CNN
 F 1 "+3.3V" H 8100 3140 50  0000 C CNN
 F 2 "" H 8100 3000 50  0000 C CNN
@@
 Wire Wire Line
 	7500 4200 8100 4200
-$Comp
-L +3.3V #PWR17
-U 1 1 56895CD4
-P 9250 1800
-F 0 "#PWR17" H 9250 1650 50  0001 C CNN
-F 1 "+3.3V" H 9250 1940 50  0000 C CNN
-F 2 "" H 9250 1800 50  0000 C CNN
-F 3 "" H 9250 1800 50  0000 C CNN
-	1    9250 1800
-	1    0    0    -1
-$EndComp
-$Comp
-L +5V #PWR19
-U 1 1 56895DE7
-P 9700 1800
-F 0 "#PWR19" H 9700 1650 50  0001 C CNN
-F 1 "+5V" H 9700 1940 50  0000 C CNN
-F 2 "" H 9700 1800 50  0000 C CNN
-F 3 "" H 9700 1800 50  0000 C CNN
-	1    9700 1800
-	1    0    0    -1
-$EndComp
-$Comp
-L GNDA #PWR18
-U 1 1 56896228
-P 9250 2400
-F 0 "#PWR18" H 9250 2150 50  0001 C CNN
-F 1 "GNDA" H 9250 2250 50  0000 C CNN
-F 2 "" H 9250 2400 50  0000 C CNN
-F 3 "" H 9250 2400 50  0000 C CNN
-	1    9250 2400
-	1    0    0    -1
-$EndComp
-$Comp
-L GND #PWR20
-U 1 1 5689633B
-P 9700 2400
-F 0 "#PWR20" H 9700 2150 50  0001 C CNN
-F 1 "GND" H 9700 2250 50  0000 C CNN
-F 2 "" H 9700 2400 50  0000 C CNN
-F 3 "" H 9700 2400 50  0000 C CNN
-	1    9700 2400
-	1    0    0    -1
-$EndComp
-$Comp
-L PWR_FLAG #FLG1
-U 1 1 568A2B2E
-P 9250 1800
-F 0 "#FLG1" H 9250 1895 50  0001 C CNN
-F 1 "PWR_FLAG" H 9250 1980 50  0000 C CNN
-F 2 "" H 9250 1800 50  0000 C CNN
-F 3 "" H 9250 1800 50  0000 C CNN
-	1    9250 1800
-	-1   0    0    1
-$EndComp
-$Comp
-L PWR_FLAG #FLG2
-U 1 1 568A2DF6
-P 9250 2400
-F 0 "#FLG2" H 9250 2495 50  0001 C CNN
-F 1 "PWR_FLAG" H 9250 2580 50  0000 C CNN
-F 2 "" H 9250 2400 50  0000 C CNN
-F 3 "" H 9250 2400 50  0000 C CNN
-	1    9250 2400
-	1    0    0    -1
-$EndComp
-$Comp
-L PWR_FLAG #FLG4
-U 1 1 568A2F13
-P 9700 2400
-F 0 "#FLG4" H 9700 2495 50  0001 C CNN
-F 1 "PWR_FLAG" H 9700 2580 50  0000 C CNN
-F 2 "" H 9700 2400 50  0000 C CNN
-F 3 "" H 9700 2400 50  0000 C CNN
-	1    9700 2400
-	1    0    0    -1
-$EndComp
-$Comp
-L PWR_FLAG #FLG3
-U 1 1 568A2FCE
-P 9700 1800
-F 0 "#FLG3" H 9700 1895 50  0001 C CNN
-F 1 "PWR_FLAG" H 9700 1980 50  0000 C CNN
-F 2 "" H 9700 1800 50  0000 C CNN
-F 3 "" H 9700 1800 50  0000 C CNN
-	1    9700 1800
-	-1   0    0    1
-$EndComp
 Wire Wire Line
 	7500 3500 7800 3500
@@
 	7500 3800 7800 3800
 $Comp
-L GNDA #PWR9
+L GNDA #PWR013
 U 1 1 56A11816
 P 6900 4600
-F 0 "#PWR9" H 6900 4350 50  0001 C CNN
+F 0 "#PWR013" H 6900 4350 50  0001 C CNN
 F 1 "GNDA" H 6900 4450 50  0000 C CNN
 F 2 "" H 6900 4600 50  0000 C CNN
@@
 $EndComp
 $Comp
-L GNDA #PWR8
+L GNDA #PWR014
 U 1 1 56A1187E
 P 6700 4600
-F 0 "#PWR8" H 6700 4350 50  0001 C CNN
+F 0 "#PWR014" H 6700 4350 50  0001 C CNN
 F 1 "GNDA" H 6700 4450 50  0000 C CNN
 F 2 "" H 6700 4600 50  0000 C CNN
@@
 $EndComp
 $Comp
-L GND #PWR12
+L GND #PWR015
 U 1 1 56A5923D
 P 7400 2400
-F 0 "#PWR12" H 7400 2150 50  0001 C CNN
+F 0 "#PWR015" H 7400 2150 50  0001 C CNN
 F 1 "GND" H 7400 2250 50  0000 C CNN
 F 2 "" H 7400 2400 50  0000 C CNN
@@
 Connection ~ 7000 2050
 $Comp
-L +3.3V #PWR11
+L +3.3V #PWR016
 U 1 1 56A593E0
 P 7400 2000
-F 0 "#PWR11" H 7400 1850 50  0001 C CNN
+F 0 "#PWR016" H 7400 1850 50  0001 C CNN
 F 1 "+3.3V" H 7400 2140 50  0000 C CNN
 F 2 "" H 7400 2000 50  0000 C CNN

Commit message: Cleaned up ERC
Connections:
- net labels removed: GNDA
Changed lines of the file:
@@
 $EndComp
 $Comp
-L GND #PWR4
+L GND #PWR04
 U 1 1 5688D779
 P 4850 3300
-F 0 "#PWR4" H 4850 3050 50  0001 C CNN
+F 0 "#PWR04" H 4850 3050 50  0001 C CNN
 F 1 "GND" H 4850 3150 50  0000 C CNN
 F 2 "" H 4850 3300 50  0000 C CNN
@@
 $EndComp
 $Comp
-L GND #PWR6
+L GND #PWR05
 U 1 1 5688D8BB
 P 6000 2400
-F 0 "#PWR6" H 6000 2150 50  0001 C CNN
+F 0 "#PWR05" H 6000 2150 50  0001 C CNN
 F 1 "GND" H 6000 2250 50  0000 C CNN
 F 2 "" H 6000 2400 50  0000 C CNN
@@
 $EndComp
 $Comp
-L GND #PWR7
+L GND #PWR06
 U 1 1 5688D8C1
 P 6300 2400
-F 0 "#PWR7" H 6300 2150 50  0001 C CNN
+F 0 "#PWR06" H 6300 2150 50  0001 C CNN
 F 1 "GND" H 6300 2250 50  0000 C CNN
 F 2 "" H 6300 2400 50  0000 C CNN
@@
 $EndComp
 $Comp
-L +5V #PWR5
+L +5V #PWR07
 U 1 1 5688D8C7
 P 6000 2000
-F 0 "#PWR5" H 6000 1850 50  0001 C CNN
+F 0 "#PWR07" H 6000 1850 50  0001 C CNN
 F 1 "+5V" H 6000 2140 50  0000 C CNN
 F 2 "" H 6000 2000 50  0000 C CNN
@@
 $EndComp
 $Comp
-L GND #PWR10
+L GND #PWR08
 U 1 1 5688D8DB
 P 7000 2400
-F 0 "#PWR10" H 7000 2150 50  0001 C CNN
+F 0 "#PWR08" H 7000 2150 50  0001 C CNN
 F 1 "GND" H 7000 2250 50  0000 C CNN
 F 2 "" H 7000 2400 50  0000 C CNN
@@
 $EndComp
 $Comp
-L GND #PWR13
+L GND #PWR09
 U 1 1 5688D8EF
 P 7800 2400
-F 0 "#PWR13" H 7800 2150 50  0001 C CNN
+F 0 "#PWR09" H 7800 2150 50  0001 C CNN
 F 1 "GND" H 7800 2250 50  0000 C CNN
 F 2 "" H 7800 2400 50  0000 C CNN
@@
 $EndComp
 $Comp
-L GND #PWR15
+L GND #PWR010
 U 1 1 5688D8F5
 P 8100 2400
-F 0 "#PWR15" H 8100 2150 50  0001 C CNN
+F 0 "#PWR010" H 8100 2150 50  0001 C CNN
 F 1 "GND" H 8100 2250 50  0000 C CNN
 F 2 "" H 8100 2400 50  0000 C CNN
@@
 $EndComp
 $Comp
-L +3.3V #PWR14
+L +3.3V #PWR011
 U 1 1 5688D8FB
 P 8100 2000
-F 0 "#PWR14" H 8100 1850 50  0001 C CNN
+F 0 "#PWR011" H 8100 1850 50  0001 C CNN
 F 1 "+3.3V" H 8100 2140 50  0000 C CNN
 F 2 "" H 8100 2000 50  0000 C CNN
@@
 	5200 3300 5600 3300
 $Comp
-L +3.3V #PWR16
+L +3.3V #PWR012
 U 1 1 5688D934
 P 8100 3000
-F 0 "#PWR16" H 8100 2850 50  0001 C CNN
+F 0 "#PWR012" H 8100 2850 50  0001 C CNN
 F 1 "+3.3V" H 8100 3140 50  0000 C CNN
 F 2 "" H 8100 3000 50  0000 C CNN
@@
 Wire Wire Line
 	7500 3800 7800 3800
-$Comp
-L GNDA #PWR9
-U 1 1 56A11816
-P 6900 4600
-F 0 "#PWR9" H 6900 4350 50  0001 C CNN
-F 1 "GNDA" H 6900 4450 50  0000 C CNN
-F 2 "" H 6900 4600 50  0000 C CNN
-F 3 "" H 6900 4600 50  0000 C CNN
-	1    6900 4600
-	1    0    0    -1
-$EndComp
-$Comp
-L GNDA #PWR8
-U 1 1 56A1187E
-P 6700 4600
-F 0 "#PWR8" H 6700 4350 50  0001 C CNN
-F 1 "GNDA" H 6700 4450 50  0000 C CNN
-F 2 "" H 6700 4600 50  0000 C CNN
-F 3 "" H 6700 4600 50  0000 C CNN
-	1    6700 4600
-	1    0    0    -1
-$EndComp
 $Sheet
 S 3600 3850 1300 400
@@
 $EndComp
 $Comp
-L GND #PWR12
+L GND #PWR013
 U 1 1 56A5923D
 P 7400 2400
-F 0 "#PWR12" H 7400 2150 50  0001 C CNN
+F 0 "#PWR013" H 7400 2150 50  0001 C CNN
 F 1 "GND" H 7400 2250 50  0000 C CNN
 F 2 "" H 7400 2400 50  0000 C CNN
@@
 Connection ~ 7000 2050
 $Comp
-L +3.3V #PWR11
+L +3.3V #PWR014
 U 1 1 56A593E0
 P 7400 2000
-F 0 "#PWR11" H 7400 1850 50  0001 C CNN
+F 0 "#PWR014" H 7400 1850 50  0001 C CNN
 F 1 "+3.3V" H 7400 2140 50  0000 C CNN
 F 2 "" H 7400 2000 50  0000 C CNN
@@
 $EndComp
 Connection ~ 7400 2050
+$Comp
+L GND #PWR015
+U 1 1 5717070F
+P 6900 4600
+F 0 "#PWR015" H 6900 4350 50  0001 C CNN
+F 1 "GND" H 6900 4450 50  0000 C CNN
+F 2 "" H 6900 4600 50  0000 C CNN
+F 3 "" H 6900 4600 50  0000 C CNN
+	1    6900 4600
+	1    0    0    -1
+$EndComp
+$Comp
+L GND #PWR016
+U 1 1 5717077D
+P 6700 4600
+F 0 "#PWR016" H 6700 4350 50  0001 C CNN
+F 1 "GND" H 6700 4450 50  0000 C CNN
+F 2 "" H 6700 4600 50  0000 C CNN
+F 3 "" H 6700 4600 50  0000 C CNN
+	1    6700 4600
+	1    0    0    -1
+$EndComp
 $EndSCHEMATC

Commit message: Latest work on footprints and BOM
Parts:
- C1: footprint (none) -> Capacitors_ThroughHole:C_Radial_D10_L20_P5; Manufacturer (none) -> Panasonic; Manufacturer Part Number (none) -> ECA-1HM221B
- C10, C3, C4, C6, C7: footprint (none) -> Capacitors_SMD:C_0603; Manufacturer (none) -> Murata; Manufacturer Part Number (none) -> GRM188R71E103KA01
- C2, C5, C8, C9: footprint (none) -> Capacitors_ThroughHole:C_Radial_D6.3_L11.2_P2.5; Manufacturer (none) -> Panasonic; Manufacturer Part Number (none) -> ECA-2EM010
- R1: value 68 -> 10K; footprint (none) -> Resistors_SMD:R_0603; Manufacturer (none) -> Panasonic; Manufacturer Part Number (none) -> ERJ-3GEYJ103V
- R2, R3: footprint (none) -> Resistors_SMD:R_0603; Manufacturer (none) -> Panasonic; Manufacturer Part Number (none) -> ERJ-3EKF68R0V
- R4: value 10K -> 68; footprint (none) -> Resistors_SMD:R_0603; Manufacturer (none) -> Panasonic; Manufacturer Part Number (none) -> ERJ-3EKF68R0V
- U1: footprint (none) -> Housings_SOIC:SOIC-24_7.5x15.4mm_Pitch1.27mm; Manufacturer (none) -> Cirrus Logic; Manufacturer Part Number (none) -> CS5381
Changed lines of the file:
@@
 	8050 3000 8100 3000
-$Comp
-L C C3
-U 1 1 5688D75D
-P 5600 3100
-F 0 "C3" H 5625 3200 50  0000 L CNN
-F 1 "0.01uF" H 5625 3000 50  0000 L CNN
-F 2 "" H 5638 2950 50  0000 C CNN
-F 3 "" H 5600 3100 50  0000 C CNN
-	1    5600 3100
-	1    0    0    -1
-$EndComp
-$Comp
-L C C4
-U 1 1 5688D764
-P 5600 3500
-F 0 "C4" H 5625 3600 50  0000 L CNN
-F 1 "0.01uF" H 5625 3400 50  0000 L CNN
-F 2 "" H 5638 3350 50  0000 C CNN
-F 3 "" H 5600 3500 50  0000 C CNN
-	1    5600 3500
-	1    0    0    -1
-$EndComp
 $Comp
 L CP C1
@@
 F 0 "C1" H 5225 3200 50  0000 L CNN
 F 1 "220uF" H 5225 3000 50  0000 L CNN
-F 2 "" H 5238 2950 50  0000 C CNN
+F 2 "Capacitors_ThroughHole:C_Radial_D10_L20_P5" H 5238 2950 50  0001 C CNN
 F 3 "" H 5200 3100 50  0000 C CNN
+F 4 "Panasonic" H 5200 3100 60  0001 C CNN "Manufacturer"
+F 5 "ECA-1HM221B" H 5200 3100 60  0001 C CNN "Manufacturer Part Number"
 	1    5200 3100
 	1    0    0    -1
-$EndComp
-$Comp
-L CP C2
-U 1 1 5688D772
-P 5200 3500
-F 0 "C2" H 5225 3600 50  0000 L CNN
-F 1 "1uF" H 5225 3400 50  0000 L CNN
-F 2 "" H 5238 3350 50  0000 C CNN
-F 3 "" H 5200 3500 50  0000 C CNN
-	1    5200 3500
-	-1   0    0    1
 $EndComp
 $Comp
@@
 F 0 "C5" H 6025 2350 50  0000 L CNN
 F 1 "1uF" H 6025 2150 50  0000 L CNN
-F 2 "" H 6038 2100 50  0000 C CNN
+F 2 "Capacitors_ThroughHole:C_Radial_D6.3_L11.2_P2.5" H 6038 2100 50  0001 C CNN
 F 3 "" H 6000 2250 50  0000 C CNN
+F 4 "Panasonic" H 6000 2250 60  0001 C CNN "Manufacturer"
+F 5 "ECA-2EM010" H 6000 2250 60  0001 C CNN "Manufacturer Part Number"
 	1    6000 2250
 	1    0    0    -1
@@
 F 0 "C6" H 6325 2350 50  0000 L CNN
 F 1 "0.01uF" H 6325 2150 50  0000 L CNN
-F 2 "" H 6338 2100 50  0000 C CNN
+F 2 "Capacitors_SMD:C_0603" H 6338 2100 50  0001 C CNN
 F 3 "" H 6300 2250 50  0000 C CNN
+F 4 "Murata" H 6300 2250 60  0001 C CNN "Manufacturer"
+F 5 "GRM188R71E103KA01" H 6300 2250 60  0001 C CNN "Manufacturer Part Number"
 	1    6300 2250
 	1    0    0    -1
@@
 $EndComp
 $Comp
-L C C7
-U 1 1 5688D8D4
-P 7000 2250
-F 0 "C7" H 7025 2350 50  0000 L CNN
-F 1 "0.01uF" H 7025 2150 50  0000 L CNN
-F 2 "" H 7038 2100 50  0000 C CNN
-F 3 "" H 7000 2250 50  0000 C CNN
-	1    7000 2250
-	1    0    0    -1
-$EndComp
-$Comp
 L GND #PWR08
 U 1 1 5688D8DB
@@
 $EndComp
 $Comp
-L CP C9
-U 1 1 5688D8E1
-P 7800 2250
-F 0 "C9" H 7825 2350 50  0000 L CNN
-F 1 "1uF" H 7825 2150 50  0000 L CNN
-F 2 "" H 7838 2100 50  0000 C CNN
-F 3 "" H 7800 2250 50  0000 C CNN
-	1    7800 2250
-	1    0    0    -1
-$EndComp
-$Comp
-L C C10
-U 1 1 5688D8E8
-P 8100 2250
-F 0 "C10" H 8125 2350 50  0000 L CNN
-F 1 "0.01uF" H 8125 2150 50  0000 L CNN
-F 2 "" H 8138 2100 50  0000 C CNN
-F 3 "" H 8100 2250 50  0000 C CNN
-	1    8100 2250
-	1    0    0    -1
-$EndComp
-$Comp
 L GND #PWR09
 U 1 1 5688D8EF
@@
 	1    8100 2000
 	1    0    0    -1
-$EndComp
-$Comp
-L R R4
-U 1 1 5688D909
-P 7900 3000
-F 0 "R4" V 7980 3000 50  0000 C CNN
-F 1 "10K" V 7900 3000 50  0000 C CNN
-F 2 "" V 7830 3000 50  0000 C CNN
-F 3 "" H 7900 3000 50  0000 C CNN
-	1    7900 3000
-	0    -1   -1   0
 $EndComp
 Wire Wire Line
@@
 F 0 "U1" H 6800 3750 50  0000 C CNN
 F 1 "CS5361" H 6800 3650 50  0000 C CNN
-F 2 "" H 6800 3500 50  0000 C CNN
+F 2 "Housings_SOIC:SOIC-24_7.5x15.4mm_Pitch1.27mm" H 6800 3500 50  0001 C CNN
 F 3 "" H 6800 3500 50  0000 C CNN
+F 4 "Cirrus Logic" H 6800 3700 60  0001 C CNN "Manufacturer"
+F 5 "CS5381" H 6800 3700 60  0001 C CNN "Manufacturer Part Number"
 	1    6800 3700
 	1    0    0    -1
@@
 L R R1
 U 1 1 56A427EF
-P 7750 4000
-F 0 "R1" V 7800 3800 50  0000 C CNN
-F 1 "68" V 7750 4000 50  0000 C CNN
-F 2 "" V 7680 4000 50  0000 C CNN
-F 3 "" H 7750 4000 50  0000 C CNN
-	1    7750 4000
+P 7900 3000
+F 0 "R1" V 8000 3050 50  0000 C CNN
+F 1 "10K" V 7900 3000 50  0000 C CNN
+F 2 "Resistors_SMD:R_0603" V 7830 3000 50  0001 C CNN
+F 3 "" H 7900 3000 50  0000 C CNN
+F 4 "Panasonic" V 7900 3000 60  0001 C CNN "Manufacturer"
+F 5 "ERJ-3GEYJ103V" V 7900 3000 60  0001 C CNN "Manufacturer Part Number"
+	1    7900 3000
 	0    -1   -1   0
 $EndComp
-$Comp
-L R R3
-U 1 1 56A42AAE
-P 7750 4300
-F 0 "R3" V 7800 4100 50  0000 C CNN
-F 1 "68" V 7750 4300 50  0000 C CNN
-F 2 "" V 7680 4300 50  0000 C CNN
-F 3 "" H 7750 4300 50  0000 C CNN
-	1    7750 4300
-	0    -1   -1   0
-$EndComp
-$Comp
-L R R2
-U 1 1 56A429C6
-P 7750 4100
-F 0 "R2" V 7800 3900 50  0000 C CNN
-F 1 "68" V 7750 4100 50  0000 C CNN
-F 2 "" V 7680 4100 50  0000 C CNN
-F 3 "" H 7750 4100 50  0000 C CNN
-	1    7750 4100
-	0    -1   -1   0
-$EndComp
 Wire Wire Line
 	7500 4000 7600 4000
@@
 Wire Wire Line
 	7900 4000 8100 4000
-$Comp
-L CP C8
-U 1 1 56A59237
-P 7400 2250
-F 0 "C8" H 7425 2350 50  0000 L CNN
-F 1 "1uF" H 7425 2150 50  0000 L CNN
-F 2 "" H 7438 2100 50  0000 C CNN
-F 3 "" H 7400 2250 50  0000 C CNN
-	1    7400 2250
-	1    0    0    -1
-$EndComp
 $Comp
 L GND #PWR013
@@
 	1    0    0    -1
 $EndComp
+$Comp
+L CP C8
+U 1 1 57147AD1
+P 7400 2250
+F 0 "C8" H 7425 2350 50  0000 L CNN
+F 1 "1uF" H 7425 2150 50  0000 L CNN
+F 2 "Capacitors_ThroughHole:C_Radial_D6.3_L11.2_P2.5" H 7438 2100 50  0001 C CNN
+F 3 "" H 7400 2250 50  0000 C CNN
+F 4 "Panasonic" H 7400 2250 60  0001 C CNN "Manufacturer"
+F 5 "ECA-2EM010" H 7400 2250 60  0001 C CNN "Manufacturer Part Number"
+	1    7400 2250
+	1    0    0    -1
+$EndComp
+$Comp
+L CP C9
+U 1 1 57147B7D
+P 7800 2250
+F 0 "C9" H 7825 2350 50  0000 L CNN
+F 1 "1uF" H 7825 2150 50  0000 L CNN
+F 2 "Capacitors_ThroughHole:C_Radial_D6.3_L11.2_P2.5" H 7838 2100 50  0001 C CNN
+F 3 "" H 7800 2250 50  0000 C CNN
+F 4 "Panasonic" H 7800 2250 60  0001 C CNN "Manufacturer"
+F 5 "ECA-2EM010" H 7800 2250 60  0001 C CNN "Manufacturer Part Number"
+	1    7800 2250
+	1    0    0    -1
+$EndComp
+$Comp
+L CP C2
+U 1 1 57148B1A
+P 5200 3500
+F 0 "C2" H 5225 3600 50  0000 L CNN
+F 1 "1uF" H 5225 3400 50  0000 L CNN
+F 2 "Capacitors_ThroughHole:C_Radial_D6.3_L11.2_P2.5" H 5238 3350 50  0001 C CNN
+F 3 "" H 5200 3500 50  0000 C CNN
+F 4 "Panasonic" H 5200 3500 60  0001 C CNN "Manufacturer"
+F 5 "ECA-2EM010" H 5200 3500 60  0001 C CNN "Manufacturer Part Number"
+	1    5200 3500
+	-1   0    0    1
+$EndComp
+$Comp
+L R R2
+U 1 1 5714D505
+P 7750 4000
+F 0 "R2" V 7700 3800 50  0000 C CNN
+F 1 "68" V 7750 4000 50  0000 C CNN
+F 2 "Resistors_SMD:R_0603" V 7680 4000 50  0001 C CNN
+F 3 "" H 7750 4000 50  0000 C CNN
+F 4 "Panasonic" V 7750 4000 60  0001 C CNN "Manufacturer"
+F 5 "ERJ-3EKF68R0V" V 7750 4000 60  0001 C CNN "Manufacturer Part Number"
+	1    7750 4000
+	0    1    1    0
+$EndComp
+$Comp
+L R R3
+U 1 1 5714D751
+P 7750 4100
+F 0 "R3" V 7700 3900 50  0000 C CNN
+F 1 "68" V 7750 4100 50  0000 C CNN
+F 2 "Resistors_SMD:R_0603" V 7680 4100 50  0001 C CNN
+F 3 "" H 7750 4100 50  0000 C CNN
+F 4 "Panasonic" V 7750 4100 60  0001 C CNN "Manufacturer"
+F 5 "ERJ-3EKF68R0V" V 7750 4100 60  0001 C CNN "Manufacturer Part Number"
+	1    7750 4100
+	0    1    1    0
+$EndComp
+$Comp
+L R R4
+U 1 1 5714D7CF
+P 7750 4300
+F 0 "R4" V 7700 4100 50  0000 C CNN
+F 1 "68" V 7750 4300 50  0000 C CNN
+F 2 "Resistors_SMD:R_0603" V 7680 4300 50  0001 C CNN
+F 3 "" H 7750 4300 50  0000 C CNN
+F 4 "Panasonic" V 7750 4300 60  0001 C CNN "Manufacturer"
+F 5 "ERJ-3EKF68R0V" V 7750 4300 60  0001 C CNN "Manufacturer Part Number"
+	1    7750 4300
+	0    1    1    0
+$EndComp
+$Comp
+L C C7
+U 1 1 571594D5
+P 7000 2250
+F 0 "C7" H 7025 2350 50  0000 L CNN
+F 1 "0.01uF" H 7025 2150 50  0000 L CNN
+F 2 "Capacitors_SMD:C_0603" H 7038 2100 50  0001 C CNN
+F 3 "" H 7000 2250 50  0000 C CNN
+F 4 "Murata" H 7000 2250 60  0001 C CNN "Manufacturer"
+F 5 "GRM188R71E103KA01" H 7000 2250 60  0001 C CNN "Manufacturer Part Number"
+	1    7000 2250
+	1    0    0    -1
+$EndComp
+$Comp
+L C C10
+U 1 1 5715956B
+P 8100 2250
+F 0 "C10" H 8125 2350 50  0000 L CNN
+F 1 "0.01uF" H 8125 2150 50  0000 L CNN
+F 2 "Capacitors_SMD:C_0603" H 8138 2100 50  0001 C CNN
+F 3 "" H 8100 2250 50  0000 C CNN
+F 4 "Murata" H 8100 2250 60  0001 C CNN "Manufacturer"
+F 5 "GRM188R71E103KA01" H 8100 2250 60  0001 C CNN "Manufacturer Part Number"
+	1    8100 2250
+	1    0    0    -1
+$EndComp
+$Comp
+L C C3
+U 1 1 57159614
+P 5600 3100
+F 0 "C3" H 5625 3200 50  0000 L CNN
+F 1 "0.01uF" H 5625 3000 50  0000 L CNN
+F 2 "Capacitors_SMD:C_0603" H 5638 2950 50  0001 C CNN
+F 3 "" H 5600 3100 50  0000 C CNN
+F 4 "Murata" H 5600 3100 60  0001 C CNN "Manufacturer"
+F 5 "GRM188R71E103KA01" H 5600 3100 60  0001 C CNN "Manufacturer Part Number"
+	1    5600 3100
+	1    0    0    -1
+$EndComp
+$Comp
+L C C4
+U 1 1 571596DC
+P 5600 3500
+F 0 "C4" H 5625 3600 50  0000 L CNN
+F 1 "0.01uF" H 5625 3400 50  0000 L CNN
+F 2 "Capacitors_SMD:C_0603" H 5638 3350 50  0001 C CNN
+F 3 "" H 5600 3500 50  0000 C CNN
+F 4 "Murata" H 5600 3500 60  0001 C CNN "Manufacturer"
+F 5 "GRM188R71E103KA01" H 5600 3500 60  0001 C CNN "Manufacturer Part Number"
+	1    5600 3500
+	1    0    0    -1
+$EndComp

Commit message: Fixing up some part numbers
Parts:
- U1: Manufacturer Part Number CS5381 -> CS5381-KSZ
Changed lines of the file:
@@
 F 3 "" H 6800 3500 50  0000 C CNN
 F 4 "Cirrus Logic" H 6800 3700 60  0001 C CNN "Manufacturer"
-F 5 "CS5381" H 6800 3700 60  0001 C CNN "Manufacturer Part Number"
+F 5 "CS5381-KSZ" H 6800 3700 60  0001 C CNN "Manufacturer Part Number"
 	1    6800 3700
 	1    0    0    -1
