File: pcb/cs5361.sch (KiCad schematic (older format))
At the start: 15 parts, among them U1 CS5361

Commit message: Added an oscillator for the ADC
Parts:
- added C110: 0.1uF, Capacitors_SMD:C_0603, symbol C
- added X4: 12.288MHz, headphones:Oscillator_SMD_2520_4Pads, symbol oscillator
Connections:
- net labels added: ADC_MCLK_EN
- net labels removed: ADC_MCLK
- wire segments 60 -> 69
Changed lines of the file:
@@
 Text HLabel 8100 4100 2    60   Output ~ 0
 ADC_SCLK
-Text HLabel 8100 4200 2    60   Input ~ 0
-ADC_MCLK
+Text HLabel 9950 3450 2    60   Input ~ 0
+ADC_MCLK_EN
 Text HLabel 8100 4300 2    60   Output ~ 0
 ADC_SDO
-Wire Wire Line
-	7500 4200 8100 4200
 Wire Wire Line
 	7500 3500 7800 3500
@@
 	1    0    0    -1
 $EndComp
+Wire Wire Line
+	9950 3450 9900 3450
+$Comp
+L GND #PWR017
+U 1 1 57484B7E
+P 8950 3500
+F 0 "#PWR017" H 8950 3250 50  0001 C CNN
+F 1 "GND" H 8950 3350 50  0000 C CNN
+F 2 "" H 8950 3500 50  0000 C CNN
+F 3 "" H 8950 3500 50  0000 C CNN
+	1    8950 3500
+	1    0    0    -1
+$EndComp
+Wire Wire Line
+	9000 3450 8950 3450
+Wire Wire Line
+	8950 3450 8950 3500
+$Comp
+L +3.3V #PWR018
+U 1 1 57484B89
+P 10250 2700
+F 0 "#PWR018" H 10250 2550 50  0001 C CNN
+F 1 "+3.3V" H 10250 2840 50  0000 C CNN
+F 2 "" H 10250 2700 50  0000 C CNN
+F 3 "" H 10250 2700 50  0000 C CNN
+	1    10250 2700
+	-1   0    0    -1
+$EndComp
+$Comp
+L GND #PWR019
+U 1 1 57484B8F
+P 10250 3100
+F 0 "#PWR019" H 10250 2850 50  0001 C CNN
+F 1 "GND" H 10250 2950 50  0000 C CNN
+F 2 "" H 10250 3100 50  0000 C CNN
+F 3 "" H 10250 3100 50  0000 C CNN
+	1    10250 3100
+	1    0    0    -1
+$EndComp
+Wire Wire Line
+	9900 3350 9950 3350
+Wire Wire Line
+	9950 3350 9950 2750
+Wire Wire Line
+	9950 2750 10250 2750
+Wire Wire Line
+	10250 2700 10250 2800
+Connection ~ 10250 2750
+$Comp
+L oscillator X4
+U 1 1 57484B9C
+P 9450 3400
+F 0 "X4" H 9250 3600 60  0000 C CNN
+F 1 "12.288MHz" H 9450 3200 60  0000 C CNN
+F 2 "headphones:Oscillator_SMD_2520_4Pads" H 9450 3400 60  0001 C CNN
+F 3 "" H 9450 3400 60  0000 C CNN
+F 4 "Microchip" H 9450 3400 60  0001 C CNN "Manufacturer"
+F 5 "DSC1033DI2-012.2880" H 9450 3400 60  0001 C CNN "Manufacturer Part Number"
+	1    9450 3400
+	-1   0    0    -1
+$EndComp
+$Comp
+L C C110
+U 1 1 57484BA5
+P 10250 2950
+F 0 "C110" H 10275 3050 50  0000 L CNN
+F 1 "0.1uF" H 10275 2850 50  0000 L CNN
+F 2 "Capacitors_SMD:C_0603" H 10288 2800 50  0001 C CNN
+F 3 "" H 10250 2950 50  0000 C CNN
+F 4 "Murata" H 10250 2950 60  0001 C CNN "Manufacturer"
+F 5 "GRM188R61C104KA01" H 10250 2950 60  0001 C CNN "Manufacturer Part Number"
+	1    10250 2950
+	-1   0    0    -1
+$EndComp
+Wire Wire Line
+	7500 4200 8800 4200
+Wire Wire Line
+	8800 4200 8800 3350
+Wire Wire Line
+	8800 3350 9000 3350
 $EndSCHEMATC

Commit message: Fixed placement of series termination resistors
I had the logical placement of the series termination resistors wrong
in the schematics (i.e. I had them placed at the source rather than
the load) so I moved all those around to the correct sheets.  I also
moved the ADC resistors in the layout, but haven't gotten to the DAC
ones yet.
Parts:
- removed R2, R3, R4: 68, Resistors_SMD:R_0603, symbol R
Connections:
- wire segments 69 -> 66
Changed lines of the file:
@@
 $EndComp
 Wire Wire Line
-	7500 4000 7600 4000
+	7500 4000 8100 4000
 Wire Wire Line
-	7500 4100 7600 4100
+	7500 4100 8100 4100
 Wire Wire Line
-	7500 4300 7600 4300
-Wire Wire Line
-	7900 4300 8100 4300
-Wire Wire Line
-	7900 4100 8100 4100
-Wire Wire Line
-	7900 4000 8100 4000
+	7500 4300 8100 4300
 $Comp
 L GND #PWR013
@@
 $EndComp
 $Comp
-L R R2
-U 1 1 5714D505
-P 7750 4000
-F 0 "R2" V 7700 3800 50  0000 C CNN
-F 1 "68" V 7750 4000 50  0000 C CNN
-F 2 "Resistors_SMD:R_0603" V 7680 4000 50  0001 C CNN
-F 3 "" H 7750 4000 50  0000 C CNN
-F 4 "Panasonic" V 7750 4000 60  0001 C CNN "Manufacturer"
-F 5 "ERJ-3EKF68R0V" V 7750 4000 60  0001 C CNN "Manufacturer Part Number"
-	1    7750 4000
-	0    -1   -1   0
-$EndComp
-$Comp
-L R R3
-U 1 1 5714D751
-P 7750 4100
-F 0 "R3" V 7700 3900 50  0000 C CNN
-F 1 "68" V 7750 4100 50  0000 C CNN
-F 2 "Resistors_SMD:R_0603" V 7680 4100 50  0001 C CNN
-F 3 "" H 7750 4100 50  0000 C CNN
-F 4 "Panasonic" V 7750 4100 60  0001 C CNN "Manufacturer"
-F 5 "ERJ-3EKF68R0V" V 7750 4100 60  0001 C CNN "Manufacturer Part Number"
-	1    7750 4100
-	0    -1   -1   0
-$EndComp
-$Comp
-L R R4
-U 1 1 5714D7CF
-P 7750 4300
-F 0 "R4" V 7700 4100 50  0000 C CNN
-F 1 "68" V 7750 4300 50  0000 C CNN
-F 2 "Resistors_SMD:R_0603" V 7680 4300 50  0001 C CNN
-F 3 "" H 7750 4300 50  0000 C CNN
-F 4 "Panasonic" V 7750 4300 60  0001 C CNN "Manufacturer"
-F 5 "ERJ-3EKF68R0V" V 7750 4300 60  0001 C CNN "Manufacturer Part Number"
-	1    7750 4300
-	0    -1   -1   0
-$EndComp
-$Comp

Commit message: Fixing up USB connector
- Had to go back through and re-annotate all the 0603 caps and
  resistors to the hand-solderding versions since those changes didn't
  make it back into the schematics the last time I tried.

- Added a new footprint for the USB connector to connect to all the
  shield pins.
Parts:
- C10, C110, C3, C4, C6, C7: footprint Capacitors_SMD:C_0603 -> Capacitors_SMD:C_0603_HandSoldering
- R1: footprint Resistors_SMD:R_0603 -> Resistors_SMD:R_0603_HandSoldering
Changed lines of the file:
@@
 F 0 "C6" H 6325 2350 50  0000 L CNN
 F 1 "0.01uF" H 6325 2150 50  0000 L CNN
-F 2 "Capacitors_SMD:C_0603" H 6338 2100 50  0001 C CNN
+F 2 "Capacitors_SMD:C_0603_HandSoldering" H 6338 2100 50  0001 C CNN
 F 3 "" H 6300 2250 50  0000 C CNN
 F 4 "Murata" H 6300 2250 60  0001 C CNN "Manufacturer"
@@
 F 0 "R1" V 8000 3050 50  0000 C CNN
 F 1 "10K" V 7900 3000 50  0000 C CNN
-F 2 "Resistors_SMD:R_0603" V 7830 3000 50  0001 C CNN
+F 2 "Resistors_SMD:R_0603_HandSoldering" V 7830 3000 50  0001 C CNN
 F 3 "" H 7900 3000 50  0000 C CNN
 F 4 "Panasonic" V 7900 3000 60  0001 C CNN "Manufacturer"
@@
 F 0 "C7" H 7025 2350 50  0000 L CNN
 F 1 "0.01uF" H 7025 2150 50  0000 L CNN
-F 2 "Capacitors_SMD:C_0603" H 7038 2100 50  0001 C CNN
+F 2 "Capacitors_SMD:C_0603_HandSoldering" H 7038 2100 50  0001 C CNN
 F 3 "" H 7000 2250 50  0000 C CNN
 F 4 "Murata" H 7000 2250 60  0001 C CNN "Manufacturer"
@@
 F 0 "C10" H 8125 2350 50  0000 L CNN
 F 1 "0.01uF" H 8125 2150 50  0000 L CNN
-F 2 "Capacitors_SMD:C_0603" H 8138 2100 50  0001 C CNN
+F 2 "Capacitors_SMD:C_0603_HandSoldering" H 8138 2100 50  0001 C CNN
 F 3 "" H 8100 2250 50  0000 C CNN
 F 4 "Murata" H 8100 2250 60  0001 C CNN "Manufacturer"
@@
 F 0 "C3" H 5625 3200 50  0000 L CNN
 F 1 "0.01uF" H 5625 3000 50  0000 L CNN
-F 2 "Capacitors_SMD:C_0603" H 5638 2950 50  0001 C CNN
+F 2 "Capacitors_SMD:C_0603_HandSoldering" H 5638 2950 50  0001 C CNN
 F 3 "" H 5600 3100 50  0000 C CNN
 F 4 "Murata" H 5600 3100 60  0001 C CNN "Manufacturer"
@@
 F 0 "C4" H 5625 3600 50  0000 L CNN
 F 1 "0.01uF" H 5625 3400 50  0000 L CNN
-F 2 "Capacitors_SMD:C_0603" H 5638 3350 50  0001 C CNN
+F 2 "Capacitors_SMD:C_0603_HandSoldering" H 5638 3350 50  0001 C CNN
 F 3 "" H 5600 3500 50  0000 C CNN
 F 4 "Murata" H 5600 3500 60  0001 C CNN "Manufacturer"
@@
 F 0 "C110" H 10275 3050 50  0000 L CNN
 F 1 "0.1uF" H 10275 2850 50  0000 L CNN
-F 2 "Capacitors_SMD:C_0603" H 10288 2800 50  0001 C CNN
+F 2 "Capacitors_SMD:C_0603_HandSoldering" H 10288 2800 50  0001 C CNN
 F 3 "" H 10250 2950 50  0000 C CNN
 F 4 "Murata" H 10250 2950 60  0001 C CNN "Manufacturer"

Commit message: Added sense resistors everywhere
Parts:
- added R105, R92, R93, R98: 0.01, symbol R
Connections:
- wire segments 66 -> 74

Commit message: Still need to route all the new resistors
Parts:
- R105, R92, R93, R98: footprint (none) -> Resistors_SMD:R_0603_HandSoldering
Changed lines of the file:
@@
 F 0 "R92" V 5780 2050 50  0000 C CNN
 F 1 "0.01" V 5700 2050 50  0000 C CNN
-F 2 "" V 5630 2050 50  0000 C CNN
+F 2 "Resistors_SMD:R_0603_HandSoldering" V 5630 2050 50  0001 C CNN
 F 3 "" H 5700 2050 50  0000 C CNN
 	1    5700 2050
@@
 F 0 "R93" V 7730 2050 50  0000 C CNN
 F 1 "0.01" V 7650 2050 50  0000 C CNN
-F 2 "" V 7580 2050 50  0000 C CNN
+F 2 "Resistors_SMD:R_0603_HandSoldering" V 7580 2050 50  0001 C CNN
 F 3 "" H 7650 2050 50  0000 C CNN
 	1    7650 2050
@@
 F 0 "R98" V 8880 2050 50  0000 C CNN
 F 1 "0.01" V 8800 2050 50  0000 C CNN
-F 2 "" V 8730 2050 50  0000 C CNN
+F 2 "Resistors_SMD:R_0603_HandSoldering" V 8730 2050 50  0001 C CNN
 F 3 "" H 8800 2050 50  0000 C CNN
 	1    8800 2050
@@
 F 0 "R105" V 10580 2750 50  0000 C CNN
 F 1 "0.01" V 10500 2750 50  0000 C CNN
-F 2 "" V 10430 2750 50  0000 C CNN
+F 2 "Resistors_SMD:R_0603_HandSoldering" V 10430 2750 50  0001 C CNN
 F 3 "" H 10500 2750 50  0000 C CNN
 	1    10500 2750

Commit message: Cleanup and added testpoints
Cleaned up some of the schematic layout without changing any nets.  Also
added testpoints to all the power rails for easy debug.
Other:
- note removed: "I/O runs at VL, so 3.3V"

Commit message: More cleanup and switched sense resistors
Increased the resistance of the current sense resistors up to 0.1 ohm.
Parts:
- R105, R92, R93, R98: value 0.01 -> 0.1
Changed lines of the file:
@@
 P 4950 2250
 F 0 "R92" V 5030 2250 50  0000 C CNN
-F 1 "0.01" V 4950 2250 50  0000 C CNN
+F 1 "0.1" V 4950 2250 50  0000 C CNN
 F 2 "Resistors_SMD:R_0603_HandSoldering" V 4880 2250 50  0001 C CNN
 F 3 "" H 4950 2250 50  0000 C CNN
@@
 P 6900 2250
 F 0 "R93" V 6980 2250 50  0000 C CNN
-F 1 "0.01" V 6900 2250 50  0000 C CNN
+F 1 "0.1" V 6900 2250 50  0000 C CNN
 F 2 "Resistors_SMD:R_0603_HandSoldering" V 6830 2250 50  0001 C CNN
 F 3 "" H 6900 2250 50  0000 C CNN
@@
 P 8050 2250
 F 0 "R98" V 8130 2250 50  0000 C CNN
-F 1 "0.01" V 8050 2250 50  0000 C CNN
+F 1 "0.1" V 8050 2250 50  0000 C CNN
 F 2 "Resistors_SMD:R_0603_HandSoldering" V 7980 2250 50  0001 C CNN
 F 3 "" H 8050 2250 50  0000 C CNN
@@
 P 9750 2950
 F 0 "R105" V 9830 2950 50  0000 C CNN
-F 1 "0.01" V 9750 2950 50  0000 C CNN
+F 1 "0.1" V 9750 2950 50  0000 C CNN
 F 2 "Resistors_SMD:R_0603_HandSoldering" V 9680 2950 50  0001 C CNN
 F 3 "" H 9750 2950 50  0000 C CNN
