File: pcb/NYCDB-01.sch (KiCad schematic (older format))
At the start: 6 parts, among them J1 AUDIO_JACK, P1 CONN_BATT, SW1 SW_POWER

Commit message: Added footprints to testpoints
Parts:
- W1, W2, W3: footprint (none) -> Wire_Pads:SolderWirePad_single_1mmDrill
Changed lines of the file:
@@
 F 0 "W1" H 9450 3020 50  0000 C CNN
 F 1 "LEFT" H 9450 2950 50  0000 C CNN
-F 2 "" H 9650 2750 50  0000 C CNN
+F 2 "Wire_Pads:SolderWirePad_single_1mmDrill" H 9650 2750 50  0001 C CNN
 F 3 "" H 9650 2750 50  0000 C CNN
 	1    9450 2750
@@
 F 0 "W2" H 9800 3020 50  0000 C CNN
 F 1 "RIGHT" H 9800 2950 50  0000 C CNN
-F 2 "" H 10000 2750 50  0000 C CNN
+F 2 "Wire_Pads:SolderWirePad_single_1mmDrill" H 10000 2750 50  0001 C CNN
 F 3 "" H 10000 2750 50  0000 C CNN
 	1    9800 2750
@@
 F 0 "W3" H 10150 3020 50  0000 C CNN
 F 1 "GND" H 10150 2950 50  0000 C CNN
-F 2 "" H 10350 2750 50  0000 C CNN
+F 2 "Wire_Pads:SolderWirePad_single_1mmDrill" H 10350 2750 50  0001 C CNN
 F 3 "" H 10350 2750 50  0000 C CNN
 	1    10150 2750

Commit message: Added an oscillator for the ADC
Changed lines of the file:
@@
 F8 "ADC_SCLK" O R 3900 3550 60
 F9 "ADC_SDO" O R 3900 3750 60
-F10 "ADC_MCLK" I R 3900 3450 60
+F10 "ADC_MCLK_EN" I R 3900 3450 60
 F11 "ADC_I2S_LJ" I R 3900 2850 60
 F12 "ADC_MS" I R 3900 2950 60
@@
 F5 "ADC_LRCLK" I L 4850 3650 60
 F6 "ADC_SCLK" I L 4850 3550 60
-F7 "ADC_MCLK" O L 4850 3450 60
+F7 "ADC_MCLK_EN" O L 4850 3450 60
 F8 "ADC_SDO" I L 4850 3750 60
 F9 "ADC_I2S_LJ" O L 4850 2850 60

Commit message: Replaced output test pads with an audio jack
Parts:
- removed W1: LEFT, Wire_Pads:SolderWirePad_single_1mmDrill, symbol TEST_1P
- removed W2: RIGHT, Wire_Pads:SolderWirePad_single_1mmDrill, symbol TEST_1P
- removed W3: GND, Wire_Pads:SolderWirePad_single_1mmDrill, symbol TEST_1P
- added J2: AUDIO_JACK, headphones:SJ1-351XN, symbol AUDIO_JACK
Connections:
- wire segments 59 -> 60
Changed lines of the file:
@@
 Wire Wire Line
 	2750 2550 2850 2550
-$Comp
-L TEST_1P W1
-U 1 1 56A69CBC
-P 9450 2750
-F 0 "W1" H 9450 3020 50  0000 C CNN
-F 1 "LEFT" H 9450 2950 50  0000 C CNN
-F 2 "Wire_Pads:SolderWirePad_single_1mmDrill" H 9650 2750 50  0001 C CNN
-F 3 "" H 9650 2750 50  0000 C CNN
-	1    9450 2750
-	-1   0    0    1
-$EndComp
-$Comp
-L TEST_1P W2
-U 1 1 56A6A2A1
-P 9800 2750
-F 0 "W2" H 9800 3020 50  0000 C CNN
-F 1 "RIGHT" H 9800 2950 50  0000 C CNN
-F 2 "Wire_Pads:SolderWirePad_single_1mmDrill" H 10000 2750 50  0001 C CNN
-F 3 "" H 10000 2750 50  0000 C CNN
-	1    9800 2750
-	-1   0    0    1
-$EndComp
-$Comp
-L TEST_1P W3
-U 1 1 56A6A43B
-P 10150 2750
-F 0 "W3" H 10150 3020 50  0000 C CNN
-F 1 "GND" H 10150 2950 50  0000 C CNN
-F 2 "Wire_Pads:SolderWirePad_single_1mmDrill" H 10350 2750 50  0001 C CNN
-F 3 "" H 10350 2750 50  0000 C CNN
-	1    10150 2750
-	-1   0    0    1
-$EndComp
-Wire Wire Line
-	8850 2550 9800 2550
-Wire Wire Line
-	9800 2550 9800 2750
-Wire Wire Line
-	8850 2650 9450 2650
-Wire Wire Line
-	9450 2650 9450 2750
-$Comp
-L GND #PWR01
-U 1 1 56A6B291
-P 10400 2800
-F 0 "#PWR01" H 10400 2550 50  0001 C CNN
-F 1 "GND" H 10400 2650 50  0000 C CNN
-F 2 "" H 10400 2800 50  0000 C CNN
-F 3 "" H 10400 2800 50  0000 C CNN
-	1    10400 2800
-	1    0    0    -1
-$EndComp
-Wire Wire Line
-	10150 2750 10150 2700
-Wire Wire Line
-	10150 2700 10400 2700
-Wire Wire Line
-	10400 2700 10400 2800
 $Sheet
 S 7600 4450 1250 1050
@@
 	8850 4550 9450 4550
 $Comp
-L GND #PWR02
+L GND #PWR01
 U 1 1 56A8BB9A
 P 9550 4550
-F 0 "#PWR02" H 9550 4300 50  0001 C CNN
+F 0 "#PWR01" H 9550 4300 50  0001 C CNN
 F 1 "GND" H 9550 4400 50  0000 C CNN
 F 2 "" H 9550 4550 50  0000 C CNN
@@
 Connection ~ 9450 4550
 $Comp
-L GND #PWR03
+L GND #PWR02
 U 1 1 56A8D7D0
 P 10000 5250
-F 0 "#PWR03" H 10000 5000 50  0001 C CNN
+F 0 "#PWR02" H 10000 5000 50  0001 C CNN
 F 1 "GND" H 10000 5100 50  0000 C CNN
 F 2 "" H 10000 5250 50  0000 C CNN
@@
 F0 "TI DAC" 60
 F1 "ti_dac.sch" 60
-F2 "OUTL" O R 8850 2650 60
-F3 "OUTR" O R 8850 2550 60
+F2 "OUTL" O R 8850 2550 60
+F3 "OUTR" O R 8850 2650 60
 F4 "DAC_LRCK" I L 7600 3750 60
 F5 "DAC_BCK" I L 7600 3850 60
@@
 Text Notes 9100 5650 0    60   ~ 0
 TODO: ESD protection
+$Comp
+L AUDIO_JACK J2
+U 1 1 574BD570
+P 9750 2900
+F 0 "J2" H 9750 3000 60  0000 C CNN
+F 1 "AUDIO_JACK" H 9750 2350 60  0000 C CNN
+F 2 "headphones:SJ1-351XN" H 9750 3100 60  0001 C CNN
+F 3 "" H 9750 3100 60  0000 C CNN
+F 4 "CUI" H 9750 2900 60  0001 C CNN "Manufacturer"
+F 5 "SJ1-3513N" H 9750 2900 60  0001 C CNN "Manufacturer Part Number"
+	1    9750 2900
+	-1   0    0    1
+$EndComp
+Wire Wire Line
+	8850 2550 9150 2550
+Wire Wire Line
+	9150 2550 9150 2450
+Wire Wire Line
+	9150 2450 9400 2450
+Wire Wire Line
+	8850 2650 9150 2650
+Wire Wire Line
+	9150 2650 9150 2800
+Wire Wire Line
+	9150 2800 9400 2800
+$Comp
+L GND #PWR03
+U 1 1 574CA450
+P 9350 3000
+F 0 "#PWR03" H 9350 2750 50  0001 C CNN
+F 1 "GND" H 9350 2850 50  0000 C CNN
+F 2 "" H 9350 3000 50  0000 C CNN
+F 3 "" H 9350 3000 50  0000 C CNN
+	1    9350 3000
+	1    0    0    -1
+$EndComp
+Wire Wire Line
+	9400 2900 9350 2900
+Wire Wire Line
+	9350 2900 9350 3000
 $EndSCHEMATC
